File: kicad/Vega816/Accessories/C64VIA1.kicad_sch (KiCad schematic)
At the start: 5 parts, among them J102 VIA Port

Commit message: update
Connections:
- net ~{RESTORE} is gone; now on net CB1: J?.3 (Pin_3)
- no-connect marks 5 -> 4
Other:
- note added: "To 8580/6581 SID"
- note added: "~{RESTORE} key is wired to NMI on the Commodore 64. Here it is wired to CB1 for use as a potential IRQ source (See W65C22 datasheet)."
Changed lines of the file:
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@@
   (no_connect (at 78.74 151.13))
   (no_connect (at 78.74 102.87))
-  (no_connect (at 78.74 105.41))
   (no_connect (at 27.94 104.14))
   (wire (pts (xy 187.96 114.3) (xy 200.66 114.3))
@@
     (stroke (width 0) (type default) (color 0 0 0 0))
   )
-  (wire (pts (xy 27.94 105.41) (xy 41.91 105.41))
+  (wire (pts (xy 27.94 105.41) (xy 38.1 105.41))
     (stroke (width 0) (type default) (color 0 0 0 0))
   )
@@
     (stroke (width 0) (type default) (color 0 0 0 0))
   )
+  (wire (pts (xy 40.64 99.06) (xy 40.64 85.09))
+    (stroke (width 0) (type default) (color 0 0 0 0))
+  )
   (wire (pts (xy 36.83 116.84) (xy 73.66 116.84))
     (stroke (width 0) (type default) (color 0 0 0 0))
@@
     (stroke (width 0) (type default) (color 0 0 0 0))
   )
-  (wire (pts (xy 41.91 105.41) (xy 41.91 69.85))
+  (wire (pts (xy 38.1 105.41) (xy 38.1 99.06))
     (stroke (width 0) (type default) (color 0 0 0 0))
   )
@@
     (stroke (width 0) (type default) (color 0 0 0 0))
   )
-  (wire (pts (xy 41.91 69.85) (xy 248.92 69.85))
+  (wire (pts (xy 38.1 99.06) (xy 40.64 99.06))
     (stroke (width 0) (type default) (color 0 0 0 0))
   )
@@
     (stroke (width 0) (type default) (color 0 0 0 0))
   )
-  (wire (pts (xy 78.74 105.41) (xy 73.66 105.41))
+  (wire (pts (xy 73.66 105.41) (xy 88.9 105.41))
     (stroke (width 0) (type default) (color 0 0 0 0))
   )
@@
     (stroke (width 0) (type default) (color 0 0 0 0))
   )
+  (wire (pts (xy 40.64 85.09) (xy 88.9 85.09))
+    (stroke (width 0) (type default) (color 0 0 0 0))
+  )
   (wire (pts (xy 55.88 143.51) (xy 55.88 139.7))
     (stroke (width 0) (type default) (color 0 0 0 0))
@@
     (stroke (width 0) (type default) (color 0 0 0 0))
   )
+  (wire (pts (xy 88.9 85.09) (xy 88.9 105.41))
+    (stroke (width 0) (type default) (color 0 0 0 0))
+  )
   (wire (pts (xy 149.86 133.35) (xy 161.29 133.35))
     (stroke (width 0) (type default) (color 0 0 0 0))
@@
   )
   (text "Port B, keyboard matrix rows and joystick #1. Bits:\nPBx 0 = A key is currently being pressed in keyboard matrix row #x, in the column selected on PA\nPB0: 0 = Port 1 joystick up pressed.\nPB1: 0 = Port 1 joystick down pressed.\nPB2: 0 = Port 1 joystick left pressed.\nPB3: 0 = Port 1 joystick right pressed.\nPB4: 0 = Port 1 joystick fire pressed."
-    (at 87.63 49.53 0)
+    (at 80.01 80.01 0)
+    (effects (font (size 1.27 1.27)) (justify left bottom))
+  )
+  (text "To 8580/6581 SID" (at 246.38 91.44 0)
     (effects (font (size 1.27 1.27)) (justify left bottom))
   )
   (text "Port A, keyboard matrix columns and joystick #2. Read bits:\nRead:\nPA0: 0 = Port 2 joystick up pressed.\nPA1: 0 = Port 2 joystick down pressed.\nPA2: 0 = Port 2 joystick left pressed.\nPA3: 0 = Port 2 joystick right pressed.\nPA4: 0 = Port 2 joystick fire pressed.\nWrite:\nBit #x: 0 = Select keyboard matrix column #x.\nPA6, PA7: Paddle selection; %01 = Paddle #1; %10 = Paddle #2."
-    (at 16.51 55.88 0)
+    (at 80.01 181.61 0)
+    (effects (font (size 1.27 1.27)) (justify left bottom))
+  )
+  (text "~{RESTORE} key \nis wired to NMI on the Commodore 64. \nHere it is wired to CB1 \nfor use as a potential IRQ \nsource (See W65C22 datasheet)."
+    (at 90.17 95.25 0)
     (effects (font (size 1.27 1.27)) (justify left bottom))
   )
@@
       (effects (font (size 1.27 1.27)) (justify left) hide)
     )
-  )
-  (global_label "~{RESTORE}" (shape output) (at 248.92 69.85 0) (fields_autoplaced)
-    (effects (font (size 1.27 1.27)) (justify left))
-    (property "Intersheet References" "${INTERSHEET_REFS}" (id 0) (at 259.6788 69.7706 0)
-      (effects (font (size 1.27 1.27)) (justify left) hide)
-    )
