File: kicad/Vega816/Accessories/EaterPS2Interface.kicad_sch (KiCad schematic)
At the start: 14 parts, among them J102 VIA Port

Commit message: update
Other:
- note added: "VIA Port Device Ben Eater PS/2 Interface https://beneater.net/6502"
- note removed: "VIA Port Device Ben Eater PS/2 Interface"
Changed lines of the file:
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@@
     (stroke (width 0) (type default) (color 0 0 0 0))
   )
-  (text "VIA Port Device\nBen Eater PS/2 Interface\n" (at 16.51 34.29 0)
+  (text "VIA Port Device\nBen Eater PS/2 Interface\nhttps://beneater.net/6502\n"
+    (at 19.05 43.18 0)
     (effects (font (size 5 5)) (justify left bottom))
   )

Commit message: irq
Parts:
- added C?: C, symbol Device:C
- added D?: 1N914, Diode_THT:D_DO-35_SOD27_P7.62mm_Horizontal, symbol Diode:1N914
- added J?: PS/2_B, symbol Connector:Mini-DIN-6
- added R?: 33 K, symbol Device:R
- added U? (x7): 74HC14, symbol 74xx:74HC14
- added U? (x2): 74HC595, symbol 74xx:74HC595
- J?: value Mini-DIN-6 -> PS/2_A
Connections:
- net CB1: now also U?.10, U?.12 (RCLK), U?.12 (RCLK)
- net GND: now also C?.2, J?.3, U?.13 (~{OE}), U?.13 (~{OE}), U?.7 (GND), U?.8 (GND), U?.8 (GND)
- net PB0: now also U?.1 (QB)
- net PB1: now also U?.15 (QA)
- net PB2: now also U?.7 (QH)
- net PB3: now also U?.6 (QG)
- net PB4: now also U?.5 (QF)
- net PB5: now also U?.4 (QE)
- net PB6: now also U?.3 (QD)
- net PB7: now also U?.2 (QC)
- net VCC: now also J?.4, U?.1, U?.10 (~{SRCLR}), U?.10 (~{SRCLR}), U?.14 (VCC), U?.16 (VCC), U?.16 (VCC), U?.3, U?.5
- new net: J?.1, U?.14 (SER)
- new net: J?.5, U?.13, U?.9
- new net: U?.11 (SRCLK), U?.11 (SRCLK), U?.8
- new net: D?.2 (A), R?.1, U?.12
- new net: C?.1, D?.1 (K), R?.2, U?.11
- new net: U?.14 (SER), U?.9 (QH')
- no-connect marks 25 -> 30
Other:
- note added: "Dual PS/2 Interface (After Ben Eater https://beneater.net/6502)"
- note removed: "VIA Port Device Ben Eater PS/2 Interface https://beneater.net/6502"
- moved on the sheet: C?, D?, J102, J?, R?, U?, U?D, U?E, U?F
