File: kicad/Vega816/Accessories/EaterPS2Interface.kicad_sch (KiCad schematic)
At the start: 27 parts, among them J102 VIA Port

Commit message: push
Other:
- note added: "Dual PS/2 Interface (Ben Eater)"
- note removed: "Dual PS/2 Interface (After Ben Eater https://beneater.net/6502)"
- moved on the sheet: C?, D?, J102, J?, R?, U?, U?A, U?B, U?C, U?D, U?E, U?F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

Commit message: Big ol update
Parts:
- removed J102: VIA Port, symbol Connector_Generic:Conn_02x22_Odd_Even
- added C58 (x3), C59, C61 (x2): 100n, symbol Device:C_Small
Connections:
- net GND: now also C58.2, C58.2, C58.2, C59.2, C61.2, C61.2
- net VCC: now also C58.1, C58.1, C58.1, C59.1, C61.1, C61.1
- no-connect marks 30 -> 28
