File: kicad/Vega816/Accessories/ACIA.kicad_sch (KiCad schematic)
At the start: 15 parts, among them J103 $38 (8B), J104 USB Reset, J105 USB_B, J106 USB_I2C, U126 W65C51NxP, U127 74HC04, U128 MCP2221AxP, X1 1.8432MHz

Commit message: system controller
Changed lines of the file:
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@@
     (effects (font (size 1.27 1.27)) (justify left bottom))
   )
-  (text "ACIA (RS-232) port\n(After Adrien Kohlbecker)" (at 19.05 25.4 0)
+  (text "ACIA (RS-232) port\n(After Adrien Kohlbecker)" (at 19.05 35.56 0)
     (effects (font (size 5 5)) (justify left bottom))
   )

Commit message: Big
Parts:
- removed J103: $38 (8B), symbol Connector_Generic:Conn_02x18_Odd_Even
Connections:
- net A0: no longer names the net of U126.13 (RS0)
- net A1: no longer names the net of U126.14 (RS1)
- net CLK: no longer names the net of U126.27 (ϕ2)
- net D0: no longer names the net of U126.18 (D0)
- net D1: no longer names the net of U126.19 (D1)
- net D2: no longer names the net of U126.20 (D2)
- net D3: no longer names the net of U126.21 (D3)
- net D4: no longer names the net of U126.22 (D4)
- net D5: no longer names the net of U126.23 (D5)
- net D6: no longer names the net of U126.24 (D6)
- net D7: no longer names the net of U126.25 (D7)
- net R~{W}: no longer names the net of U126.28 (R/~{W})
- net VA: no longer names the net of U126.2 (CS1)
- net ~{CS}: no longer names the net of U126.3 (~{CS2})
- net ~{IRQ}: no longer names the net of U126.26 (~{IRQ})
- net ~{RST}: no longer names the net of U126.4 (~{RES})
Other:
- moved on the sheet: C1, C2, C3, U127A, U127B, U127C, X1
