File: kicad/Vega816/Accessories/SID.kicad_sch (KiCad schematic)
At the start: 18 parts

Commit message: dfsg
Parts:
- removed C? (x2): 1800 pF, symbol Device:C
- removed C?: 100nF, symbol Device:C
- removed C? (x2): 470 pF, symbol Device:C
- removed C?: 10uF, symbol Device:C
- removed C?: 1nF, symbol Device:C
- removed C?: 470pF, symbol Device:C
- removed J?: Audio Out, symbol Connector:AudioJack2
- removed J?: $00 (32B), symbol Connector_Generic:Conn_02x24_Odd_Even
- removed J?: +9V/+12V, symbol Connector:Jack-DC
- removed J?: Audio In, symbol Connector:AudioJack2_SwitchT
- removed Q?: 2SC1815, Package_TO_SOT_THT:TO-92_Inline, symbol Transistor_BJT:2SC1815
- removed R?: 10K, symbol Device:R
- removed R? (x2): 1K, symbol Device:R
- removed R?: 100K, symbol Device:R
- removed U?: 6581_SID, Package_DIP:DIP-28_W15.24mm_Socket, symbol Vega816:6581_SID
Connections:
- no-connect marks 5 -> 0
Other:
- note removed: "+9V 8580 +12V 6581"
- note removed: "8580/6581 (SID)"
- note removed: "From Commodore 64 CIA (VIA) 1"
