File: kicad/Vega816/Accessories/VIC-II.kicad_sch (KiCad schematic)
At the start: 8 parts, among them J0A? Conn_02x40_Odd_Even, J0B? CPU

Commit message: dfsg
Parts:
- removed J0A?: Conn_02x40_Odd_Even, Connector_PinHeader_2.54mm:PinHeader_2x40_P2.54mm_Vertical, symbol Connector_Generic:Conn_02x40_Odd_Even
- removed J0B?: CPU, Connector_PinHeader_2.54mm:PinHeader_2x18_P2.54mm_Vertical, symbol Connector_Generic:Conn_02x18_Odd_Even
- removed J?: $00 (64 B), symbol Connector_Generic:Conn_02x28_Odd_Even
- removed J?: VPA/VDA, symbol Connector:Conn_01x02_Male
- removed U? (x2): 74LS244, symbol 74xx:74LS244
- removed U?: 74HC373, symbol 74xx:74HC373
- removed U?: VIC-II, Package_DIP:DIP-40_W15.24mm_Socket, symbol Vega816:VIC-II
Connections:
- no-connect marks 11 -> 0
Other:
- note removed: "64B Device"
- note removed: "8580/6581 (VIC-II)"
- note removed: "A10-A07 is stable for the entire memory cycle. The lower six address pins, A05-A00, are also bi-directional. During a processor read or write of the video device, address pins A05-A00 are inputs which latch on the low edge of RAS/. The data on these address inputs selects the register for read or write as defined in the register map."
- note removed: "Address pins A06-A00 are multiplexed to allow direct connection to dynamic RAMs. During the row address time, A06-A00 are driven on pins A06-A00, while A13-A08 are driven on pins A05-A00 and pin A06 is "1" during the column time."
