File: kicad/Vega816/Accessories/DualSPI.kicad_sch (KiCad schematic)
At the start: 5 parts, among them J102 VIA Port

Commit message: Big ol update
Parts:
- removed J102: VIA Port, symbol Connector_Generic:Conn_02x22_Odd_Even
- added C114, C115: 100n, symbol Device:C_Small
- added J21: Conn_02x02_Odd_Even, symbol Connector_Generic:Conn_02x02_Odd_Even
Connections:
- net GND: now also C114.2, C115.2, J21.2 (Pin_2), J21.4 (Pin_4)
- net VCC: now also C114.1, C115.1
- net ~{SPI_CS0} renamed ~{SPI_CS0}_A
- net ~{SPI_CS0}_A: no longer J?.19 (Pin_19), U?.15 (O0)
- net ~{SPI_CS1} renamed ~{SPI_CS1}_A
- net ~{SPI_CS1}_A: no longer J?.17 (Pin_17), U?.14 (O1)
- net ~{SPI_CS2} renamed ~{SPI_CS2}_A
- net ~{SPI_CS2}_A: no longer J?.15 (Pin_15), U?.13 (O2)
- net ~{SPI_CS3} renamed ~{SPI_CS3}_A
- net ~{SPI_CS3}_A: no longer J?.13 (Pin_13), U?.12 (O3)
- net ~{SPI_CS4} renamed ~{SPI_CS4}_A
- net ~{SPI_CS4}_A: no longer J?.11 (Pin_11), U?.11 (O4)
- net ~{SPI_CS5} renamed ~{SPI_CS5}_A
- net ~{SPI_CS5}_A: no longer J?.9 (Pin_9), U?.10 (O5)
- net ~{SPI_CS6} renamed ~{SPI_CS6}_A
- net ~{SPI_CS6}_A: no longer J?.7 (Pin_7), U?.9 (O6)
- net ~{SPI_CS7} renamed ~{SPI_CS7}_A
- net ~{SPI_CS7}_A: no longer J?.5 (Pin_5), U?.7 (O7)
- new net PB6: J21.3 (Pin_3)
- new net PB7: J21.1 (Pin_1)
- new net ~{SPI_CS0}_B: J?.19 (Pin_19), U?.15 (O0)
- new net ~{SPI_CS1}_B: J?.17 (Pin_17), U?.14 (O1)
- new net ~{SPI_CS2}_B: J?.15 (Pin_15), U?.13 (O2)
- new net ~{SPI_CS3}_B: J?.13 (Pin_13), U?.12 (O3)
- new net ~{SPI_CS4}_B: J?.11 (Pin_11), U?.11 (O4)
- new net ~{SPI_CS5}_B: J?.9 (Pin_9), U?.10 (O5)
- new net ~{SPI_CS6}_B: J?.7 (Pin_7), U?.9 (O6)
- new net ~{SPI_CS7}_B: J?.5 (Pin_5), U?.7 (O7)
- no-connect marks 4 -> 6
Other:
- note added: "Dual 8 Channel SPI VIA Port Device"
- note added: "PA0 PA1 PA2 PA3 PA4 PA5"
- note removed: "On ~{RES}, PA is set to inputs with bus holding devices. Pulldown resistors pull all System Controls low. Write $00 to PA before changing PA DDR to output."
- note removed: "PA0 Output CPU A ~{A_CLK_SLOW} PA1 Output CPU B ~{B_CLK_SLOW} PA2 Output CPU B B_RDY_IN PA3 Output CPU B ~{B_DMA_PRIORITY} PA4 Output DMA 0 ~{EEPROM_RD_0} PA5 Output DMA 0 EEPROM_WR_0 PA6 Output DMA 1 ~{EEPROM_RD_1} PA7 Output DMA 1 EEPROM_WR_1"
- note removed: "VIA Port Device Dual 8 Channel SPI"
