File: kicad/Vega816/Vega816.kicad_sch (KiCad schematic)
At the start: 0 parts

Commit message: dfg
Other:
- added sheet C64 SID+CIAS (MemoryExpansionBus/c64sidandcias.kicad_sch)
Changed lines of the file:
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@@
+    )
+  )
+  (sheet (at 128.27 41.91) (size 26.67 13.97)
+    (stroke (width 0.1524) (type solid) (color 0 0 0 0))
+    (fill (color 0 0 0 0.0000))
+    (property "Sheet name" "C64 SID+CIAS" (id 0) (at 125.73 40.3334 0)
+      (effects (font (size 3 3)) (justify left bottom))
+    )
+    (property "Sheet file" "MemoryExpansionBus/c64sidandcias.kicad_sch" (id 1) (at 128.27 56.4646 0)
+      (effects (font (size 1.27 1.27)) (justify left top) hide)
     )
   )
@@
     (path "/e77c13b8-e97e-4fc3-8aa5-349c9b99f1d4" (page "19"))
     (path "/188a6def-66f4-4ee7-b358-dda63164c91c" (page "20"))
+    (path "/21c33125-dba5-497b-830f-02ea1d5dc0da" (page "21"))
   )
   (symbol_instances
@@
       (reference "#PWR0125") (unit 1) (value "GND") (footprint "")
     )
-    (path "/ed4e59dc-e26e-4739-aa1d-80a767eacd8d/25be4e02-5fde-43f7-a2de-42b5255c2dd1"
+    (path "/ed4e59dc-e26e-4739-aa1d-80a767eacd8d/35941f83-353f-4d78-bbcf-97569e269599"
       (reference "#PWR0125") (unit 1) (value "GND") (footprint "")
-    )
-    (path "/ed4e59dc-e26e-4739-aa1d-80a767eacd8d/00e7f294-0dbe-4ad7-9870-8318f046842f"
-      (reference "#PWR0126") (unit 1) (value "VCC") (footprint "")
     )
     (path "/188a6def-66f4-4ee7-b358-dda63164c91c/00e7f294-0dbe-4ad7-9870-8318f046842f"
       (reference "#PWR0126") (unit 1) (value "VCC") (footprint "")
     )
+    (path "/ed4e59dc-e26e-4739-aa1d-80a767eacd8d/cbd9110f-78bb-4167-a74b-88953e747dda"
+      (reference "#PWR0126") (unit 1) (value "VCC") (footprint "")
+    )
     (path "/188a6def-66f4-4ee7-b358-dda63164c91c/1a10cb1b-eaf5-48a4-9fad-40186293365b"
       (reference "#PWR0127") (unit 1) (value "VCC") (footprint "")
@@
       (reference "#PWR0191") (unit 1) (value "VCC") (footprint "")
     )
+    (path "/21c33125-dba5-497b-830f-02ea1d5dc0da/70e7bdf3-ee48-4f67-922d-1006e2c7900b"
+      (reference "#PWR0191") (unit 1) (value "VCC") (footprint "")
+    )
     (path "/c8c771df-7dcc-45f6-b525-febf6b559971/870815e8-15d1-4d50-90a2-939ff0e2488b"
       (reference "#PWR0192") (unit 1) (value "GND") (footprint "")
     )
+    (path "/21c33125-dba5-497b-830f-02ea1d5dc0da/870815e8-15d1-4d50-90a2-939ff0e2488b"
+      (reference "#PWR0192") (unit 1) (value "GND") (footprint "")
+    )
     (path "/c8c771df-7dcc-45f6-b525-febf6b559971/9189e38e-dfb0-48e5-8379-be973b488542"
       (reference "#PWR0193") (unit 1) (value "GND") (footprint "")
@@
       (reference "#PWR0194") (unit 1) (value "GND") (footprint "")
     )
+    (path "/21c33125-dba5-497b-830f-02ea1d5dc0da/94534c2b-4e06-45d8-bb2c-7e1105a64af3"
+      (reference "#PWR0195") (unit 1) (value "GND") (footprint "")
+    )
     (path "/c8c771df-7dcc-45f6-b525-febf6b559971/94534c2b-4e06-45d8-bb2c-7e1105a64af3"
       (reference "#PWR0195") (unit 1) (value "GND") (footprint "")
@@
       (reference "#PWR0196") (unit 1) (value "GND") (footprint "")
     )
+    (path "/21c33125-dba5-497b-830f-02ea1d5dc0da/86d3a3c3-d284-41c3-947f-26cb377c3634"
+      (reference "#PWR0196") (unit 1) (value "GND") (footprint "")
+    )
+    (path "/21c33125-dba5-497b-830f-02ea1d5dc0da/06a08184-5a9d-45ee-984d-e25d219c4194"
+      (reference "#PWR0197") (unit 1) (value "GND") (footprint "")
+    )
     (path "/c8c771df-7dcc-45f6-b525-febf6b559971/06a08184-5a9d-45ee-984d-e25d219c4194"
       (reference "#PWR0197") (unit 1) (value "GND") (footprint "")
@@
       (reference "J62") (unit 1) (value "IRQ_OUT") (footprint "")
     )
+    (path "/21c33125-dba5-497b-830f-02ea1d5dc0da/457e9377-c361-49a2-bf7d-94322bb2e9bc"
+      (reference "J62") (unit 1) (value "IRQ_OUT") (footprint "")
+    )
     (path "/c8c771df-7dcc-45f6-b525-febf6b559971/615d8813-c14a-4885-9a1f-09ba197654a1"
       (reference "J63") (unit 1) (value "Device Select") (footprint "")
     )
+    (path "/21c33125-dba5-497b-830f-02ea1d5dc0da/615d8813-c14a-4885-9a1f-09ba197654a1"
+      (reference "J63") (unit 1) (value "Device Select") (footprint "")
+    )
     (path "/c8c771df-7dcc-45f6-b525-febf6b559971/e38cb711-5917-49dd-8a11-1ca30a3b1a0c"
       (reference "J64") (unit 1) (value "A/D Bus") (footprint "")
     )
+    (path "/21c33125-dba5-497b-830f-02ea1d5dc0da/e38cb711-5917-49dd-8a11-1ca30a3b1a0c"
+      (reference "J64") (unit 1) (value "A/D Bus") (footprint "")
+    )
     (path "/c8c771df-7dcc-45f6-b525-febf6b559971/6f4d6c76-884a-4b56-af0c-e59b11a26e74"
       (reference "J65") (unit 1) (value "IRQ_OUT") (footprint "")
@@
       (reference "J72") (unit 1) (value "$80 (32B)") (footprint "")
     )
+    (path "/21c33125-dba5-497b-830f-02ea1d5dc0da/780e4b97-170a-491a-8073-c1b667a021ed"
+      (reference "J72") (unit 1) (value "$80 (32B)") (footprint "")
+    )
     (path "/c8c771df-7dcc-45f6-b525-febf6b559971/17bd5c34-b8e0-49df-a593-9ea1a2a5dbcd"
       (reference "J73") (unit 1) (value "$38 (8B IRQ 7)") (footprint "")
@@
       (reference "J75") (unit 1) (value "$20(16B IRQ 4-5)") (footprint "")
     )
+    (path "/21c33125-dba5-497b-830f-02ea1d5dc0da/c49ce25b-f66d-41da-b45b-0fc865ff3a61"
+      (reference "J76") (unit 1) (value "$00 (16B)") (footprint "")
+    )
     (path "/c8c771df-7dcc-45f6-b525-febf6b559971/c49ce25b-f66d-41da-b45b-0fc865ff3a61"
       (reference "J76") (unit 1) (value "$00 (16B)") (footprint "")
     )
+    (path "/21c33125-dba5-497b-830f-02ea1d5dc0da/abfc5302-d19d-4542-9cbb-c68e8867ab61"
+      (reference "J77") (unit 1) (value "$40 (16B)") (footprint "")
+    )
     (path "/c8c771df-7dcc-45f6-b525-febf6b559971/abfc5302-d19d-4542-9cbb-c68e8867ab61"
       (reference "J77") (unit 1) (value "$40 (16B)") (footprint "")
@@
       (reference "U?") (unit 4) (value "74HC00") (footprint "")
     )
+    (path "/21c33125-dba5-497b-830f-02ea1d5dc0da/7fd04819-f975-462a-8923-edfec8928b26"
+      (reference "U?") (unit 4) (value "74HC00") (footprint "")
+    )

Commit message: expansion port hi ram
Other:
- sheet C64 SID+CIAS renamed C64 SID+CIAS Breakout
- added sheet C64 CIA #2 (Accessories/C64VIA2.kicad_sch)

Commit message: new plots
Other:
- sheet System Controller + SPI renamed System Controller
- removed sheet PIC (2 IRQ)
- added sheet 4 Channel DMA Ctrl (DMA/DMAController4.kicad_sch)
- added sheet 6510 CPU Registers (MemoryExpansionBus/6510.kicad_sch)
- added sheet C64 IO Decoder (MemoryExpansionBus/C64_IO_Decoder.kicad_sch)
- added sheet Dual SPI (Accessories/DualSPI.kicad_sch)
- added sheet PIC (MemoryExpansionBus/pic_single.kicad_sch)

Commit message: wug
Other:
- sheet 4 Channel DMA Ctrl renamed 4 CPU x 4 DMA Controller
- sheet CPU-DMA Buffer renamed CPU Buffer
- removed sheet DMA Controller
- removed sheet Quad PIC (8 IRQ)

Commit message: fdt
Other:
- sheet 4 CPU x 4 DMA Controller renamed 4x4 DMA Controller
- sheet 6510 CPU Registers renamed 6510 $[01] Regs
- sheet C64 IO Decoder renamed Address Decode + PLA
- sheet C64 SID+CIAS Breakout renamed CIAs + 2xSID
- sheet DMA + VPB Shim renamed CPU Shim
- removed sheet C64 CIA #1
- removed sheet C64 CIA #2
- removed sheet SID (8580 or 6581)
- added sheet SID(x2) (Accessories/SID.kicad_sch)
- note added: "Commodore 64 Hardware"

Commit message: xcvx
Parts:
- added U? (x4): BB816Breakout, symbol Vega816:BB816Breakout
Other:
- sheet CPU Buffer renamed CPU Buffer0
- removed sheet Quad 64B IO Bus
- added sheet 16MB Memory Bus1 (MemoryExpansionBus/16MB_Expansion_Bus.kicad_sch)
- added sheet 16MB Memory Bus2 (MemoryExpansionBus/16MB_Expansion_Bus.kicad_sch)
- added sheet 16MB Memory Bus3 (MemoryExpansionBus/16MB_Expansion_Bus.kicad_sch)
- added sheet CPU Buffer1 (DMA/CPU Buffer/CPU Buffer.kicad_sch)
- added sheet CPU Buffer10 (DMA/CPU Buffer/CPU Buffer.kicad_sch)
- added sheet CPU Buffer11 (DMA/CPU Buffer/CPU Buffer.kicad_sch)
- added sheet CPU Buffer12 (DMA/CPU Buffer/CPU Buffer.kicad_sch)
- added sheet CPU Buffer13 (DMA/CPU Buffer/CPU Buffer.kicad_sch)
- added sheet CPU Buffer14 (DMA/CPU Buffer/CPU Buffer.kicad_sch)
- added sheet CPU Buffer15 (DMA/CPU Buffer/CPU Buffer.kicad_sch)
- added sheet CPU Buffer2 (DMA/CPU Buffer/CPU Buffer.kicad_sch)
- added sheet CPU Buffer3 (DMA/CPU Buffer/CPU Buffer.kicad_sch)
- added sheet CPU Buffer4 (DMA/CPU Buffer/CPU Buffer.kicad_sch)
- added sheet CPU Buffer5 (DMA/CPU Buffer/CPU Buffer.kicad_sch)
- added sheet CPU Buffer6 (DMA/CPU Buffer/CPU Buffer.kicad_sch)
- added sheet CPU Buffer7 (DMA/CPU Buffer/CPU Buffer.kicad_sch)
- added sheet CPU Buffer8 (DMA/CPU Buffer/CPU Buffer.kicad_sch)
- added sheet CPU Buffer9 (DMA/CPU Buffer/CPU Buffer.kicad_sch)
- added sheet CPU Shim1 (DMA/DMABreakout.kicad_sch)
- added sheet CPU Shim2 (DMA/DMABreakout.kicad_sch)
- added sheet CPU Shim3 (DMA/DMABreakout.kicad_sch)
- added sheet xN Single Page IO Bus (MemoryExpansionBus/irq_multiplex.kicad_sch)
- note added: "Four CPUs x 4 DMA Channels"
- note added: "Four DMA Channels"

Commit message: git ignor
Other:
- sheet 4x4 DMA Controller renamed DMA Controller
- sheet Accessories renamed Device Ports
- sheet CPU Shim renamed CPU Shim A
- sheet CPU Shim1 renamed CPU Shim B
- sheet CPU Shim2 renamed CPU Shim C
- sheet CPU Shim3 renamed CPU Shim D
- sheet xN Single Page IO Bus renamed Bank0 Single Page IO Buses ($00-$FE)
- removed sheet 16MB Memory Bus1
- removed sheet 16MB Memory Bus2
- removed sheet 16MB Memory Bus3
- removed sheet 4 MB RAM + EEPROM
- added sheet 4 MB RAM (MemoryExpansionBus/4MB_Memory_Module.kicad_sch)
- added sheet Device Port (Accessories/Accessories.kicad_sch)
- note added: "32KB EEPROM"
- note added: "DMA 0"
- note added: "DMA 1"
- note added: "DMA 2"
- note added: "DMA 3"
- note added: "DMA Channels"
- note removed: "Four DMA Channels"
- moved on the sheet: U?
