File: kicad/Vega816/Vega816.kicad_sch (KiCad schematic)
At the start: 4 parts

Commit message: Big push, Sysctl, DMA Reg
Parts:
- removed U? (x4): BB816Breakout, symbol Vega816:BB816Breakout
Other:
- removed sheet CPU Buffer0
- removed sheet CPU Buffer1
- removed sheet CPU Buffer10
- removed sheet CPU Buffer11
- removed sheet CPU Buffer12
- removed sheet CPU Buffer13
- removed sheet CPU Buffer14
- removed sheet CPU Buffer15
- removed sheet CPU Buffer2
- removed sheet CPU Buffer3
- removed sheet CPU Buffer4
- removed sheet CPU Buffer5
- removed sheet CPU Buffer6
- removed sheet CPU Buffer7
- removed sheet CPU Buffer8
- removed sheet CPU Buffer9
- removed sheet CPU Shim A
- removed sheet CPU Shim B
- removed sheet CPU Shim C
- removed sheet CPU Shim D
- removed sheet DMA Controller
- removed sheet Device Port
- note removed: "32KB EEPROM"
- note removed: "DMA 0"
- note removed: "DMA 1"
- note removed: "DMA 2"
- note removed: "DMA 3"
- note removed: "DMA Channels"
- note removed: "Four CPUs x 4 DMA Channels"
- note removed: "Vega 816 SMP Computer System"

Commit message: Big
Other:
- sheet 16MB Memory Bus renamed Memory Bus
- sheet 4 MB RAM renamed 4MB RAM
- sheet Bank0 Single Page IO Buses ($00-$FE) renamed IO Bus
- sheet System Controller renamed Sysctrl Registers
- sheet VIA (W65C22) renamed System IO
- removed sheet 64B IO Port
- removed sheet CIAs + 2xSID
- removed sheet Device Ports
- removed sheet Priority IRQ Dispatch
- removed sheet RS-232 (W65C51)
- added sheet ACIA Adapter (Accessories/ACIAAdapter.kicad_sch)
- added sheet CPU Buffer (CPU Buffer/CPU Buffer.kicad_sch)
- added sheet CPU Shim (CPUShim/CPUShim.kicad_sch)
- added sheet DMA Controller (DMAController/DMAController.kicad_sch)
- sheet IO Bus: file MemoryExpansionBus/irq_multiplex.kicad_sch -> IOBus/IOBus.kicad_sch
- note removed: "16 Byte Device"
- note removed: "32 Byte Device"
- note removed: "64 Byte Device"
- note removed: "8 Byte Device"
- note removed: "Controls One, e.g.:"

Commit message: asf
Other:
- sheet Address Decode + PLA renamed Decode + VIA
- sheet Front Panel renamed Front Console
- sheet SID(x2) renamed SID
- sheet System IO renamed System Devices
- removed sheet 6510 $[01] Regs
- sheet CPU Shim: file CPUShim/CPUShim.kicad_sch -> CPU Shim/CPU Shim.kicad_sch
- sheet DMA Controller: file DMAController/DMAController.kicad_sch -> DMA Controller/DMA Controller.kicad_sch
- sheet Decode + VIA: file MemoryExpansionBus/C64_IO_Decoder.kicad_sch -> C64 Hardware/C64 Hardware.kicad_sch
- sheet Front Console: file Accessories/VIADevices.kicad_sch -> Front Console/Front Console.kicad_sch
- sheet SID: file Accessories/SID.kicad_sch -> C64 Hardware/SID.kicad_sch
- sheet Sysctrl Registers: file Accessories/SystemController.kicad_sch -> Sysctrl Registers/Sysctrl Registers.kicad_sch
- sheet System Devices: file Accessories/VIAPort.kicad_sch -> System Devices/System Devices.kicad_sch
- sheet VIC-II: file Accessories/VIC-II.kicad_sch -> C64 Hardware/VIC-II.kicad_sch

Commit message: Big ol update
Other:
- sheet SID renamed Dual SID
- removed sheet ACIA Adapter
- added sheet ACIA (System Devices/ACIA.kicad_sch)
- added sheet VIA Port Conn (System Devices/VIAPort.kicad_sch)
- added sheet VIA Port NoConn (System Devices/VIAPortNoConn.kicad_sch)
- added sheet XR88C192 UART (XR88C192_UART/XR88C192_UART.kicad_sch)
Changed lines of the file:
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@@
     (effects (font (size 3 3)) (justify right bottom))
   )
+  (sheet (at 114.3 119.38) (size 24.13 13.97) (fields_autoplaced)
+    (stroke (width 0.1524) (type solid))
+    (fill (color 0 0 0 0.0000))
+    (property "Sheetname" "XR88C192 UART" (at 114.3 117.8034 0)
+      (effects (font (size 3 3)) (justify left bottom))
+    )
+    (property "Sheetfile" "XR88C192_UART/XR88C192_UART.kicad_sch" (at 114.3 133.9346 0)
+      (effects (font (size 1.27 1.27)) (justify left top) hide)
+    )
+    (instances
+      (project "Vega816"
+        (path "/162a94ce-b5da-40d1-ba41-c7bb68a4398a" (page "19"))
+      )
+    )
+  )
+  (sheet (at 83.82 129.54) (size 24.13 5.08)
+    (stroke (width 0.1524) (type solid))
+    (fill (color 0 0 0 0.0000))
+    (property "Sheetname" "VIA Port NoConn" (at 85.09 127.9634 0)
+      (effects (font (size 2 2)) (justify left bottom))
+    )
+    (property "Sheetfile" "System Devices/VIAPortNoConn.kicad_sch" (at 83.82 144.0946 0)
+      (effects (font (size 1.27 1.27)) (justify left top) hide)
+    )
+    (instances
+      (project "Vega816"
+        (path "/162a94ce-b5da-40d1-ba41-c7bb68a4398a" (page "9"))
+      )
+    )
+  )
   (sheet (at 22.86 95.25) (size 24.13 13.97)
     (stroke (width 0.1524) (type solid))
@@
     (stroke (width 0.1524) (type solid))
     (fill (color 0 0 0 0.0000))
-    (property "Sheetname" "System Devices" (at 50.8 117.8034 0)
-      (effects (font (size 3 3)) (justify left bottom))
+    (property "Sheetname" "System Devices" (at 54.61 117.8034 0)
+      (effects (font (size 2 2)) (justify left bottom))
     )
     (property "Sheetfile" "System Devices/System Devices.kicad_sch" (at 53.34 133.9346 0)
@@
     )
   )
+  (sheet (at 83.82 119.38) (size 24.13 5.08)
+    (stroke (width 0.1524) (type solid))
+    (fill (color 0 0 0 0.0000))
+    (property "Sheetname" "VIA Port Conn" (at 85.09 117.8034 0)
+      (effects (font (size 2 2)) (justify left bottom))
+    )
+    (property "Sheetfile" "System Devices/VIAPort.kicad_sch" (at 83.82 133.9346 0)
+      (effects (font (size 1.27 1.27)) (justify left top) hide)
+    )
+    (instances
+      (project "Vega816"
+        (path "/162a94ce-b5da-40d1-ba41-c7bb68a4398a" (page "8"))
+      )
+    )
+  )
+  (sheet (at 233.68 119.38) (size 24.13 13.97)
+    (stroke (width 0.1524) (type solid))
+    (fill (color 0 0 0 0.0000))
+    (property "Sheetname" "ACIA" (at 241.3 117.8034 0)
+      (effects (font (size 3 3)) (justify left bottom))
+    )
+    (property "Sheetfile" "System Devices/ACIA.kicad_sch" (at 233.68 133.9346 0)
+      (effects (font (size 1.27 1.27)) (justify left top) hide)
+    )
+    (instances
+      (project "System Devices"
+        (path "/bc87933a-d9f8-4898-8cff-86eee8396f35" (page "2"))
+      )
+      (project "Vega816"
+        (path "/162a94ce-b5da-40d1-ba41-c7bb68a4398a" (page "3"))
+      )
+    )
+  )
   (sheet (at 24.13 172.72) (size 26.67 13.97) (fields_autoplaced)
     (stroke (width 0.1524) (type solid))
@@
     (stroke (width 0.1524) (type solid))
     (fill (color 0 0 0 0.0000))
-    (property "Sheetname" "SID" (at 207.01 150.0534 0)
+    (property "Sheetname" "Dual SID" (at 207.01 150.0534 0)
       (effects (font (size 2 2)) (justify left bottom))
     )
@@
       )
     )
-  )
-  (sheet (at 100.33 119.38) (size 27.94 13.97) (fields_autoplaced)
-    (stroke (width 0.1524) (type solid))
-    (fill (color 0 0 0 0.0000))
-    (property "Sheetname" "ACIA Adapter" (at 100.33 117.8034 0)
-      (effects (font (size 3 3)) (justify left bottom))
-    )
-    (property "Sheetfile" "Accessories/ACIAAdapter.kicad_sch" (at 100.33 133.9346 0)
-      (effects (font (size 1.27 1.27)) (justify left top) hide)
-    )
-    (instances
-      (project "Vega816"
-        (path "/162a94ce-b5da-40d1-ba41-c7bb68a4398a" (page "2"))
-      )
-    )

Commit message: wrtolei
Other:
- removed sheet 4MB RAM
- removed sheet ACIA
- removed sheet Decode + VIA
- removed sheet Dual PS2
- removed sheet Dual SID
- removed sheet Dual SPI
- removed sheet Front Console
- removed sheet IO Bus
- removed sheet Memory Bus
- removed sheet PIC
- removed sheet System Devices
- removed sheet VIA Port Conn
- removed sheet VIA Port NoConn
- removed sheet VIC-II
- removed sheet XR88C192 UART
- note added: "Vega816 - SMP+DMA+VPB for BB816 Breakout"
- note removed: "Commodore 64 Hardware"
- note removed: "VIA Port Devices"
