File: kicad/Vega816/DMA/DMABreakout.kicad_sch (KiCad schematic)
At the start: 26 parts, among them J17 VPA/VDA, J18 Conn_02x40_Odd_Even, J19 CPU, J20 8MB, J21 4MB, J22 2MB, J23 1MB, J24 512KB, J25 256KB, J26 128KB, J27 64KB, J28 ~{DMA 1}, J29 ~{DMA 0}, J30 DMA Ctrl, J31 VPA/VDA, J32 Conn_02x40_Odd_Even, J33 DMA, U26 74HC00, U30 74HC08, U31 74HC283

Commit message: irq shim
Parts:
- removed J?: VP Rewrite Ctrl, symbol Connector_Generic:Conn_02x04_Odd_Even
- added J?: VP Shim, symbol Connector_Generic:Conn_02x08_Odd_Even
Connections:
- net VP_REQ is gone; now on net VP: U30.8
- net GND: now also J?.10 (Pin_10), J?.12 (Pin_12), J?.14 (Pin_14), J?.16 (Pin_16), J?.2 (Pin_2), J?.3 (Pin_3), J?.4 (Pin_4), J?.6 (Pin_6), J?.8 (Pin_8)
- net VCC: now also J?.1 (Pin_1)
- net VP: now also J?.15 (Pin_15)
- net Y1: now also J?.13 (Pin_13)
- net Y2: now also J?.11 (Pin_11)
- net Y3: now also J?.9 (Pin_9)
- net ~{IRQ}: now also J?.7 (Pin_7)
- net ~{NMI}: now also J?.5 (Pin_5)
- net ~{DMA 0} renamed ~{BUFFER 0 CS}
- net ~{DMA 1} renamed ~{BUFFER_1_CS}
Other:
- moved on the sheet: J28, J29, RN1

Commit message: xvsvd
Connections:
- net VP: no longer J?.15 (Pin_15), U30.8
- new net VP_REQ: J?.15 (Pin_15), U30.8
Changed lines of the file:
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@@
     (effects (font (size 1.27 1.27)) (justify left bottom))
   )
-  (label "VP" (at 205.74 347.98 0)
+  (label "VP_REQ" (at 205.74 347.98 0)
     (effects (font (size 1.27 1.27)) (justify left bottom))
   )

Commit message: C
Parts:
- removed J20: 8MB, symbol Connector_Generic:Conn_01x03
- removed J21: 4MB, symbol Connector_Generic:Conn_01x03
- removed J22: 2MB, symbol Connector_Generic:Conn_01x03
- removed J23: 1MB, symbol Connector_Generic:Conn_01x03
- removed J24: 512KB, symbol Connector_Generic:Conn_01x03
- removed J25: 256KB, symbol Connector_Generic:Conn_01x03
- removed J26: 128KB, symbol Connector_Generic:Conn_01x03
- removed J27: 64KB, symbol Connector_Generic:Conn_01x03
- removed J30: DMA Ctrl, symbol Connector_Generic:Conn_02x08_Odd_Even
- removed RN1: 10K, Resistor_THT:R_Array_SIP9, symbol Device:R_Network08
- added J?: ~{BUFFER CS 0}, symbol Connector_Generic:Conn_02x01
- added J?: ~{BUFFER CS 1}, symbol Connector_Generic:Conn_02x01
- added J?: DMA Controller, symbol Connector_Generic:Conn_02x11_Odd_Even
- added J?: DMA_REQ_LO, symbol Connector_Generic:Conn_02x08_Odd_Even
- added J?: DMA Bypass, symbol Connector_Generic:Conn_02x08_Odd_Even
- added J?: DMA_REQ_HI, symbol Connector_Generic:Conn_02x08_Odd_Even
- added R? (x2): 10K, symbol Device:R
- added RN?: 10K, Resistor_THT:R_Array_SIP9, symbol Device:R_Network08
- added U? (x7): 74AHC32, Package_DIP:DIP-14_W7.62mm, symbol 74xx:74LS32
- added U? (x2): 74HC00, symbol 74xx:74HC00
- J28: value ~{DMA 1} -> ~{BUFFER CS 2}
- J29: value ~{DMA 0} -> ~{BUFFER CS 3}
Connections:
- net A16: now also J?.15 (Pin_15), J?.15 (Pin_15), J?.15 (Pin_15), J?.16 (Pin_16), RN?.9 (R8), U?.1
- net A17: now also J?.13 (Pin_13), J?.13 (Pin_13), J?.13 (Pin_13), J?.14 (Pin_14), RN?.8 (R7), U?.2
- net A18: now also J?.11 (Pin_11), J?.11 (Pin_11), J?.11 (Pin_11), J?.12 (Pin_12), RN?.7 (R6), U?.13
- net A19: now also J?.10 (Pin_10), J?.9 (Pin_9), J?.9 (Pin_9), J?.9 (Pin_9), RN?.6 (R5), U?.12
- net A20: now also J?.7 (Pin_7), J?.7 (Pin_7), J?.7 (Pin_7), J?.8 (Pin_8), RN?.5 (R4), U?.4
- net A21: now also J?.5 (Pin_5), J?.5 (Pin_5), J?.5 (Pin_5), J?.6 (Pin_6), RN?.4 (R3), U?.5
- net A22: now also J?.3 (Pin_3), J?.3 (Pin_3), J?.3 (Pin_3), J?.4 (Pin_4), RN?.3 (R2), U?.10
- net A23: now also J?.1 (Pin_1), J?.1 (Pin_1), J?.1 (Pin_1), J?.2 (Pin_2), RN?.2 (R1), U?.9
- net CLK: now also J?.13 (Pin_13)
- net GND: now also J?.10 (Pin_10), J?.12 (Pin_12), J?.14 (Pin_14), J?.16 (Pin_16), J?.18 (Pin_18), J?.2 (Pin_2), J?.2 (Pin_2), J?.2 (Pin_2), J?.20 (Pin_20), J?.22 (Pin_22), J?.4 (Pin_4), J?.6 (Pin_6), J?.8 (Pin_8), R?.1, R?.1, RN?.1 (common)
- net RDY_IN: now also J?.19 (Pin_19)
- net VA: now also J?.21 (Pin_21)
- net ~{ABORT}: now also J?.17 (Pin_17)
- net ~{BANK0}: now also U?.8
- net ~{CLK}: now also J?.15 (Pin_15)
- net ~{BUFFER 0 CS} renamed ~{DMA 3}
- net ~{DMA 3}: now also J?.7 (Pin_7)
- net ~{BUFFER_1_CS} renamed ~{DMA 2}
- net ~{DMA 2}: now also J?.5 (Pin_5)
- new net: U?.11, U?.4
- new net: U?.1, U?.8
- new net: J?.10 (Pin_10), J?.12 (Pin_12), J?.14 (Pin_14), J?.16 (Pin_16), J?.2 (Pin_2), J?.4 (Pin_4), J?.6 (Pin_6), J?.8 (Pin_8), R?.2, U?.4, U?.5
- new net: U?.2, U?.6
- new net: U?.10, U?.3
- new net: U?.6, U?.9
- new net: U?.3, U?.5
- new net: J?.10 (Pin_10), J?.12 (Pin_12), J?.14 (Pin_14), J?.16 (Pin_16), J?.2 (Pin_2), J?.4 (Pin_4), J?.6 (Pin_6), J?.8 (Pin_8), R?.2, U?.10, U?.9
- new net DMA_REQ_HI: J?.11 (Pin_11), U?.8
- new net DMA_REQ_LO: J?.9 (Pin_9), U?.6
- new net ~{DMA 0}: J?.1 (Pin_1), J?.1 (Pin_1)
- new net ~{DMA 1}: J?.1 (Pin_1), J?.3 (Pin_3)
- no-connect marks 1 -> 2
Other:
- note added: "~{BANK0} Rewrite"
- note removed: "DMA_REQ"
- note removed: "Install one jumper in top (DMA_REQ) position to set DMA Bank alternation granularity. All other jumpers in bottom (PASS_THRU) position."
- note removed: "PASS_THRU"
- moved on the sheet: J17, J18, J19, J28, J29, J31, J32, J33, J?, R1, R2, R3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

Commit message: wug
Other:
- note added: "CPU Shim (1 per CPU): 1. DMA Control Shim 2. Vector Pull Rewrite Shim"
- note added: "DMA Control Shim"
- note added: "Vector Pull Rewrite Shim"
- note added: "~{BANK0} Recalc"
- note removed: "Vector Pull + Dual Channel DMA Control Shim (1 per CPU)"
- note removed: "~{BANK0} Rewrite"
Changed lines of the file:
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@@
     (stroke (width 0) (type default) (color 0 0 0 0))
   )
+  (polyline (pts (xy 129.54 224.79) (xy 129.54 158.75))
+    (stroke (width 0) (type default) (color 0 0 0 0))
+  )
   (wire (pts (xy 139.7 163.83) (xy 139.7 165.1))
     (stroke (width 0) (type default) (color 0 0 0 0))
@@
     (stroke (width 0) (type default) (color 0 0 0 0))
   )
+  (polyline (pts (xy 203.2 293.37) (xy 138.43 293.37))
+    (stroke (width 0) (type default) (color 0 0 0 0))
+  )
   (wire (pts (xy 144.78 243.84) (xy 144.78 246.38))
     (stroke (width 0) (type default) (color 0 0 0 0))
@@
     (stroke (width 0) (type default) (color 0 0 0 0))
   )
+  (polyline (pts (xy 68.58 375.92) (xy 46.99 375.92))
+    (stroke (width 0) (type default) (color 0 0 0 0))
+  )
   (wire (pts (xy 110.49 129.54) (xy 110.49 218.44))
     (stroke (width 0) (type default) (color 0 0 0 0))
@@
     (stroke (width 0) (type default) (color 0 0 0 0))
   )
+  (polyline (pts (xy 69.85 224.79) (xy 129.54 224.79))
+    (stroke (width 0) (type default) (color 0 0 0 0))
+  )
   (wire (pts (xy 160.02 250.19) (xy 139.7 250.19))
     (stroke (width 0) (type default) (color 0 0 0 0))
@@
     (stroke (width 0) (type default) (color 0 0 0 0))
   )
+  (polyline (pts (xy 264.16 229.87) (xy 264.16 180.34))
+    (stroke (width 0) (type default) (color 0 0 0 0))
+  )
   (wire (pts (xy 139.7 179.07) (xy 139.7 180.34))
     (stroke (width 0) (type default) (color 0 0 0 0))
@@
     (stroke (width 0) (type default) (color 0 0 0 0))
   )
+  (polyline (pts (xy 138.43 158.75) (xy 138.43 186.69))
+    (stroke (width 0) (type default) (color 0 0 0 0))
+  )
   (wire (pts (xy 35.56 264.16) (xy 139.7 264.16))
     (stroke (width 0) (type default) (color 0 0 0 0))
@@
     (stroke (width 0) (type default) (color 0 0 0 0))
   )
+  (polyline (pts (xy 129.54 242.57) (xy 68.58 242.57))
+    (stroke (width 0) (type default) (color 0 0 0 0))
+  )
   (wire (pts (xy 165.1 203.2) (xy 176.53 203.2))
     (stroke (width 0) (type default) (color 0 0 0 0))
@@
     (stroke (width 0) (type default) (color 0 0 0 0))
   )
+  (polyline (pts (xy 138.43 160.02) (xy 129.54 160.02))
+    (stroke (width 0) (type default) (color 0 0 0 0))
+  )
   (wire (pts (xy 144.78 261.62) (xy 144.78 264.16))
     (stroke (width 0) (type default) (color 0 0 0 0))
@@
     (stroke (width 0) (type default) (color 0 0 0 0))
   )
+  (polyline (pts (xy 69.85 69.85) (xy 69.85 224.79))
+    (stroke (width 0) (type default) (color 0 0 0 0))
+  )
   (wire (pts (xy 144.78 139.7) (xy 144.78 142.24))
     (stroke (width 0) (type default) (color 0 0 0 0))
@@
     (stroke (width 0) (type default) (color 0 0 0 0))
   )
+  (polyline (pts (xy 46.99 375.92) (xy 46.99 398.78))
+    (stroke (width 0) (type default) (color 0 0 0 0))
+  )
   (wire (pts (xy 135.89 107.95) (xy 143.51 107.95))
     (stroke (width 0) (type default) (color 0 0 0 0))
@@
     (stroke (width 0) (type default) (color 0 0 0 0))
   )
+  (polyline (pts (xy 138.43 293.37) (xy 138.43 160.02))
+    (stroke (width 0) (type default) (color 0 0 0 0))
+  )
   (wire (pts (xy 160.02 163.83) (xy 139.7 163.83))
     (stroke (width 0) (type default) (color 0 0 0 0))
@@
     (stroke (width 0) (type default) (color 0 0 0 0))
   )
+  (polyline (pts (xy 264.16 180.34) (xy 223.52 180.34))
+    (stroke (width 0) (type default) (color 0 0 0 0))
+  )
   (wire (pts (xy 102.87 95.25) (xy 101.6 95.25))
     (stroke (width 0) (type default) (color 0 0 0 0))
@@
     (stroke (width 0) (type default) (color 0 0 0 0))
   )
+  (polyline (pts (xy 129.54 158.75) (xy 138.43 158.75))
+    (stroke (width 0) (type default) (color 0 0 0 0))
+  )
   (wire (pts (xy 144.78 154.94) (xy 144.78 157.48))
     (stroke (width 0) (type default) (color 0 0 0 0))
@@
     (stroke (width 0) (type default) (color 0 0 0 0))
   )
+  (polyline (pts (xy 129.54 160.02) (xy 129.54 242.57))
+    (stroke (width 0) (type default) (color 0 0 0 0))
+  )
   (wire (pts (xy 160.02 217.17) (xy 139.7 217.17))
     (stroke (width 0) (type default) (color 0 0 0 0))
@@
     (stroke (width 0) (type default) (color 0 0 0 0))
   )
+  (polyline (pts (xy 46.99 398.78) (xy 203.2 398.78))
+    (stroke (width 0) (type default) (color 0 0 0 0))
+  )
   (wire (pts (xy 106.68 251.46) (xy 120.65 251.46))
     (stroke (width 0) (type default) (color 0 0 0 0))
   )
+  (polyline (pts (xy 138.43 186.69) (xy 158.75 186.69))
+    (stroke (width 0) (type default) (color 0 0 0 0))
+  )
   (wire (pts (xy 191.77 110.49) (xy 191.77 111.76))
     (stroke (width 0) (type default) (color 0 0 0 0))
@@
     (stroke (width 0) (type default) (color 0 0 0 0))
   )
+  (polyline (pts (xy 68.58 242.57) (xy 68.58 375.92))
+    (stroke (width 0) (type default) (color 0 0 0 0))
+  )
   (wire (pts (xy 144.78 165.1) (xy 147.32 165.1))
     (stroke (width 0) (type default) (color 0 0 0 0))
@@
     (stroke (width 0) (type default) (color 0 0 0 0))
   )
+  (polyline (pts (xy 203.2 398.78) (xy 203.2 293.37))
+    (stroke (width 0) (type default) (color 0 0 0 0))
+  )
   (wire (pts (xy 97.79 128.27) (xy 100.33 128.27))
     (stroke (width 0) (type default) (color 0 0 0 0))
@@
     (stroke (width 0) (type default) (color 0 0 0 0))
   )
+  (polyline (pts (xy 158.75 186.69) (xy 158.75 229.87))
+    (stroke (width 0) (type default) (color 0 0 0 0))
+  )
   (wire (pts (xy 160.02 179.07) (xy 139.7 179.07))
     (stroke (width 0) (type default) (color 0 0 0 0))
@@
     (stroke (width 0) (type default) (color 0 0 0 0))
   )
+  (polyline (pts (xy 158.75 229.87) (xy 264.16 229.87))
+    (stroke (width 0) (type default) (color 0 0 0 0))
+  )
   (wire (pts (xy 125.73 256.54) (xy 139.7 256.54))
     (stroke (width 0) (type default) (color 0 0 0 0))
@@
     (stroke (width 0) (type default) (color 0 0 0 0))
   )
+  (polyline (pts (xy 223.52 69.85) (xy 69.85 69.85))
+    (stroke (width 0) (type default) (color 0 0 0 0))
+  )
   (wire (pts (xy 139.7 255.27) (xy 139.7 256.54))
     (stroke (width 0) (type default) (color 0 0 0 0))
@@
     (stroke (width 0) (type default) (color 0 0 0 0))
   )
+  (polyline (pts (xy 223.52 180.34) (xy 223.52 69.85))
+    (stroke (width 0) (type default) (color 0 0 0 0))
+  )
   (wire (pts (xy 139.7 166.37) (xy 139.7 167.64))
     (stroke (width 0) (type default) (color 0 0 0 0))
@@
     (stroke (width 0) (type default) (color 0 0 0 0))
   )
-  (text "~{BANK0} Rewrite" (at 224.79 224.79 0)
+  (text "~{BANK0} Recalc" (at 224.79 224.79 0)
     (effects (font (size 2.54 2.54)) (justify left bottom))
   )
@@
     (effects (font (size 1.27 1.27)) (justify left bottom))
   )
-  (text "Vector Pull + Dual Channel DMA Control Shim\n(1 per CPU)\n"
-    (at 17.145 31.75 0)
+  (text "CPU Shim (1 per CPU):\n1. DMA Control Shim\n2. Vector Pull Rewrite Shim\n\n"
+    (at 20.955 52.07 0)
+    (effects (font (size 5 5)) (justify left bottom))
+  )
+  (text "Vector Pull Rewrite Shim\n\n" (at 53.34 401.32 0)
+    (effects (font (size 5 5)) (justify left bottom))
+  )
+  (text "DMA Control Shim\n" (at 74.93 81.28 0)
     (effects (font (size 5 5)) (justify left bottom))
   )
@@
     (pin "1")
   )
-  (symbol (lib_id "power:VCC") (at 102.87 417.83 0) (unit 1)
-    (in_bom yes) (on_board yes) (fields_autoplaced)
-    (property "Reference" "#PWR037" (id 0) (at 102.87 421.64 0)
-      (effects (font (size 1.27 1.27)) hide)
-    )
-    (property "Value" "VCC" (id 1) (at 102.87 412.75 0))
-    (property "Footprint" "" (id 2) (at 102.87 417.83 0)
-      (effects (font (size 1.27 1.27)) hide)
-    )
-    (property "Datasheet" "" (id 3) (at 102.87 417.83 0)
-      (effects (font (size 1.27 1.27)) hide)
-    )
-    (pin "1")
-  )
   (symbol (lib_id "power:GND") (at 82.55 292.1 0) (unit 1)
     (in_bom yes) (on_board yes)
@@
     (pin "1")
   )
-  (symbol (lib_id "power:PWR_FLAG") (at 102.87 431.8 0) (unit 1)
-    (in_bom yes) (on_board yes) (fields_autoplaced)
-    (property "Reference" "#FLG04" (id 0) (at 102.87 429.895 0)
-      (effects (font (size 1.27 1.27)) hide)
-    )
-    (property "Value" "PWR_FLAG" (id 1) (at 102.87 426.72 0))
-    (property "Footprint" "" (id 2) (at 102.87 431.8 0)
-      (effects (font (size 1.27 1.27)) hide)
-    )
-    (property "Datasheet" "~" (id 3) (at 102.87 431.8 0)
-      (effects (font (size 1.27 1.27)) hide)
-    )
-    (pin "1")
-  )
   (symbol (lib_id "Connector_Generic:Conn_02x40_Odd_Even") (at 154.94 185.42 0) (mirror y) (unit 1)
     (in_bom yes) (on_board yes)
@@
     (pin "2")
   )
-  (symbol (lib_id "power:GND") (at 102.87 431.8 0) (unit 1)
-    (in_bom yes) (on_board yes)
-    (property "Reference" "#PWR038" (id 0) (at 102.87 438.15 0)
-      (effects (font (size 1.27 1.27)) hide)
-    )
-    (property "Value" "GND" (id 1) (at 102.87 435.61 0))
-    (property "Footprint" "" (id 2) (at 102.87 431.8 0)
-      (effects (font (size 1.27 1.27)) hide)
-    )
-    (property "Datasheet" "" (id 3) (at 102.87 431.8 0)
-      (effects (font (size 1.27 1.27)) hide)
-    )
-    (pin "1")
-  )
   (symbol (lib_id "Connector_Generic:Conn_02x08_Odd_Even") (at 123.19 210.82 0) (mirror y) (unit 1)
     (in_bom yes) (on_board yes) (fields_autoplaced)
@@
       (effects (font (size 1.27 1.27)) hide)
     )
-    (pin "1")
-  )
-  (symbol (lib_id "power:PWR_FLAG") (at 102.87 417.83 0) (mirror x) (unit 1)
-    (in_bom yes) (on_board yes) (fields_autoplaced)
-    (property "Reference" "#FLG03" (id 0) (at 102.87 419.735 0)
-      (effects (font (size 1.27 1.27)) hide)
-    )
-    (property "Value" "PWR_FLAG" (id 1) (at 102.87 422.91 0))
-    (property "Footprint" "" (id 2) (at 102.87 417.83 0)
-      (effects (font (size 1.27 1.27)) hide)
-    )
-    (property "Datasheet" "~" (id 3) (at 102.87 417.83 0)
-      (effects (font (size 1.27 1.27)) hide)
-    )

Commit message: Big push, Sysctl, DMA Reg
Parts:
- removed J17, J31: VPA/VDA, symbol Connector:Conn_01x02_Male
- removed J18, J32: Conn_02x40_Odd_Even, Connector_PinHeader_2.54mm:PinHeader_2x40_P2.54mm_Vertical, symbol Connector_Generic:Conn_02x40_Odd_Even
- removed J19: CPU, Connector_PinHeader_2.54mm:PinHeader_2x18_P2.54mm_Vertical, symbol Connector_Generic:Conn_02x18_Odd_Even
- removed J28: ~{BUFFER CS 2}, symbol Connector_Generic:Conn_02x01
- removed J29: ~{BUFFER CS 3}, symbol Connector_Generic:Conn_02x01
- removed J33: DMA, Connector_PinHeader_2.54mm:PinHeader_2x18_P2.54mm_Vertical, symbol Connector_Generic:Conn_02x18_Odd_Even
- removed J?: ~{BUFFER CS 0}, symbol Connector_Generic:Conn_02x01
- removed J?: VP Shim, symbol Connector_Generic:Conn_02x08_Odd_Even
- removed J?: VP Bypass, symbol Connector_Generic:Conn_02x04_Counter_Clockwise
- removed J?: ~{BUFFER CS 1}, symbol Connector_Generic:Conn_02x01
- removed J?: DMA Controller, symbol Connector_Generic:Conn_02x11_Odd_Even
- removed J?: DMA_REQ_LO, symbol Connector_Generic:Conn_02x08_Odd_Even
- removed J?: DMA Bypass, symbol Connector_Generic:Conn_02x08_Odd_Even
- removed J?: DMA_REQ_HI, symbol Connector_Generic:Conn_02x08_Odd_Even
- removed R1, R2, R3, R? (x2): 10K, symbol Device:R
- removed RN?: 10K, Resistor_THT:R_Array_SIP9, symbol Device:R_Network08
- removed U26, U? (x2): 74HC00, symbol 74xx:74HC00
- removed U30: 74HC08, symbol Vega816:74HC08
- removed U31: 74HC283, symbol Vega816:74HC283
- removed U? (x7): 74AHC32, Package_DIP:DIP-14_W7.62mm, symbol 74xx:74LS32
Connections:
- no-connect marks 2 -> 0
Other:
- note removed: "CPU Shim (1 per CPU): 1. DMA Control Shim 2. Vector Pull Rewrite Shim"
- note removed: "DMA Control Shim"
- note removed: "VP_REQ is high when A1-A3 are high ($E or $F) and VP is active (low), indicating fetch of IRQ vector."
- note removed: "Vector Pull Rewrite Shim"
- note removed: "~{BANK0} Recalc"
