File: kicad/Vega816/MemoryExpansionBus/irq_multiplex.kicad_sch (KiCad schematic)
At the start: 38 parts, among them J0A1 Conn_02x40_Odd_Even, J0B1 CPU, J43 VPA/VDA, J44 IO_AREA, J46 IRQ_OUT, J47 IRQ MUX IN, J48 I/O Ctrl, J49 A/D Bus 0, J50 IRQ MUX IN, J51 I/O Ctrl, J52 A/D Bus 1, J53 IRQ MUX IN, J54 I/O Ctrl, J55 A/D Bus 2, J56 IRQ MUX IN, J57 I/O Ctrl, J58 A/D Bus 3, U28 74HC00, U47 74LS30, U48 74LS30, U49 CD4012BE, U50 CD4012BE, U51 CD4012BE, U52 CD4012BE, U53 74LS138, U54 74LS138, U55 74HC238, U56 74LS138, U57 74HC32, U58 74HC00, U59 CD4012BE, U60 CD4012BE, U61 CD4012BE, U62 CD4012BE

Commit message: images
Changed lines of the file:
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@@
   (junction (at 54.61 388.62) (diameter 0) (color 0 0 0 0)
   )
-  (junction (at 176.53 212.09) (diameter 0) (color 0 0 0 0)
-  )
   (junction (at 487.68 806.45) (diameter 0) (color 0 0 0 0)
   )
@@
     (stroke (width 0) (type default) (color 0 0 0 0))
   )
-  (wire (pts (xy 176.53 212.09) (xy 176.53 254))
-    (stroke (width 0) (type default) (color 0 0 0 0))
-  )
   (wire (pts (xy 334.01 424.18) (xy 334.01 426.72))
     (stroke (width 0) (type default) (color 0 0 0 0))
@@
     (effects (font (size 1.27 1.27)) (justify left bottom))
   )
+  (label "A7" (at 236.22 655.32 180)
+    (effects (font (size 1.27 1.27)) (justify right bottom))
+  )
   (label "~{CSDEV0-3}" (at 237.49 457.2 0)
     (effects (font (size 1.27 1.27)) (justify left bottom))
@@
     (effects (font (size 1.27 1.27)) (justify left bottom))
   )
-  (label "~{RS}" (at 240.03 474.98 180)
+  (label "RS" (at 240.03 474.98 180)
     (effects (font (size 1.27 1.27)) (justify right bottom))
   )
@@
     (effects (font (size 1.27 1.27)) (justify left bottom))
   )
-  (label "~{RS}" (at 349.25 474.98 0)
+  (label "RS" (at 349.25 474.98 0)
     (effects (font (size 1.27 1.27)) (justify left bottom))
   )
@@
     (effects (font (size 1.27 1.27)) (justify left bottom))
   )
-  (label "~{RS}" (at 405.13 474.98 0)
+  (label "RS" (at 405.13 474.98 0)
     (effects (font (size 1.27 1.27)) (justify left bottom))
   )
@@
     (effects (font (size 1.27 1.27)) (justify left bottom))
   )
-  (label "~{RS}" (at 293.37 474.98 0)
+  (label "RS" (at 293.37 474.98 0)
     (effects (font (size 1.27 1.27)) (justify left bottom))
   )

Commit message: irq
Parts:
- removed J46: IRQ_OUT, Connector_PinHeader_2.54mm:PinHeader_2x40_P2.54mm_Vertical, symbol Connector_Generic:Conn_02x20_Odd_Even
- removed U28: 74HC00, symbol 74xx:74HC00
- removed U49, U50, U51, U52, U59, U60, U61, U62: CD4012BE, symbol VegaSyms:CD4012BE
- added J?: IRQ Out, symbol Connector_Generic:Conn_02x16_Odd_Even
- added J?: NMI Dispatch Bypass, symbol Connector_Generic:Conn_02x03_Odd_Even
- added U?: 74HC00, symbol 74xx:74HC00
Connections:
- net GND: now also J?.10 (Pin_10), J?.12 (Pin_12), J?.14 (Pin_14), J?.16 (Pin_16), J?.18 (Pin_18), J?.2 (Pin_2), J?.20 (Pin_20), J?.22 (Pin_22), J?.24 (Pin_24), J?.26 (Pin_26), J?.28 (Pin_28), J?.30 (Pin_30), J?.32 (Pin_32), J?.4 (Pin_4), J?.6 (Pin_6), J?.8 (Pin_8); no longer U47.1, U48.1
- net IRQ A: now also J?.5 (Pin_5), U48.8, U?.2; no longer J?.4 (Pin_4), U47.8
- net IRQ A+B: now also J?.1 (Pin_1), U?.3; no longer J?.2 (Pin_2)
- net IRQ B: now also J?.3 (Pin_3), U47.8, U?.1; no longer J?.6 (Pin_6), U48.8
- net ~{IRQA0}: now also U48.12, J?.31 (Pin_31); no longer J47.1 (Pin_1), J50.1 (Pin_1), J53.1 (Pin_1), J56.1 (Pin_1), U47.12
- net ~{IRQA1}: now also U48.11, J?.29 (Pin_29); no longer U47.11
- net ~{IRQA2}: now also U48.6, J?.27 (Pin_27); no longer U47.6
- net ~{IRQA3}: now also U48.5, J?.25 (Pin_25); no longer U47.5
- net ~{IRQA4}: now also U48.4, J?.23 (Pin_23); no longer U47.4
- net ~{IRQA5}: now also U48.3, J?.21 (Pin_21); no longer U47.3
- net ~{IRQA6}: now also U48.2, J?.19 (Pin_19); no longer U47.2
- net ~{IRQA7}: now also U48.1, U58.2, J?.17 (Pin_17), J?.5 (Pin_5)
- net ~{IRQB0}: now also U47.12, J?.15 (Pin_15); no longer U48.12
- net ~{IRQB1}: now also U47.11, J?.13 (Pin_13); no longer U48.11
- net ~{IRQB2}: now also U47.6, J?.11 (Pin_11); no longer U48.6
- net ~{IRQB3}: now also U47.5, J?.9 (Pin_9); no longer U48.5
- net ~{IRQB4}: now also U47.4, J?.7 (Pin_7); no longer U48.4
- net ~{IRQB5}: now also U47.3, J?.5 (Pin_5); no longer U48.3
- net ~{IRQB6}: now also U47.2, J?.3 (Pin_3); no longer U48.2
- net ~{IRQ}: now also J?.2 (Pin_2), J?.4 (Pin_4), J?.6 (Pin_6); no longer J?.1 (Pin_1), J?.3 (Pin_3), J?.5 (Pin_5)
- net ~{NMI}: now also J?.2 (Pin_2), J?.4 (Pin_4), J?.6 (Pin_6)
- new net ~{IRQA7} NAND ~{IRQB7}: J?.1 (Pin_1), U58.3
- new net ~{IRQB7}: J47.1 (Pin_1), J50.1 (Pin_1), J53.1 (Pin_1), J56.1 (Pin_1), J?.1 (Pin_1), J?.3 (Pin_3), U47.1, U58.1
- no-connect marks 20 -> 4
Other:
- note added: "Install one jumper maximum"
- note added: "Jumpers set base address between $0000 and $7E00. Page above base page reserved for IRQ metadata. Decodes ~{CS} for up to 16 devices on 16 byte boundaries. Provides four I/O device slots of 64 bytes address space each."
- note removed: "Decodes ~{CS} for up to 16 devices on 16 byte boundaries in $0200 $0300 is also sensed for Programmable Interrupt Controller configuration."
- note removed: "Install only one jumper."
- moved on the sheet: J0A1, J0B1, J43, J?, U47B, U48B, U53, U54, U55, U57A, U57B, U57C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

Commit message: svg
Parts:
- added D?: 1N4148, Diode_THT:D_DO-35_SOD27_P7.62mm_Horizontal, symbol Diode:1N4148
- added J?: IO_AREA_IN, symbol Connector_Generic:Conn_02x01
- J44: value IO_AREA -> IO_AREA_OUT
Connections:
- net GND: now also J?.2 (Pin_2)
- net at U57.3: now also D?.1 (K); no longer J44.1 (Pin_1)
- net $0200/0300-$027F/037F renamed $0000/0100-$007F/017F
- new net: D?.2 (A), J44.1 (Pin_1), J?.1 (Pin_1)
Changed lines of the file:
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@@
   (junction (at 262.89 283.21) (diameter 0) (color 0 0 0 0)
   )
+  (junction (at 26.67 302.26) (diameter 0) (color 0 0 0 0)
+  )
   (junction (at 191.77 184.15) (diameter 0) (color 0 0 0 0)
   )
@@
   (junction (at 142.24 140.97) (diameter 0) (color 0 0 0 0)
   )
+  (junction (at 40.64 302.26) (diameter 0) (color 0 0 0 0)
+  )
   (junction (at 157.48 143.51) (diameter 0) (color 0 0 0 0)
   )
@@
     (stroke (width 0) (type default) (color 0 0 0 0))
   )
+  (wire (pts (xy 40.64 508) (xy 295.91 508))
+    (stroke (width 0) (type default) (color 0 0 0 0))
+  )
   (wire (pts (xy 247.65 245.11) (xy 250.19 245.11))
     (stroke (width 0) (type default) (color 0 0 0 0))
@@
     (stroke (width 0) (type default) (color 0 0 0 0))
   )
+  (wire (pts (xy 40.64 302.26) (xy 40.64 299.72))
+    (stroke (width 0) (type default) (color 0 0 0 0))
+  )
   (wire (pts (xy 247.65 273.05) (xy 247.65 275.59))
     (stroke (width 0) (type default) (color 0 0 0 0))
@@
     (stroke (width 0) (type default) (color 0 0 0 0))
   )
-  (wire (pts (xy 295.91 508) (xy 40.64 508))
-    (stroke (width 0) (type default) (color 0 0 0 0))
-  )
   (wire (pts (xy 359.41 214.63) (xy 361.95 214.63))
     (stroke (width 0) (type default) (color 0 0 0 0))
@@
     (stroke (width 0) (type default) (color 0 0 0 0))
   )
+  (wire (pts (xy 40.64 302.26) (xy 39.37 302.26))
+    (stroke (width 0) (type default) (color 0 0 0 0))
+  )
   (wire (pts (xy 245.11 260.35) (xy 245.11 259.08))
     (stroke (width 0) (type default) (color 0 0 0 0))
@@
     (stroke (width 0) (type default) (color 0 0 0 0))
   )
+  (wire (pts (xy 26.67 302.26) (xy 26.67 299.72))
+    (stroke (width 0) (type default) (color 0 0 0 0))
+  )
   (wire (pts (xy 200.66 485.14) (xy 207.01 485.14))
     (stroke (width 0) (type default) (color 0 0 0 0))
@@
     (stroke (width 0) (type default) (color 0 0 0 0))
   )
-  (wire (pts (xy 40.64 508) (xy 40.64 299.72))
+  (wire (pts (xy 40.64 508) (xy 40.64 309.88))
     (stroke (width 0) (type default) (color 0 0 0 0))
   )
@@
     (stroke (width 0) (type default) (color 0 0 0 0))
   )
+  (wire (pts (xy 26.67 306.07) (xy 26.67 302.26))
+    (stroke (width 0) (type default) (color 0 0 0 0))
+  )
   (wire (pts (xy 350.52 162.56) (xy 350.52 163.83))
     (stroke (width 0) (type default) (color 0 0 0 0))
@@
     (effects (font (size 1.27 1.27)) (justify right bottom))
   )
-  (label "$0200{slash}0300-$027F{slash}037F" (at 231.14 430.53 0)
+  (label "$0000{slash}0100-$007F{slash}017F" (at 231.14 430.53 0)
     (effects (font (size 1.27 1.27)) (justify left bottom))
   )
@@
     (effects (font (size 1.27 1.27)) (justify right bottom))
   )
-  (label "$0280{slash}0380-$02FF{slash}03FF" (at 231.14 440.69 0)
+  (label "$0080{slash}0180-$00FF{slash}01FF" (at 231.14 440.69 0)
     (effects (font (size 1.27 1.27)) (justify left bottom))
   )
@@
     (pin "7")
   )
+  (symbol (lib_id "Connector_Generic:Conn_02x01") (at 34.29 302.26 0) (mirror y) (unit 1)
+    (in_bom yes) (on_board yes)
+    (property "Reference" "J?" (id 0) (at 33.02 295.91 0)
+      (effects (font (size 1.27 1.27)) hide)
+    )
+    (property "Value" "IO_AREA_IN" (id 1) (at 33.02 304.8 0))
+    (property "Footprint" "" (id 2) (at 34.29 302.26 0)
+      (effects (font (size 1.27 1.27)) hide)
+    )
+    (property "Datasheet" "~" (id 3) (at 34.29 302.26 0)
+      (effects (font (size 1.27 1.27)) hide)
+    )
+    (pin "1")
+    (pin "2")
+  )
   (symbol (lib_id "74xx:74LS138") (at 143.51 450.85 0) (unit 1)
     (in_bom yes) (on_board yes)
@@
     (pin "1")
   )
+  (symbol (lib_id "Diode:1N4148") (at 40.64 306.07 270) (mirror x) (unit 1)
+    (in_bom yes) (on_board yes) (fields_autoplaced)
+    (property "Reference" "D?" (id 0) (at 43.18 304.7999 90)
+      (effects (font (size 1.27 1.27)) (justify left))
+    )
+    (property "Value" "1N4148" (id 1) (at 43.18 307.3399 90)
+      (effects (font (size 1.27 1.27)) (justify left))
+    )
+    (property "Footprint" "Diode_THT:D_DO-35_SOD27_P7.62mm_Horizontal" (id 2) (at 40.64 306.07 0)
+      (effects (font (size 1.27 1.27)) hide)
+    )
+    (property "Datasheet" "https://assets.nexperia.com/documents/data-sheet/1N4148_1N4448.pdf" (id 3) (at 40.64 306.07 0)
+      (effects (font (size 1.27 1.27)) hide)
+    )
+    (pin "1")
+    (pin "2")
+  )
   (symbol (lib_id "74xx:74LS30") (at 130.81 143.51 0) (mirror y) (unit 1)
     (in_bom yes) (on_board yes)
@@
   )
   (symbol (lib_id "Connector_Generic:Conn_02x01") (at 34.29 299.72 0) (mirror y) (unit 1)
-    (in_bom yes) (on_board yes) (fields_autoplaced)
+    (in_bom yes) (on_board yes)
     (property "Reference" "J44" (id 0) (at 33.02 293.37 0)
       (effects (font (size 1.27 1.27)) hide)
     )
-    (property "Value" "IO_AREA" (id 1) (at 33.02 295.91 0))
+    (property "Value" "IO_AREA_OUT" (id 1) (at 33.02 297.18 0))
     (property "Footprint" "" (id 2) (at 34.29 299.72 0)
       (effects (font (size 1.27 1.27)) hide)
@@
     (pin "2")
   )
-  (symbol (lib_name "GND_2") (lib_id "power:GND") (at 26.67 299.72 0) (unit 1)
+  (symbol (lib_name "GND_2") (lib_id "power:GND") (at 26.67 306.07 0) (unit 1)
     (in_bom yes) (on_board yes)
-    (property "Reference" "#PWR086" (id 0) (at 26.67 306.07 0)
+    (property "Reference" "#PWR086" (id 0) (at 26.67 312.42 0)
       (effects (font (size 1.27 1.27)) hide)
     )
-    (property "Value" "GND" (id 1) (at 26.67 303.53 0))
-    (property "Footprint" "" (id 2) (at 26.67 299.72 0)
+    (property "Value" "GND" (id 1) (at 26.67 309.88 0))
+    (property "Footprint" "" (id 2) (at 26.67 306.07 0)
       (effects (font (size 1.27 1.27)) hide)
     )
-    (property "Datasheet" "" (id 3) (at 26.67 299.72 0)
+    (property "Datasheet" "" (id 3) (at 26.67 306.07 0)
       (effects (font (size 1.27 1.27)) hide)
     )
