File: kicad/Vega816/MemoryExpansionBus/irq_multiplex.kicad_sch (KiCad schematic)
At the start: 33 parts, among them J0A1 Conn_02x40_Odd_Even, J0B1 CPU, J43 VPA/VDA, J44 IO_AREA_OUT, J47 IRQ MUX IN, J48 I/O Ctrl, J49 A/D Bus 0, J50 IRQ MUX IN, J51 I/O Ctrl, J52 A/D Bus 1, J53 IRQ MUX IN, J54 I/O Ctrl, J55 A/D Bus 2, J56 IRQ MUX IN, J57 I/O Ctrl, J58 A/D Bus 3, U47 74LS30, U48 74LS30, U53 74LS138, U54 74LS138, U55 74HC238, U56 74LS138, U57 74HC32, U58 74HC00

Commit message: svg
Other:
- note added: "Incoming IRQ Multiplex"
- note added: "Jumpers set base address to even numbered pages between $0000 and $7E00. Page above base page reserved for PIC configuration."
- note added: "Provides four I/O device slots of 64 bytes address space each. Decodes ~{CS} for into 4 16-byte ranges per slot."
- note added: "Quad 64 B IO Bus"
- note removed: "Demultiplexes incoming IRQs for IRQ Vector Pull Dispatch 8 priorities x 2 CPU targets"
- note removed: "Jumpers set base address between $0000 and $7E00. Page above base page reserved for IRQ metadata. Decodes ~{CS} for up to 16 devices on 16 byte boundaries. Provides four I/O device slots of 64 bytes address space each."
- note removed: "Quad I/O Bus + IRQ Demux + IO Address Decode"
Changed lines of the file:
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@@
     (stroke (width 0) (type default) (color 0 0 0 0))
+  )
+  (text "Provides four I/O device slots of 64 bytes address space each.\n\nDecodes ~{CS} for into 4 16-byte ranges per slot.\n\n\n\n\n"
+    (at 30.48 133.35 0)
+    (effects (font (size 5 5)) (justify left bottom))
   )
   (text "Install one jumper maximum\n\n" (at 99.06 170.18 180)
     (effects (font (size 1.27 1.27)) (justify right bottom))
   )
-  (text "Demultiplexes incoming IRQs for IRQ Vector Pull Dispatch\n8 priorities x 2 CPU targets"
-    (at 158.75 125.73 0)
+  (text "Incoming IRQ Multiplex" (at 223.52 127 0)
+    (effects (font (size 3 3)) (justify left bottom))
+  )
+  (text "Quad 64 B IO Bus" (at 22.86 40.64 0)
+    (effects (font (size 10 10)) (justify left bottom))
+  )
+  (text "Jumpers set base address to even numbered pages\nbetween $0000 and $7E00.\nPage above base page reserved for PIC configuration.\n\n"
+    (at 30.48 78.74 0)
     (effects (font (size 5 5)) (justify left bottom))
   )
-  (text "Quad I/O Bus + IRQ Demux + IO Address Decode" (at 22.86 40.64 0)
-    (effects (font (size 10 10)) (justify left bottom))
-  )
-  (text "Jumpers set base address between $0000 and $7E00.\nPage above base page reserved for IRQ metadata.\n\nDecodes ~{CS} for up to 16 devices on 16 byte boundaries.\nProvides four I/O device slots of 64 bytes address space each.\n\n\n\n"
-    (at 26.67 110.49 0)
-    (effects (font (size 5 5)) (justify left bottom))
-  )

Commit message: xvsvd
Other:
- note added: "Provides four I/O device slots of 64 bytes address space each. Decodes ~{CS} for 4 16-byte ranges per slot."
- note removed: "Provides four I/O device slots of 64 bytes address space each. Decodes ~{CS} for into 4 16-byte ranges per slot."
Changed lines of the file:
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@@
     (stroke (width 0) (type default) (color 0 0 0 0))
   )
-  (text "Provides four I/O device slots of 64 bytes address space each.\n\nDecodes ~{CS} for into 4 16-byte ranges per slot.\n\n\n\n\n"
+  (text "Provides four I/O device slots of 64 bytes address space each.\n\nDecodes ~{CS} for 4 16-byte ranges per slot.\n\n\n\n\n"
     (at 30.48 133.35 0)
     (effects (font (size 5 5)) (justify left bottom))
@@
     (effects (font (size 5 5)) (justify left bottom))
   )
+  (text "Install one jumper maximum\n\n" (at 97.79 204.47 180)
+    (effects (font (size 1.27 1.27)) (justify right bottom))
+  )
   (label "D2" (at 374.65 278.13 0)

Commit message: expansion port hi ram
Parts:
- added JP?: HI_32KB, symbol Jumper:Jumper_3_Open
Connections:
- net A15: now also U58.10, U58.9, JP?.1 (A); no longer U56.5 (E2)
- net at U58.8: now also JP?.3 (B)
- net ~{$0000-$0FFF} renamed ~{+$0000-$0FFF}
- net ~{$1000-$1FFF} renamed ~{+$1000-$1FFF}
- net ~{$2000-$2FFF} renamed ~{+$2000-$2FFF}
- net ~{$3000-$3FFF} renamed ~{+$3000-$3FFF}
- net ~{$4000-$4FFF} renamed ~{+$4000-$4FFF}
- net ~{$5000-$5FFF} renamed ~{+$5000-$5FFF}
- net ~{$6000-$6FFF} renamed ~{+$6000-$6FFF}
- net ~{$7000-$7FFF} renamed ~{+$7000-$7FFF}
- new net: JP?.2 (C), U56.5 (E2)
Other:
- note added: "Page $00-$7E"
- note added: "Page $80-$FE"
- moved on the sheet: U58C
Changed lines of the file:
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@@
   (junction (at 207.01 161.29) (diameter 0) (color 0 0 0 0)
   )
+  (junction (at 158.75 487.68) (diameter 0) (color 0 0 0 0)
+  )
   (junction (at 191.77 229.87) (diameter 0) (color 0 0 0 0)
   )
@@
   (junction (at 261.62 482.6) (diameter 0) (color 0 0 0 0)
   )
+  (junction (at 162.56 494.03) (diameter 0) (color 0 0 0 0)
+  )
   (junction (at 191.77 247.65) (diameter 0) (color 0 0 0 0)
   )
@@
     (stroke (width 0) (type default) (color 0 0 0 0))
   )
+  (wire (pts (xy 177.8 494.03) (xy 180.34 494.03))
+    (stroke (width 0) (type default) (color 0 0 0 0))
+  )
   (wire (pts (xy 173.99 144.78) (xy 173.99 146.05))
     (stroke (width 0) (type default) (color 0 0 0 0))
@@
     (stroke (width 0) (type default) (color 0 0 0 0))
   )
+  (wire (pts (xy 158.75 494.03) (xy 162.56 494.03))
+    (stroke (width 0) (type default) (color 0 0 0 0))
+  )
   (wire (pts (xy 359.41 186.69) (xy 361.95 186.69))
     (stroke (width 0) (type default) (color 0 0 0 0))
@@
     (stroke (width 0) (type default) (color 0 0 0 0))
   )
+  (wire (pts (xy 207.01 499.11) (xy 207.01 490.22))
+    (stroke (width 0) (type default) (color 0 0 0 0))
+  )
   (wire (pts (xy 318.77 238.76) (xy 318.77 240.03))
     (stroke (width 0) (type default) (color 0 0 0 0))
@@
     (stroke (width 0) (type default) (color 0 0 0 0))
   )
+  (wire (pts (xy 158.75 481.33) (xy 180.34 481.33))
+    (stroke (width 0) (type default) (color 0 0 0 0))
+  )
   (wire (pts (xy 359.41 146.05) (xy 361.95 146.05))
     (stroke (width 0) (type default) (color 0 0 0 0))
@@
     (stroke (width 0) (type default) (color 0 0 0 0))
   )
-  (wire (pts (xy 78.74 490.22) (xy 207.01 490.22))
+  (wire (pts (xy 78.74 499.11) (xy 207.01 499.11))
     (stroke (width 0) (type default) (color 0 0 0 0))
   )
@@
     (stroke (width 0) (type default) (color 0 0 0 0))
   )
-  (wire (pts (xy 78.74 222.25) (xy 78.74 490.22))
+  (wire (pts (xy 162.56 494.03) (xy 162.56 491.49))
+    (stroke (width 0) (type default) (color 0 0 0 0))
+  )
+  (wire (pts (xy 78.74 222.25) (xy 78.74 499.11))
     (stroke (width 0) (type default) (color 0 0 0 0))
   )
@@
     (stroke (width 0) (type default) (color 0 0 0 0))
   )
-  (wire (pts (xy 76.2 487.68) (xy 207.01 487.68))
+  (wire (pts (xy 76.2 487.68) (xy 158.75 487.68))
     (stroke (width 0) (type default) (color 0 0 0 0))
   )
@@
     (stroke (width 0) (type default) (color 0 0 0 0))
   )
+  (wire (pts (xy 158.75 481.33) (xy 158.75 487.68))
+    (stroke (width 0) (type default) (color 0 0 0 0))
+  )
   (wire (pts (xy 115.57 430.53) (xy 115.57 443.23))
     (stroke (width 0) (type default) (color 0 0 0 0))
@@
     (stroke (width 0) (type default) (color 0 0 0 0))
   )
+  (wire (pts (xy 158.75 487.68) (xy 158.75 494.03))
+    (stroke (width 0) (type default) (color 0 0 0 0))
+  )
   (wire (pts (xy 356.87 261.62) (xy 374.65 261.62))
     (stroke (width 0) (type default) (color 0 0 0 0))
@@
     (stroke (width 0) (type default) (color 0 0 0 0))
   )
+  (wire (pts (xy 184.15 487.68) (xy 207.01 487.68))
+    (stroke (width 0) (type default) (color 0 0 0 0))
+  )
   (wire (pts (xy 191.77 201.93) (xy 191.77 204.47))
     (stroke (width 0) (type default) (color 0 0 0 0))
@@
     (stroke (width 0) (type default) (color 0 0 0 0))
   )
+  (wire (pts (xy 162.56 494.03) (xy 162.56 496.57))
+    (stroke (width 0) (type default) (color 0 0 0 0))
+  )
   (wire (pts (xy 24.13 245.11) (xy 26.67 245.11))
     (stroke (width 0) (type default) (color 0 0 0 0))
@@
     (effects (font (size 10 10)) (justify left bottom))
   )
+  (text "Page $00-$7E" (at 181.61 491.49 0)
+    (effects (font (size 1.27 1.27)) (justify left bottom))
+  )
   (text "Jumpers set base address to even numbered pages\nbetween $0000 and $7E00.\nPage above base page reserved for PIC configuration.\n\n"
     (at 30.48 78.74 0)
     (effects (font (size 5 5)) (justify left bottom))
   )
+  (text "Page $80-$FE" (at 181.61 486.41 0)
+    (effects (font (size 1.27 1.27)) (justify left bottom))
+  )
   (text "Install one jumper maximum\n\n" (at 97.79 204.47 180)
     (effects (font (size 1.27 1.27)) (justify right bottom))
@@
     (effects (font (size 1.27 1.27)) (justify left bottom))
   )
-  (label "~{$6000-$6FFF}" (at 232.41 487.68 0)
+  (label "~{+$6000-$6FFF}" (at 232.41 487.68 0)
     (effects (font (size 1.27 1.27)) (justify left bottom))
   )
@@
     (effects (font (size 1.27 1.27)) (justify left bottom))
   )
-  (label "~{$0000-$0FFF}" (at 232.41 472.44 0)
+  (label "~{+$0000-$0FFF}" (at 232.41 472.44 0)
     (effects (font (size 1.27 1.27)) (justify left bottom))
   )
@@
     (effects (font (size 1.27 1.27)) (justify left bottom))
   )
-  (label "~{$7000-$7FFF}" (at 232.41 490.22 0)
+  (label "~{+$7000-$7FFF}" (at 232.41 490.22 0)
     (effects (font (size 1.27 1.27)) (justify left bottom))
   )
@@
     (effects (font (size 1.27 1.27)) (justify left bottom))
   )
-  (label "~{$4000-$4FFF}" (at 232.41 482.6 0)
+  (label "~{+$4000-$4FFF}" (at 232.41 482.6 0)
     (effects (font (size 1.27 1.27)) (justify left bottom))
   )
@@
     (effects (font (size 1.27 1.27)) (justify left bottom))
   )
-  (label "~{$2000-$2FFF}" (at 232.41 477.52 0)
+  (label "~{+$2000-$2FFF}" (at 232.41 477.52 0)
     (effects (font (size 1.27 1.27)) (justify left bottom))
   )
@@
     (effects (font (size 1.27 1.27)) (justify left bottom))
   )
-  (label "~{$1000-$1FFF}" (at 232.41 474.98 0)
+  (label "~{+$1000-$1FFF}" (at 232.41 474.98 0)
     (effects (font (size 1.27 1.27)) (justify left bottom))
   )
@@
     (effects (font (size 1.27 1.27)) (justify left bottom))
   )
-  (label "~{$3000-$3FFF}" (at 232.41 480.06 0)
+  (label "~{+$3000-$3FFF}" (at 232.41 480.06 0)
     (effects (font (size 1.27 1.27)) (justify left bottom))
   )
@@
     (effects (font (size 1.27 1.27)) (justify left bottom))
   )
-  (label "A15" (at 207.01 487.68 180)
+  (label "A15" (at 158.75 487.68 180)
     (effects (font (size 1.27 1.27)) (justify right bottom))
   )
@@
     (effects (font (size 1.27 1.27)) (justify right bottom))
   )
-  (label "~{$5000-$5FFF}" (at 232.41 485.14 0)
+  (label "~{+$5000-$5FFF}" (at 232.41 485.14 0)
     (effects (font (size 1.27 1.27)) (justify left bottom))
   )
@@
     (effects (font (size 1.27 1.27)) (justify right bottom))
   )
-  (label "~{BANK0}" (at 205.74 490.22 180)
+  (label "~{BANK0}" (at 205.74 499.11 180)
     (effects (font (size 1.27 1.27)) (justify right bottom))
   )
@@
     (pin "7")
   )
-  (symbol (lib_id "74xx:74HC00") (at 321.31 468.63 0) (unit 3)
+  (symbol (lib_id "74xx:74HC00") (at 170.18 494.03 0) (unit 3)
     (in_bom yes) (on_board yes)
-    (property "Reference" "U58" (id 0) (at 321.31 467.36 0))
-    (property "Value" "74HC00" (id 1) (at 321.31 469.9 0))
-    (property "Footprint" "" (id 2) (at 321.31 468.63 0)
+    (property "Reference" "U58" (id 0) (at 170.18 492.76 0))
+    (property "Value" "74HC00" (id 1) (at 170.18 495.3 0))
+    (property "Footprint" "" (id 2) (at 170.18 494.03 0)
       (effects (font (size 1.27 1.27)) hide)
     )
-    (property "Datasheet" "http://www.ti.com/lit/gpn/sn74hc00" (id 3) (at 321.31 468.63 0)
+    (property "Datasheet" "http://www.ti.com/lit/gpn/sn74hc00" (id 3) (at 170.18 494.03 0)
       (effects (font (size 1.27 1.27)) hide)
     )
@@
     (pin "9")
   )
+  (symbol (lib_id "Jumper:Jumper_3_Open") (at 180.34 487.68 90) (mirror x) (unit 1)
+    (in_bom yes) (on_board yes)
+    (property "Reference" "JP?" (id 0) (at 177.8 486.4099 90)
+      (effects (font (size 1.27 1.27)) (justify left))
+    )
+    (property "Value" "HI_32KB" (id 1) (at 177.8 483.8699 90)
+      (effects (font (size 1.27 1.27)) (justify left))
+    )
+    (property "Footprint" "" (id 2) (at 180.34 487.68 0)
+      (effects (font (size 1.27 1.27)) hide)
+    )
+    (property "Datasheet" "~" (id 3) (at 180.34 487.68 0)
+      (effects (font (size 1.27 1.27)) hide)
+    )
+    (pin "1")
+    (pin "2")
+    (pin "3")
+  )
   (symbol (lib_id "Connector_Generic:Conn_02x20_Odd_Even") (at 201.93 257.81 0) (mirror y) (unit 1)

Commit message: C
Parts:
- removed D?: 1N4148, Diode_THT:D_DO-35_SOD27_P7.62mm_Horizontal, symbol Diode:1N4148
- removed J?: IO_AREA_IN, symbol Connector_Generic:Conn_02x01
- added D?: 1N4148, Diode_THT:D_DO-35_SOD27_P7.62mm_Horizontal, symbol Diode:1N4148
- added J?: IO_AREA_IN, symbol Connector_Generic:Conn_02x01
Connections:
- net GND: now also J?.2 (Pin_2)
- net at U57.3: now also D?.1 (K)
- net at J44.1 (Pin_1): now also D?.2 (A), J?.1 (Pin_1)

Commit message: Big push, Sysctl, DMA Reg
Parts:
- renumbered J0A1 to J0A?, J0B1 to J0B?, J58 to J?, J56 to J?, J57 to J?, J48 to J?, J44 to J?, J47 to J?, J55 to J?, J54 to J?, J51 to J?, J52 to J?, J50 to J?, J53 to J?, J49 to J?, J43 to J?, U54 to U?, U57 to U?, U58 to U?, U56 to U?, U48 to U?, U47 to U?, U53 to U?, U55 to U?
