File: kicad/Vega816/MemoryExpansionBus/pic.kicad_sch (KiCad schematic)
At the start: 68 parts, among them J59 IRQ_OUT, J60 I/O Ctrl, J61 A/D Bus, U10 74LS08, U100 74HC238, U101 74LS241, U102 74LS241, U103 74LS241, U104 74LS241, U105 74HC373, U106 74HC238, U107 74LS244, U108 74HC238, U109 74LS241, U110 74LS241, U111 74LS241, U112 74LS241, U113 74LS30, U114 74LS30, U115 74LS30, U116 74LS30, U117 74LS30, U118 74LS30, U119 74LS30, U120 74LS30, U2 74LS08, U24 74HC00, U26 74HC00, U29 74HC00, U5 74LS08, U58 74HC00, U63 74HC00, U64 74HC00, U65 74LS02, U66 74HC00, U67 74HC00, U68 74LS02, U69 74LS02, U70 74LS08, U71 74HC00, U72 74LS00, U73 74HC373, U74 74HC238, U75 74LS244, U76 74HC238, U77 74LS30, U78 74LS30, U79 74LS30, U80 74LS30, U81 74LS30, U82 74LS30, U83 74LS30, U84 74LS30, U85 74LS241, U86 74LS241, U87 74LS241, U88 74LS241, U89 74HC373, U90 74HC238, U91 74LS244, U92 74HC238, U93 74LS241, U94 74LS241, U95 74LS241, U96 74LS241, U97 74HC373, U98 74HC238, U99 74LS244

Commit message: images
Connections:
- net D6 is gone; now on net D0: J61.27 (Pin_27), U105.4 (D1), U107.16 (O1a), U75.16 (O1a), U89.4 (D1), U91.16 (O1a), U97.4 (D1), U99.16 (O1a)
- net D7 is gone; now on net D1: J61.25 (Pin_25), U105.3 (D0), U107.18 (O0a), U75.18 (O0a), U89.3 (D0), U91.18 (O0a), U97.3 (D0), U99.18 (O0a)
- net D0: now also U73.18 (D7), U73.4 (D1)
- net D1: now also U73.17 (D6), U73.3 (D0)
- net D2: now also U73.14 (D5)
- net D3: now also U73.13 (D4)
- net D4: now also U73.8 (D3)
- net D5: now also U73.7 (D2)

Commit message: update
Connections:
- net ~{NMIA} renamed ~{IRQA7}
- net ~{NMIB} renamed ~{IRQB7}
Other:
- note added: "7"
- note removed: "NMI"
Changed lines of the file:
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@@
     (effects (font (size 10 10)) (justify left bottom))
   )
-  (text "3" (at 1080.77 201.93 0)
+  (text "3" (at 1070.61 201.93 0)
     (effects (font (size 10 10)) (justify left bottom))
   )
@@
     (effects (font (size 3 3)) (justify left bottom))
   )
-  (text "2" (at 1080.77 181.61 0)
-    (effects (font (size 10 10)) (justify left bottom))
-  )
-  (text "NMI" (at 345.44 132.08 0)
-    (effects (font (size 10 10)) (justify left bottom))
-  )
-  (text "5" (at 1080.77 242.57 0)
+  (text "2" (at 1070.61 181.61 0)
+    (effects (font (size 10 10)) (justify left bottom))
+  )
+  (text "7" (at 359.41 132.08 0)
+    (effects (font (size 10 10)) (justify left bottom))
+  )
+  (text "5" (at 1070.61 242.57 0)
     (effects (font (size 10 10)) (justify left bottom))
   )
@@
     (effects (font (size 10 10)) (justify left bottom))
   )
-  (text "6" (at 1080.77 262.89 0)
-    (effects (font (size 10 10)) (justify left bottom))
-  )
-  (text "0\n" (at 1080.77 142.24 0)
+  (text "6" (at 1070.61 262.89 0)
+    (effects (font (size 10 10)) (justify left bottom))
+  )
+  (text "0\n" (at 1070.61 142.24 0)
     (effects (font (size 10 10)) (justify left bottom))
   )
@@
     (effects (font (size 10 10)) (justify left bottom))
   )
-  (text "1" (at 1080.77 161.29 0)
-    (effects (font (size 10 10)) (justify left bottom))
-  )
-  (text "4" (at 1080.77 220.98 0)
-    (effects (font (size 10 10)) (justify left bottom))
-  )
-  (text "NMI" (at 1071.88 284.48 0)
+  (text "1" (at 1070.61 161.29 0)
+    (effects (font (size 10 10)) (justify left bottom))
+  )
+  (text "4" (at 1070.61 220.98 0)
+    (effects (font (size 10 10)) (justify left bottom))
+  )
+  (text "7" (at 1070.61 284.48 0)
     (effects (font (size 10 10)) (justify left bottom))
   )
@@
     (effects (font (size 1.27 1.27)) (justify left bottom))
   )
-  (label "~{NMIA}" (at 31.75 391.16 0)
+  (label "~{IRQA7}" (at 31.75 391.16 0)
     (effects (font (size 1.27 1.27)) (justify left bottom))
   )
@@
     (effects (font (size 1.27 1.27)) (justify left bottom))
   )
-  (label "~{NMIB}" (at 31.75 370.84 0)
-    (effects (font (size 1.27 1.27)) (justify left bottom))
-  )
+  (label "~{IRQB7}" (at 31.75 370.84 0)
+    (effects (font (size 1.27 1.27)) (justify left bottom))
+  )

Commit message: irq
Parts:
- added D? (x16): 1N4148, Diode_THT:D_DO-35_SOD27_P7.62mm_Horizontal, symbol Diode:1N4148
Connections:
- net ~{IRQA0}: now also D?.2 (A); no longer U84.8
- net ~{IRQA1}: now also D?.2 (A); no longer U83.8
- net ~{IRQA2}: now also D?.2 (A); no longer U82.8
- net ~{IRQA3}: now also D?.2 (A); no longer U81.8
- net ~{IRQA4}: now also D?.2 (A); no longer U80.8
- net ~{IRQA5}: now also D?.2 (A); no longer U79.8
- net ~{IRQA6}: now also D?.2 (A); no longer U78.8
- net ~{IRQA7}: now also D?.2 (A); no longer U77.8
- net ~{IRQB0}: now also D?.2 (A); no longer U113.8
- net ~{IRQB1}: now also D?.2 (A); no longer U114.8
- net ~{IRQB2}: now also D?.2 (A); no longer U115.8
- net ~{IRQB3}: now also D?.2 (A); no longer U116.8
- net ~{IRQB4}: now also D?.2 (A); no longer U117.8
- net ~{IRQB5}: now also D?.2 (A); no longer U118.8
- net ~{IRQB6}: now also D?.2 (A); no longer U119.8
- net ~{IRQB7}: now also D?.2 (A); no longer U120.8
- new net ~{IRQA0_0}: D?.1 (K), U84.8
- new net ~{IRQA1_0}: D?.1 (K), U83.8
- new net ~{IRQA2_0}: D?.1 (K), U82.8
- new net ~{IRQA3_0}: D?.1 (K), U81.8
- new net ~{IRQA4_0}: D?.1 (K), U80.8
- new net ~{IRQA5_0}: D?.1 (K), U79.8
- new net ~{IRQA6_0}: D?.1 (K), U78.8
- new net ~{IRQA7_0}: D?.1 (K), U77.8
- new net ~{IRQB0_0}: D?.1 (K), U113.8
- new net ~{IRQB1_0}: D?.1 (K), U114.8
- new net ~{IRQB2_0}: D?.1 (K), U115.8
- new net ~{IRQB3_0}: D?.1 (K), U116.8
- new net ~{IRQB4_0}: D?.1 (K), U117.8
- new net ~{IRQB5_0}: D?.1 (K), U118.8
- new net ~{IRQB6_0}: D?.1 (K), U119.8
- new net ~{IRQB7_0}: D?.1 (K), U120.8
Other:
- note added: "+$"
- note added: "Control Nybble format: 8421 TPPP High bit is Target (T) 0 = This DMA channel's primary CPU, 1 = The other DMA channel's primary CPU Low three bits (PPP) are priority, 0-7."
- note added: "Device Control Byte Offset Offset Nybble +$00 +$100 low +$08 +$100 high +$10 +$110 low +$18 +$110 high +$20 +$120 low +$28 +$120 high +$30 +$130 low +$38 +$130 high"
- note added: "Diode NAND for IRQ chaining"

Commit message: dvg
Connections:
- net D0: no longer J61.27 (Pin_27), U105.4 (D1), U107.16 (O1a), U73.4 (D1), U75.16 (O1a), U89.4 (D1), U91.16 (O1a), U97.4 (D1), U99.16 (O1a)
- net D1: no longer J61.25 (Pin_25), U105.3 (D0), U107.18 (O0a), U73.3 (D0), U75.18 (O0a), U89.3 (D0), U91.18 (O0a), U97.3 (D0), U99.18 (O0a)
- new net D6: J61.27 (Pin_27), U105.4 (D1), U107.16 (O1a), U73.4 (D1), U75.16 (O1a), U89.4 (D1), U91.16 (O1a), U97.4 (D1), U99.16 (O1a)
- new net D7: J61.25 (Pin_25), U105.3 (D0), U107.18 (O0a), U73.3 (D0), U75.18 (O0a), U89.3 (D0), U91.18 (O0a), U97.3 (D0), U99.18 (O0a)
Changed lines of the file:
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@@
   (junction (at 862.33 576.58) (diameter 0) (color 0 0 0 0)
   )
-  (junction (at 262.89 603.25) (diameter 0) (color 0 0 0 0)
-  )
   (junction (at 113.03 434.34) (diameter 0) (color 0 0 0 0)
   )
@@
   (junction (at 16.51 398.78) (diameter 0) (color 0 0 0 0)
   )
-  (junction (at 264.16 605.79) (diameter 0) (color 0 0 0 0)
-  )
   (junction (at 398.78 576.58) (diameter 0) (color 0 0 0 0)
   )
@@
     (stroke (width 0) (type default) (color 0 0 0 0))
   )
-  (wire (pts (xy 262.89 603.25) (xy 262.89 618.49))
+  (wire (pts (xy 262.89 574.04) (xy 262.89 618.49))
     (stroke (width 0) (type default) (color 0 0 0 0))
   )
@@
     (stroke (width 0) (type default) (color 0 0 0 0))
   )
-  (wire (pts (xy 255.27 603.25) (xy 262.89 603.25))
-    (stroke (width 0) (type default) (color 0 0 0 0))
-  )
   (wire (pts (xy 1008.38 204.47) (xy 1008.38 490.22))
     (stroke (width 0) (type default) (color 0 0 0 0))
@@
     (stroke (width 0) (type default) (color 0 0 0 0))
   )
-  (wire (pts (xy 262.89 574.04) (xy 262.89 603.25))
-    (stroke (width 0) (type default) (color 0 0 0 0))
-  )
   (wire (pts (xy 16.51 459.74) (xy 19.05 459.74))
     (stroke (width 0) (type default) (color 0 0 0 0))
@@
     (stroke (width 0) (type default) (color 0 0 0 0))
   )
-  (wire (pts (xy 264.16 576.58) (xy 264.16 605.79))
-    (stroke (width 0) (type default) (color 0 0 0 0))
-  )
   (wire (pts (xy 922.02 453.39) (xy 919.48 453.39))
     (stroke (width 0) (type default) (color 0 0 0 0))
@@
     (stroke (width 0) (type default) (color 0 0 0 0))
   )
-  (wire (pts (xy 256.54 605.79) (xy 264.16 605.79))
-    (stroke (width 0) (type default) (color 0 0 0 0))
-  )
   (wire (pts (xy 384.81 433.07) (xy 373.38 433.07))
     (stroke (width 0) (type default) (color 0 0 0 0))
@@
     (stroke (width 0) (type default) (color 0 0 0 0))
   )
-  (wire (pts (xy 262.89 603.25) (xy 389.89 603.25))
+  (wire (pts (xy 255.27 603.25) (xy 389.89 603.25))
     (stroke (width 0) (type default) (color 0 0 0 0))
   )
@@
     (stroke (width 0) (type default) (color 0 0 0 0))
   )
-  (wire (pts (xy 264.16 605.79) (xy 391.16 605.79))
+  (wire (pts (xy 256.54 605.79) (xy 391.16 605.79))
     (stroke (width 0) (type default) (color 0 0 0 0))
   )
@@
     (stroke (width 0) (type default) (color 0 0 0 0))
   )
-  (wire (pts (xy 264.16 605.79) (xy 264.16 621.03))
+  (wire (pts (xy 264.16 576.58) (xy 264.16 621.03))
     (stroke (width 0) (type default) (color 0 0 0 0))
   )

Commit message: svg
Parts:
- removed D? (x16): 1N4148, Diode_THT:D_DO-35_SOD27_P7.62mm_Horizontal, symbol Diode:1N4148
- removed U10, U2, U5, U70: 74LS08, symbol 74xx:74LS08
- removed U100, U106, U108, U74, U76, U90, U92, U98: 74HC238, symbol 74xx:74HC238
- removed U101, U102, U103, U104, U109, U110, U111, U112, U85, U86, U87, U88, U93, U94, U95, U96: 74LS241, symbol 74xx:74LS241
- removed U105, U73, U89, U97: 74HC373, symbol 74xx:74HC373
- removed U107, U75, U91, U99: 74LS244, symbol 74xx:74LS244
- removed U113, U114, U115, U116, U117, U118, U119, U120, U77, U78, U79, U80, U81, U82, U83, U84: 74LS30, symbol 74xx:74LS30
- removed U24, U26, U29, U58, U63, U64, U66, U67, U71: 74HC00, symbol 74xx:74HC00
- removed U65, U68, U69: 74LS02, symbol 74xx:74LS02
- removed U72: 74LS00, symbol 74xx:74LS00
- added J?: DEV4-5 PIC, symbol Connector_Generic:Conn_02x31_Odd_Even
- added J?: DEV0-1 PIC, symbol Connector_Generic:Conn_02x31_Odd_Even
- added J?: DEV6-7 PIC, symbol Connector_Generic:Conn_02x31_Odd_Even
- added J?: DEV2-3 PIC, symbol Connector_Generic:Conn_02x31_Odd_Even
Connections:
- net ~{CSDEV2-3} is gone; now on net ~{CSDEV0-1}: J60.37 (Pin_37)
- net ~{CSDEV4-5} is gone; now on net ~{CSDEV0-1}: J60.35 (Pin_35)
- net ~{CSDEV6-7} is gone; now on net ~{CSDEV0-1}: J60.33 (Pin_33)
- net D0: now also J?.61 (Pin_61), J?.61 (Pin_61), J?.61 (Pin_61), J?.61 (Pin_61)
- net D1: now also J?.59 (Pin_59), J?.59 (Pin_59), J?.59 (Pin_59), J?.59 (Pin_59)
- net D2: now also J?.57 (Pin_57), J?.57 (Pin_57), J?.57 (Pin_57), J?.57 (Pin_57)
- net D3: now also J?.55 (Pin_55), J?.55 (Pin_55), J?.55 (Pin_55), J?.55 (Pin_55)
- net D4: now also J?.53 (Pin_53), J?.53 (Pin_53), J?.53 (Pin_53), J?.53 (Pin_53)
- net D5: now also J?.51 (Pin_51), J?.51 (Pin_51), J?.51 (Pin_51), J?.51 (Pin_51)
- net D6: now also J?.49 (Pin_49), J?.49 (Pin_49), J?.49 (Pin_49), J?.49 (Pin_49)
- net D7: now also J?.47 (Pin_47), J?.47 (Pin_47), J?.47 (Pin_47), J?.47 (Pin_47)
- net GND: now also J?.10 (Pin_10), J?.10 (Pin_10), J?.10 (Pin_10), J?.10 (Pin_10), J?.12 (Pin_12), J?.12 (Pin_12), J?.12 (Pin_12), J?.12 (Pin_12), J?.14 (Pin_14), J?.14 (Pin_14), J?.14 (Pin_14), J?.14 (Pin_14), J?.16 (Pin_16), J?.16 (Pin_16), J?.16 (Pin_16), J?.16 (Pin_16), J?.18 (Pin_18), J?.18 (Pin_18), J?.18 (Pin_18), J?.18 (Pin_18), J?.2 (Pin_2), J?.2 (Pin_2), J?.2 (Pin_2), J?.2 (Pin_2), J?.20 (Pin_20), J?.20 (Pin_20), J?.20 (Pin_20), J?.20 (Pin_20), J?.22 (Pin_22), J?.22 (Pin_22), J?.22 (Pin_22), J?.22 (Pin_22), J?.24 (Pin_24), J?.24 (Pin_24), J?.24 (Pin_24), J?.24 (Pin_24), J?.26 (Pin_26), J?.26 (Pin_26), J?.26 (Pin_26), J?.26 (Pin_26), J?.28 (Pin_28), J?.28 (Pin_28), J?.28 (Pin_28), J?.28 (Pin_28), J?.30 (Pin_30), J?.30 (Pin_30), J?.30 (Pin_30), J?.30 (Pin_30), J?.32 (Pin_32), J?.32 (Pin_32), J?.32 (Pin_32), J?.32 (Pin_32), J?.34 (Pin_34), J?.34 (Pin_34), J?.34 (Pin_34), J?.34 (Pin_34), J?.36 (Pin_36), J?.36 (Pin_36), J?.36 (Pin_36), J?.36 (Pin_36), J?.38 (Pin_38), J?.38 (Pin_38), J?.38 (Pin_38), J?.38 (Pin_38), J?.4 (Pin_4), J?.4 (Pin_4), J?.4 (Pin_4), J?.4 (Pin_4), J?.40 (Pin_40), J?.40 (Pin_40), J?.40 (Pin_40), J?.40 (Pin_40), J?.42 (Pin_42), J?.42 (Pin_42), J?.42 (Pin_42), J?.42 (Pin_42), J?.44 (Pin_44), J?.44 (Pin_44), J?.44 (Pin_44), J?.44 (Pin_44), J?.45 (Pin_45), J?.45 (Pin_45), J?.45 (Pin_45), J?.45 (Pin_45), J?.46 (Pin_46), J?.46 (Pin_46), J?.46 (Pin_46), J?.46 (Pin_46), J?.48 (Pin_48), J?.48 (Pin_48), J?.48 (Pin_48), J?.48 (Pin_48), J?.50 (Pin_50), J?.50 (Pin_50), J?.50 (Pin_50), J?.50 (Pin_50), J?.52 (Pin_52), J?.52 (Pin_52), J?.52 (Pin_52), J?.52 (Pin_52), J?.54 (Pin_54), J?.54 (Pin_54), J?.54 (Pin_54), J?.54 (Pin_54), J?.56 (Pin_56), J?.56 (Pin_56), J?.56 (Pin_56), J?.56 (Pin_56), J?.58 (Pin_58), J?.58 (Pin_58), J?.58 (Pin_58), J?.58 (Pin_58), J?.6 (Pin_6), J?.6 (Pin_6), J?.6 (Pin_6), J?.6 (Pin_6), J?.60 (Pin_60), J?.60 (Pin_60), J?.60 (Pin_60), J?.60 (Pin_60), J?.62 (Pin_62), J?.62 (Pin_62), J?.62 (Pin_62), J?.62 (Pin_62), J?.8 (Pin_8), J?.8 (Pin_8), J?.8 (Pin_8), J?.8 (Pin_8)
- net R~{W}: now also J?.39 (Pin_39), J?.39 (Pin_39), J?.39 (Pin_39), J?.39 (Pin_39)
- net VCC: now also J?.43 (Pin_43), J?.43 (Pin_43), J?.43 (Pin_43), J?.43 (Pin_43)
- net ~{CSDEV0-1}: now also J?.37 (Pin_37), J?.37 (Pin_37), J?.37 (Pin_37), J?.37 (Pin_37)
- net ~{IRQA0}: now also J?.31 (Pin_31), J?.31 (Pin_31), J?.31 (Pin_31), J?.31 (Pin_31)
- net ~{IRQA1}: now also J?.29 (Pin_29), J?.29 (Pin_29), J?.29 (Pin_29), J?.29 (Pin_29)
- net ~{IRQA2}: now also J?.27 (Pin_27), J?.27 (Pin_27), J?.27 (Pin_27), J?.27 (Pin_27)
- net ~{IRQA3}: now also J?.25 (Pin_25), J?.25 (Pin_25), J?.25 (Pin_25), J?.25 (Pin_25)
- net ~{IRQA4}: now also J?.23 (Pin_23), J?.23 (Pin_23), J?.23 (Pin_23), J?.23 (Pin_23)
- net ~{IRQA5}: now also J?.21 (Pin_21), J?.21 (Pin_21), J?.21 (Pin_21), J?.21 (Pin_21)
- net ~{IRQA6}: now also J?.19 (Pin_19), J?.19 (Pin_19), J?.19 (Pin_19), J?.19 (Pin_19)
- net ~{IRQA7}: now also J?.17 (Pin_17), J?.17 (Pin_17), J?.17 (Pin_17), J?.17 (Pin_17)
- net ~{IRQB0}: now also J?.15 (Pin_15), J?.15 (Pin_15), J?.15 (Pin_15), J?.15 (Pin_15)
- net ~{IRQB1}: now also J?.13 (Pin_13), J?.13 (Pin_13), J?.13 (Pin_13), J?.13 (Pin_13)
- net ~{IRQB2}: now also J?.11 (Pin_11), J?.11 (Pin_11), J?.11 (Pin_11), J?.11 (Pin_11)
- net ~{IRQB3}: now also J?.9 (Pin_9), J?.9 (Pin_9), J?.9 (Pin_9), J?.9 (Pin_9)
- net ~{IRQB4}: now also J?.7 (Pin_7), J?.7 (Pin_7), J?.7 (Pin_7), J?.7 (Pin_7)
- net ~{IRQB5}: now also J?.5 (Pin_5), J?.5 (Pin_5), J?.5 (Pin_5), J?.5 (Pin_5)
- net ~{IRQB6}: now also J?.3 (Pin_3), J?.3 (Pin_3), J?.3 (Pin_3), J?.3 (Pin_3)
- net ~{IRQB7}: now also J?.1 (Pin_1), J?.1 (Pin_1), J?.1 (Pin_1), J?.1 (Pin_1)
- net ~{IRQDEV0}: now also J?.35 (Pin_35)
- net ~{IRQDEV1}: now also J?.33 (Pin_33)
- net ~{IRQDEV2}: now also J?.35 (Pin_35)
- net ~{IRQDEV3}: now also J?.33 (Pin_33)
- net ~{IRQDEV4}: now also J?.35 (Pin_35)
- net ~{IRQDEV5}: now also J?.33 (Pin_33)
- net ~{IRQDEV6}: now also J?.35 (Pin_35)
- net ~{IRQDEV7}: now also J?.33 (Pin_33)
- net A8 renamed RS
- net RS: now also J?.41 (Pin_41), J?.41 (Pin_41), J?.41 (Pin_41), J?.41 (Pin_41)
Other:
- note added: "Quad PIC (8 IRQ)"
- note removed: "+$"
- note removed: "0"
- note removed: "1"
- note removed: "2"
- note removed: "3"
- note removed: "4"
- note removed: "5"
- note removed: "6"
- note removed: "7"
- note removed: "Diode NAND for IRQ chaining"
- note removed: "IRQ A"
- note removed: "IRQ B"
- note removed: "Latch Enable"
- note removed: "Latch Output Enable"
- note removed: "Programmable Interrupt Controller"

Commit message: C
Changed lines of the file:
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@@
   (junction (at 373.38 317.5) (diameter 0) (color 0 0 0 0)
   )
-  (junction (at 330.2 307.34) (diameter 0) (color 0 0 0 0)
-  )
   (junction (at 63.5 273.05) (diameter 0) (color 0 0 0 0)
   )
@@
   (junction (at 63.5 217.17) (diameter 0) (color 0 0 0 0)
   )
-  (junction (at 271.78 307.34) (diameter 0) (color 0 0 0 0)
-  )
   (junction (at 256.54 284.48) (diameter 0) (color 0 0 0 0)
   )
@@
   (junction (at 213.36 261.5666) (diameter 0) (color 0 0 0 0)
   )
-  (junction (at 213.36 307.34) (diameter 0) (color 0 0 0 0)
-  )
   (junction (at 63.5 311.15) (diameter 0) (color 0 0 0 0)
   )
@@
     (stroke (width 0) (type default) (color 0 0 0 0))
   )
-  (wire (pts (xy 330.2 307.34) (xy 372.11 307.34))
-    (stroke (width 0) (type default) (color 0 0 0 0))
-  )
   (wire (pts (xy 314.96 276.86) (xy 317.5 276.86))
     (stroke (width 0) (type default) (color 0 0 0 0))
@@
     (stroke (width 0) (type default) (color 0 0 0 0))
   )
-  (wire (pts (xy 196.85 306.07) (xy 213.36 306.07))
-    (stroke (width 0) (type default) (color 0 0 0 0))
-  )
   (wire (pts (xy 198.12 264.16) (xy 198.12 266.7))
     (stroke (width 0) (type default) (color 0 0 0 0))
@@
     (stroke (width 0) (type default) (color 0 0 0 0))
   )
-  (wire (pts (xy 271.78 306.07) (xy 271.78 307.34))
-    (stroke (width 0) (type default) (color 0 0 0 0))
-  )
   (wire (pts (xy 63.5 351.79) (xy 66.04 351.79))
     (stroke (width 0) (type default) (color 0 0 0 0))
@@
     (stroke (width 0) (type default) (color 0 0 0 0))
   )
-  (wire (pts (xy 213.36 306.07) (xy 213.36 307.34))
-    (stroke (width 0) (type default) (color 0 0 0 0))
-  )
   (wire (pts (xy 213.36 311.15) (xy 213.36 312.42))
     (stroke (width 0) (type default) (color 0 0 0 0))
@@
     (stroke (width 0) (type default) (color 0 0 0 0))
   )
-  (wire (pts (xy 271.78 307.34) (xy 313.69 307.34))
-    (stroke (width 0) (type default) (color 0 0 0 0))
-  )
   (wire (pts (xy 373.38 297.18) (xy 375.92 297.18))
     (stroke (width 0) (type default) (color 0 0 0 0))
@@
     (stroke (width 0) (type default) (color 0 0 0 0))
   )
-  (wire (pts (xy 372.11 306.07) (xy 388.62 306.07))
-    (stroke (width 0) (type default) (color 0 0 0 0))
-  )
   (wire (pts (xy 271.78 326.39) (xy 271.78 327.66))
     (stroke (width 0) (type default) (color 0 0 0 0))
@@
     (stroke (width 0) (type default) (color 0 0 0 0))
   )
-  (wire (pts (xy 372.11 307.34) (xy 372.11 306.07))
-    (stroke (width 0) (type default) (color 0 0 0 0))
-  )
   (wire (pts (xy 120.65 330.2) (xy 120.65 356.87))
     (stroke (width 0) (type default) (color 0 0 0 0))
@@
     (stroke (width 0) (type default) (color 0 0 0 0))
   )
-  (wire (pts (xy 93.98 307.34) (xy 196.85 307.34))
-    (stroke (width 0) (type default) (color 0 0 0 0))
-  )
   (wire (pts (xy 78.74 262.89) (xy 140.97 262.89))
     (stroke (width 0) (type default) (color 0 0 0 0))
@@
     (stroke (width 0) (type default) (color 0 0 0 0))
   )
-  (wire (pts (xy 93.98 323.85) (xy 78.74 323.85))
-    (stroke (width 0) (type default) (color 0 0 0 0))
-  )
   (wire (pts (xy 271.78 273.05) (xy 271.78 274.2666))
     (stroke (width 0) (type default) (color 0 0 0 0))
@@
     (stroke (width 0) (type default) (color 0 0 0 0))
   )
-  (wire (pts (xy 255.27 307.34) (xy 255.27 306.07))
-    (stroke (width 0) (type default) (color 0 0 0 0))
-  )
   (wire (pts (xy 373.38 261.62) (xy 373.38 264.16))
     (stroke (width 0) (type default) (color 0 0 0 0))
@@
     (stroke (width 0) (type default) (color 0 0 0 0))
   )
-  (wire (pts (xy 93.98 307.34) (xy 93.98 323.85))
-    (stroke (width 0) (type default) (color 0 0 0 0))
-  )
   (wire (pts (xy 166.37 281.94) (xy 166.37 237.49))
     (stroke (width 0) (type default) (color 0 0 0 0))
@@
     (stroke (width 0) (type default) (color 0 0 0 0))
   )
-  (wire (pts (xy 313.69 306.07) (xy 330.2 306.07))
-    (stroke (width 0) (type default) (color 0 0 0 0))
-  )
   (wire (pts (xy 330.2 271.78) (xy 372.11 271.78))
     (stroke (width 0) (type default) (color 0 0 0 0))
@@
     (stroke (width 0) (type default) (color 0 0 0 0))
   )
-  (wire (pts (xy 388.62 306.07) (xy 388.62 307.34))
-    (stroke (width 0) (type default) (color 0 0 0 0))
-  )
   (wire (pts (xy 330.2 312.42) (xy 372.11 312.42))
     (stroke (width 0) (type default) (color 0 0 0 0))
@@
     (stroke (width 0) (type default) (color 0 0 0 0))
   )
-  (wire (pts (xy 313.69 307.34) (xy 313.69 306.07))
-    (stroke (width 0) (type default) (color 0 0 0 0))
-  )
   (wire (pts (xy 373.38 256.54) (xy 375.92 256.54))
     (stroke (width 0) (type default) (color 0 0 0 0))
@@
     (stroke (width 0) (type default) (color 0 0 0 0))
   )
-  (wire (pts (xy 213.36 307.34) (xy 255.27 307.34))
-    (stroke (width 0) (type default) (color 0 0 0 0))
-  )
   (wire (pts (xy 256.54 304.8) (xy 256.54 307.34))
     (stroke (width 0) (type default) (color 0 0 0 0))
@@
     (stroke (width 0) (type default) (color 0 0 0 0))
   )
-  (wire (pts (xy 196.85 307.34) (xy 196.85 306.07))
-    (stroke (width 0) (type default) (color 0 0 0 0))
-  )
   (wire (pts (xy 63.5 323.85) (xy 63.5 326.39))
     (stroke (width 0) (type default) (color 0 0 0 0))
@@
     (stroke (width 0) (type default) (color 0 0 0 0))
   )
-  (wire (pts (xy 330.2 306.07) (xy 330.2 307.34))
-    (stroke (width 0) (type default) (color 0 0 0 0))
-  )
   (wire (pts (xy 372.11 260.35) (xy 388.62 260.35))
     (stroke (width 0) (type default) (color 0 0 0 0))
@@
     (stroke (width 0) (type default) (color 0 0 0 0))
   )
-  (wire (pts (xy 255.27 306.07) (xy 271.78 306.07))
-    (stroke (width 0) (type default) (color 0 0 0 0))
-  )
