File: kicad/Vega816/MemoryExpansionBus/64_to_32_16_8_byte_device_breakout.kicad_sch (KiCad schematic)
At the start: 26 parts, among them J62 IRQ_OUT, J63 Device Select, J64 A/D Bus, J65 IRQ_OUT, J66 Device Select, J67 A/D Bus, J68 $00 (64 B), J69 $00 (32B), J70 $30 (8B IRQ 6), J71 $00 (16B IRQ 0-1), J72 $80 (32B), J73 $38 (8B IRQ 7), J74 $10 (16B IRQ 2-3), J75 $20(16B IRQ 4-5), J76 $00 (16B), J77 $40 (16B), J78 $80 (16B), J79 $A0 (16B), J80 $00 (8B), J81 $08 (8B), J82 $10 (8B), J83 $18 (8B), J84 $20 (8B), J85 $28 (8B), J86 $30 (8B), J87 $38 (8B)

Commit message: svg
Parts:
- added J? (x2): ~{CS} Decode, symbol Connector_Generic:Conn_02x20_Odd_Even
- added U? (x12): 74HC00, symbol 74xx:74HC00
Connections:
- net A3: now also J?.35 (Pin_35), J?.35 (Pin_35), J?.37 (Pin_37), J?.39 (Pin_39), U?.1, U?.1, U?.12, U?.2, U?.4, U?.9
- net GND: now also J?.10 (Pin_10), J?.10 (Pin_10), J?.12 (Pin_12), J?.12 (Pin_12), J?.14 (Pin_14), J?.14 (Pin_14), J?.16 (Pin_16), J?.16 (Pin_16), J?.18 (Pin_18), J?.18 (Pin_18), J?.2 (Pin_2), J?.2 (Pin_2), J?.20 (Pin_20), J?.20 (Pin_20), J?.22 (Pin_22), J?.22 (Pin_22), J?.24 (Pin_24), J?.24 (Pin_24), J?.26 (Pin_26), J?.26 (Pin_26), J?.28 (Pin_28), J?.28 (Pin_28), J?.30 (Pin_30), J?.30 (Pin_30), J?.32 (Pin_32), J?.32 (Pin_32), J?.33 (Pin_33), J?.33 (Pin_33), J?.34 (Pin_34), J?.34 (Pin_34), J?.36 (Pin_36), J?.36 (Pin_36), J?.38 (Pin_38), J?.38 (Pin_38), J?.4 (Pin_4), J?.4 (Pin_4), J?.40 (Pin_40), J?.40 (Pin_40), J?.6 (Pin_6), J?.6 (Pin_6), J?.8 (Pin_8), J?.8 (Pin_8)
- net VCC: now also J?.31 (Pin_31), J?.31 (Pin_31)
- net ~{CSDEV0-1}: now also J?.23 (Pin_23), J?.23 (Pin_23), U?.13, U?.13, U?.13
- net ~{CSDEV0-3}: now also J?.27 (Pin_27), J?.27 (Pin_27), U?.11, U?.12
- net ~{CSDEV0-7}: now also J?.29 (Pin_29), J?.29 (Pin_29), U?.11
- net ~{CSDEV0}: now also J?.15 (Pin_15), J?.15 (Pin_15), U?.11
- net ~{CSDEV1}: now also J?.13 (Pin_13), J?.13 (Pin_13), U?.11
- net ~{CSDEV2-3}: now also J?.21 (Pin_21), J?.21 (Pin_21), U?.10, U?.10, U?.12
- net ~{CSDEV2}: now also J?.11 (Pin_11), J?.11 (Pin_11), U?.8
- net ~{CSDEV3}: now also J?.9 (Pin_9), J?.9 (Pin_9), U?.8
- net ~{CSDEV4-5}: now also J?.19 (Pin_19), J?.19 (Pin_19), U?.13, U?.5, U?.5
- net ~{CSDEV4-7}: now also J?.25 (Pin_25), J?.25 (Pin_25), U?.11, U?.13
- net ~{CSDEV4}: now also J?.7 (Pin_7), J?.7 (Pin_7), U?.6
- net ~{CSDEV5}: now also J?.5 (Pin_5), J?.5 (Pin_5), U?.6
- net ~{CSDEV6-7}: now also J?.17 (Pin_17), J?.17 (Pin_17), U?.12, U?.2, U?.2
- net ~{CSDEV6}: now also J?.3 (Pin_3), J?.3 (Pin_3), U?.3
- net ~{CSDEV7}: now also J?.1 (Pin_1), J?.1 (Pin_1), U?.3
- new net ~{A3}: U?.1, U?.12, U?.3, U?.4, U?.9
- no-connect marks 13 -> 17
Other:
- note added: "16 B ~{CS} Inputs Aggregation: 16 -> 32/64 Byte Device Disaggregation: 16 -> 8 Byte Device"
- note added: "Full 64 Byte IO Bus Breakout"
- note added: "~{CS} Decode"
- note removed: "Fully Populated IO Bus Breakout (Delete unneeded connectors for a custom breakout)"

Commit message: new plots
Connections:
- net A3: no longer J?.37 (Pin_37), J?.39 (Pin_39)
Changed lines of the file:
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@@
   (junction (at 308.61 344.17) (diameter 0) (color 0 0 0 0)
   )
-  (junction (at 54.61 148.59) (diameter 0) (color 0 0 0 0)
-  )
   (junction (at 546.1 171.45) (diameter 0) (color 0 0 0 0)
   )
@@
   (junction (at 254 156.21) (diameter 0) (color 0 0 0 0)
   )
-  (junction (at 54.61 146.05) (diameter 0) (color 0 0 0 0)
-  )
   (junction (at 83.82 151.13) (diameter 0) (color 0 0 0 0)
   )
@@
     (stroke (width 0) (type default) (color 0 0 0 0))
   )
-  (wire (pts (xy 54.61 146.05) (xy 54.61 143.51))
-    (stroke (width 0) (type default) (color 0 0 0 0))
-  )
   (wire (pts (xy 591.82 344.17) (xy 608.33 344.17))
     (stroke (width 0) (type default) (color 0 0 0 0))
@@
     (stroke (width 0) (type default) (color 0 0 0 0))
   )
-  (wire (pts (xy 54.61 158.75) (xy 54.61 148.59))
+  (wire (pts (xy 58.42 143.51) (xy 58.42 158.75))
     (stroke (width 0) (type default) (color 0 0 0 0))
   )
@@
     (stroke (width 0) (type default) (color 0 0 0 0))
   )
+  (wire (pts (xy 58.42 143.51) (xy 54.61 143.51))
+    (stroke (width 0) (type default) (color 0 0 0 0))
+  )
   (wire (pts (xy 592.455 156.21) (xy 592.455 82.55))
     (stroke (width 0) (type default) (color 0 0 0 0))
@@
     (stroke (width 0) (type default) (color 0 0 0 0))
   )
-  (wire (pts (xy 54.61 148.59) (xy 54.61 146.05))
-    (stroke (width 0) (type default) (color 0 0 0 0))
-  )
   (wire (pts (xy 457.2 185.42) (xy 457.2 186.69))
     (stroke (width 0) (type default) (color 0 0 0 0))
@@
     (stroke (width 0) (type default) (color 0 0 0 0))
   )
-  (wire (pts (xy 82.55 158.75) (xy 54.61 158.75))
+  (wire (pts (xy 82.55 158.75) (xy 58.42 158.75))
     (stroke (width 0) (type default) (color 0 0 0 0))
   )
@@
     (pin "9")
   )
+  (symbol (lib_id "power:GND") (at 41.91 151.13 0) (mirror y) (unit 1)
+    (in_bom yes) (on_board yes)
+    (property "Reference" "#PWR?" (id 0) (at 41.91 157.48 0)
+      (effects (font (size 1.27 1.27)) hide)
+    )
+    (property "Value" "GND" (id 1) (at 44.323 155.5242 0))
+    (property "Footprint" "" (id 2) (at 41.91 151.13 0)
+      (effects (font (size 1.27 1.27)) hide)
+    )
+    (property "Datasheet" "" (id 3) (at 41.91 151.13 0)
+      (effects (font (size 1.27 1.27)) hide)
+    )
+    (pin "1")
+  )
   (symbol (lib_name "GND_2") (lib_id "power:GND") (at 495.3 199.39 0) (unit 1)
