File: kicad/Vega816/MemoryExpansionBus/c64sidandcias.kicad_sch (KiCad schematic)
At the start: 7 parts, among them J62 IRQ_OUT, J63 Device Select, J64 A/D Bus, J72 $80 (32B), J76 $00 (16B), J77 $40 (16B)

Commit message: expansion port hi ram
Parts:
- removed U?: 74HC00, symbol 74xx:74HC00
- added U?: 74HC00, symbol 74xx:74HC00
Connections:
- net ~{CSDEV4-5}: now also U?.13
- net ~{CSDEV4-7}: now also U?.11
- net ~{CSDEV6-7}: now also U?.12
Other:
- note added: "8580/6581 (SID)"
- note added: "VIA (CIA) #1"
- note added: "VIA (CIA) #2"

Commit message: C
Parts:
- added J? (x2): ~{CS} Decode, symbol Connector_Generic:Conn_02x20_Odd_Even
Connections:
- net A3: now also J?.35 (Pin_35), J?.35 (Pin_35)
- net GND: now also J?.10 (Pin_10), J?.10 (Pin_10), J?.12 (Pin_12), J?.12 (Pin_12), J?.14 (Pin_14), J?.14 (Pin_14), J?.16 (Pin_16), J?.16 (Pin_16), J?.18 (Pin_18), J?.18 (Pin_18), J?.2 (Pin_2), J?.2 (Pin_2), J?.20 (Pin_20), J?.20 (Pin_20), J?.22 (Pin_22), J?.22 (Pin_22), J?.24 (Pin_24), J?.24 (Pin_24), J?.26 (Pin_26), J?.26 (Pin_26), J?.28 (Pin_28), J?.28 (Pin_28), J?.30 (Pin_30), J?.30 (Pin_30), J?.32 (Pin_32), J?.32 (Pin_32), J?.33 (Pin_33), J?.33 (Pin_33), J?.34 (Pin_34), J?.34 (Pin_34), J?.36 (Pin_36), J?.36 (Pin_36), J?.38 (Pin_38), J?.38 (Pin_38), J?.4 (Pin_4), J?.4 (Pin_4), J?.40 (Pin_40), J?.40 (Pin_40), J?.6 (Pin_6), J?.6 (Pin_6), J?.8 (Pin_8), J?.8 (Pin_8)
- net VCC: now also J?.31 (Pin_31), J?.31 (Pin_31)
- net ~{CSDEV0-1}: now also J?.23 (Pin_23), J?.23 (Pin_23)
- net ~{CSDEV0-3}: now also J?.27 (Pin_27), J?.27 (Pin_27)
- net ~{CSDEV0-7}: now also J?.29 (Pin_29), J?.29 (Pin_29)
- net ~{CSDEV0}: now also J?.15 (Pin_15), J?.15 (Pin_15)
- net ~{CSDEV1}: now also J?.13 (Pin_13), J?.13 (Pin_13)
- net ~{CSDEV2-3}: now also J?.21 (Pin_21), J?.21 (Pin_21)
- net ~{CSDEV2}: now also J?.11 (Pin_11), J?.11 (Pin_11)
- net ~{CSDEV3}: now also J?.9 (Pin_9), J?.9 (Pin_9)
- net ~{CSDEV4-5}: now also J?.19 (Pin_19), J?.19 (Pin_19)
- net ~{CSDEV4-7}: now also J?.25 (Pin_25), J?.25 (Pin_25)
- net ~{CSDEV4}: now also J?.7 (Pin_7), J?.7 (Pin_7)
- net ~{CSDEV5}: now also J?.5 (Pin_5), J?.5 (Pin_5)
- net ~{CSDEV6-7}: now also J?.17 (Pin_17), J?.17 (Pin_17)
- net ~{CSDEV6}: now also J?.3 (Pin_3), J?.3 (Pin_3)
- net ~{CSDEV7}: now also J?.1 (Pin_1), J?.1 (Pin_1)
- no-connect marks 1 -> 5
