File: kicad/Vega816/MemoryExpansionBus/pic_single.kicad_sch (KiCad schematic)
At the start: 46 parts, among them U2 74LS08, U65 74LS02, U68 74LS02, U69 74LS02, U72 74LS00, U73 74HC373, U74 74HC238, U75 74LS244, U76 74HC238, U85 74LS241, U86 74LS241, U87 74LS241, U88 74LS241

Commit message: expansion port hi ram
Other:
- note added: "Control Nybble format: 3210 TPPP High bit is Target (T) 0 = CPU A 1 = CPU B Low three bits (PPP) are priority, 0-7. Example 0x1110 0101 Low nybble is 0x0101: ~{IRQDEV0} goes to CPU 0 at Priority 0x101 (5). High nybble is 0x1110 ~{IRQDEV1} goes to CPU 1 at Priority 0x110 (6)."
- note removed: "Control Nybble format: 8421 TPPP High bit is Target (T) 0 = This channel's primary CPU 1 = Other channel's primary CPU Low three bits (PPP) are priority, 0-7. Example 0x1110 0101 ~{IRQDEV0} goes to CPU 1 at Priority 0x110 (6). ~{IRQDEV1} goes to CPU 0 at Priority 0x101 (5)."
- moved on the sheet: U2D, U72D, U73, U75

Commit message: new plots
Parts:
- removed D? (x32): 1N4148, Diode_THT:D_DO-35_SOD27_P7.62mm_Horizontal, symbol Diode:1N4148
- removed J?: IRQ Controller, symbol Connector_Generic:Conn_02x31_Odd_Even
- removed U2: 74LS08, symbol 74xx:74LS08
- removed U69: 74LS02, symbol 74xx:74LS02
- removed U72: 74LS00, symbol 74xx:74LS00
- removed U74, U76: 74HC238, symbol 74xx:74HC238
- removed U75: 74LS244, symbol 74xx:74LS244
- removed U85, U86, U87, U88: 74LS241, symbol 74xx:74LS241
- added D? (x32): 1N4148, Diode_THT:D_DO-35_SOD27_P7.62mm_Horizontal, symbol Diode:1N4148
- added J?: PIC, symbol Connector_Generic:Conn_02x13_Odd_Even
- added J? (x2): IRQ Bus Channel B, symbol Connector_Generic:Conn_02x08_Odd_Even
- added J? (x4): IRQ Bus Channel A, symbol Connector_Generic:Conn_02x08_Odd_Even
- added J?: IRQ Bus Channel C, symbol Connector_Generic:Conn_02x08_Odd_Even
- added J?: IRQ Bus Channel D, symbol Connector_Generic:Conn_02x08_Odd_Even
- added U? (x5): 74HC541, symbol Vega816:74HC541
- added U? (x2): 74ACH138, symbol Vega816:74ACH138
- renumbered U68 to U?, U65 to U?, U73 to U?
Connections:
- net ~{RS} is gone; now on net ~{CS}: U?.2, U?.6
- net D0: now also J?.25 (Pin_25), U?.11 (Y7)
- net D1: now also J?.23 (Pin_23), U?.12 (Y6)
- net D2: now also J?.21 (Pin_21), U?.13 (Y5)
- net D3: now also J?.19 (Pin_19), U?.14 (Y4)
- net D4: now also J?.17 (Pin_17), U?.15 (Y3)
- net D5: now also J?.15 (Pin_15), U?.16 (Y2)
- net D6: now also J?.13 (Pin_13), U?.17 (Y1)
- net D7: now also J?.11 (Pin_11), U?.18 (Y0)
- net GND: now also J?.10 (Pin_10), J?.10 (Pin_10), J?.10 (Pin_10), J?.10 (Pin_10), J?.10 (Pin_10), J?.10 (Pin_10), J?.10 (Pin_10), J?.10 (Pin_10), J?.10 (Pin_10), J?.12 (Pin_12), J?.12 (Pin_12), J?.12 (Pin_12), J?.12 (Pin_12), J?.12 (Pin_12), J?.12 (Pin_12), J?.12 (Pin_12), J?.12 (Pin_12), J?.12 (Pin_12), J?.14 (Pin_14), J?.14 (Pin_14), J?.14 (Pin_14), J?.14 (Pin_14), J?.14 (Pin_14), J?.14 (Pin_14), J?.14 (Pin_14), J?.14 (Pin_14), J?.14 (Pin_14), J?.16 (Pin_16), J?.16 (Pin_16), J?.16 (Pin_16), J?.16 (Pin_16), J?.16 (Pin_16), J?.16 (Pin_16), J?.16 (Pin_16), J?.16 (Pin_16), J?.16 (Pin_16), J?.18 (Pin_18), J?.2 (Pin_2), J?.2 (Pin_2), J?.2 (Pin_2), J?.2 (Pin_2), J?.2 (Pin_2), J?.2 (Pin_2), J?.2 (Pin_2), J?.2 (Pin_2), J?.2 (Pin_2), J?.20 (Pin_20), J?.22 (Pin_22), J?.24 (Pin_24), J?.26 (Pin_26), J?.3 (Pin_3), J?.4 (Pin_4), J?.4 (Pin_4), J?.4 (Pin_4), J?.4 (Pin_4), J?.4 (Pin_4), J?.4 (Pin_4), J?.4 (Pin_4), J?.4 (Pin_4), J?.4 (Pin_4), J?.6 (Pin_6), J?.6 (Pin_6), J?.6 (Pin_6), J?.6 (Pin_6), J?.6 (Pin_6), J?.6 (Pin_6), J?.6 (Pin_6), J?.6 (Pin_6), J?.6 (Pin_6), J?.8 (Pin_8), J?.8 (Pin_8), J?.8 (Pin_8), J?.8 (Pin_8), J?.8 (Pin_8), J?.8 (Pin_8), J?.8 (Pin_8), J?.8 (Pin_8), J?.8 (Pin_8), U?.10 (GND), U?.10 (GND), U?.10 (GND), U?.10 (GND), U?.10 (GND), U?.19 (G2), U?.19 (G2), U?.19 (G2), U?.19 (G2), U?.8 (GND), U?.8 (GND)
- net R~{W}: now also J?.9 (Pin_9)
- net VCC: now also J?.1 (Pin_1), U?.16 (VCC), U?.16 (VCC), U?.20 (VCC), U?.20 (VCC), U?.20 (VCC), U?.20 (VCC), U?.20 (VCC), U?.6 (E3), U?.6 (E3)
- net ~{CS}: now also J?.7 (Pin_7)
- net ~{LE}: now also U?.11 (LE)
- net ~{LRD}: now also U?.1 (G1)
- net at U?.19 (O7): now also U?.9 (A7)
- net at U?.12 (O4): now also U?.2 (A1), U?.6 (A4)
- net at U?.15 (O5): now also U?.3 (A2), U?.7 (A5)
- net at U?.16 (O6): now also U?.8 (A6)
- net at U?.2 (O0): now also U?.1 (A0), U?.2 (A0)
- net at U?.5 (O1): now also U?.2 (A1), U?.3 (A1)
- net at U?.6 (O2): now also U?.3 (A2), U?.4 (A2)
- net at U?.9 (O3): now also U?.1 (A0), U?.5 (A3)
- new net: D?.2 (A), U?.11 (Y7) (x4)
- new net: D?.2 (A), U?.12 (Y6) (x4)
- new net: D?.2 (A), U?.13 (Y5) (x4)
- new net: D?.2 (A), U?.14 (Y4) (x4)
- new net: D?.2 (A), U?.15 (Y3) (x4)
- new net: D?.2 (A), U?.16 (Y2) (x4)
- new net: D?.2 (A), U?.17 (Y1) (x4)
- new net: D?.2 (A), U?.18 (Y0) (x4)
- new net: U?.15 (O0), U?.2 (A0), U?.2 (A0), U?.2 (A0), U?.2 (A0)
- new net: U?.14 (O1), U?.3 (A1), U?.3 (A1), U?.3 (A1), U?.3 (A1)
- new net: U?.13 (O2), U?.4 (A2), U?.4 (A2), U?.4 (A2), U?.4 (A2)
- new net: U?.12 (O3), U?.5 (A3), U?.5 (A3), U?.5 (A3), U?.5 (A3)
- new net: U?.11 (O4), U?.6 (A4), U?.6 (A4), U?.6 (A4), U?.6 (A4)
- new net: U?.10 (O5), U?.7 (A5), U?.7 (A5), U?.7 (A5), U?.7 (A5)
- new net: U?.8 (A6), U?.8 (A6), U?.8 (A6), U?.8 (A6), U?.9 (O6)
- new net: U?.7 (O7), U?.9 (A7), U?.9 (A7), U?.9 (A7), U?.9 (A7)
- new net CPU 0: U?.1 (G1), U?.15 (O0)
- new net CPU 1: U?.1 (G1), U?.14 (O1)
- new net CPU 2: U?.1 (G1), U?.13 (O2)
- new net CPU 3: U?.1 (G1), U?.12 (O3)
- new net CPU 4: U?.11 (O4)
- new net CPU 5: U?.10 (O5)
- new net CPU 6: U?.9 (O6)
- new net CPU 7: U?.7 (O7)
- new net ~{IRQ0}: D?.1 (K), D?.1 (K), D?.1 (K), D?.1 (K), J?.15 (Pin_15), J?.15 (Pin_15), J?.15 (Pin_15), J?.15 (Pin_15), J?.15 (Pin_15), J?.15 (Pin_15), J?.15 (Pin_15), J?.15 (Pin_15)
- new net ~{IRQ1}: D?.1 (K), D?.1 (K), D?.1 (K), D?.1 (K), J?.13 (Pin_13), J?.13 (Pin_13), J?.13 (Pin_13), J?.13 (Pin_13), J?.13 (Pin_13), J?.13 (Pin_13), J?.13 (Pin_13), J?.13 (Pin_13)
- new net ~{IRQ2}: D?.1 (K), D?.1 (K), D?.1 (K), D?.1 (K), J?.11 (Pin_11), J?.11 (Pin_11), J?.11 (Pin_11), J?.11 (Pin_11), J?.11 (Pin_11), J?.11 (Pin_11), J?.11 (Pin_11), J?.11 (Pin_11)
- new net ~{IRQ3}: D?.1 (K), D?.1 (K), D?.1 (K), D?.1 (K), J?.9 (Pin_9), J?.9 (Pin_9), J?.9 (Pin_9), J?.9 (Pin_9), J?.9 (Pin_9), J?.9 (Pin_9), J?.9 (Pin_9), J?.9 (Pin_9)
- new net ~{IRQ4}: D?.1 (K), D?.1 (K), D?.1 (K), D?.1 (K), J?.7 (Pin_7), J?.7 (Pin_7), J?.7 (Pin_7), J?.7 (Pin_7), J?.7 (Pin_7), J?.7 (Pin_7), J?.7 (Pin_7), J?.7 (Pin_7)
- new net ~{IRQ5}: D?.1 (K), D?.1 (K), D?.1 (K), D?.1 (K), J?.5 (Pin_5), J?.5 (Pin_5), J?.5 (Pin_5), J?.5 (Pin_5), J?.5 (Pin_5), J?.5 (Pin_5), J?.5 (Pin_5), J?.5 (Pin_5)
- new net ~{IRQ6}: D?.1 (K), D?.1 (K), D?.1 (K), D?.1 (K), J?.3 (Pin_3), J?.3 (Pin_3), J?.3 (Pin_3), J?.3 (Pin_3), J?.3 (Pin_3), J?.3 (Pin_3), J?.3 (Pin_3), J?.3 (Pin_3)
- new net ~{IRQ7}: D?.1 (K), D?.1 (K), D?.1 (K), D?.1 (K), J?.1 (Pin_1), J?.1 (Pin_1), J?.1 (Pin_1), J?.1 (Pin_1), J?.1 (Pin_1), J?.1 (Pin_1), J?.1 (Pin_1), J?.1 (Pin_1)
- new net ~{IRQ}: J?.5 (Pin_5), U?.4 (E1), U?.4 (E1), U?.5 (E2), U?.5 (E2)
- no-connect marks 0 -> 4
Other:
- note added: "(CPU E-H, etc.)"
- note added: "A"
- note added: "B"
- note added: "C"
- note added: "Control Register"
- note added: "Control Register format: Bit #: 76543210 Value: XXTTTPPP"
- note added: "D"
- note added: "Priority"
- note added: "Priority PPP (lowest wins) 000 0 001 1 010 2 011 3 100 4 101 5 110 6 111 7"
- note added: "Programmable Interrupt Controller (8 Priority x 4 Target PIC)"
- note added: "Read Control Register"
- note added: "Target CPU"
- note added: "Target Select"
- note added: "Target TTT CPU 000 A 001 B 010 C 011 D 100 E 101 F 110 G 111 H"
- note removed: "2 IRQ sources, times: 2 programmable targets (CPU A or CPU B) 8 programmable priorities (0-7)"
- note removed: "Control Nybble format: 3210 TPPP High bit is Target (T) 0 = CPU A 1 = CPU B Low three bits (PPP) are priority, 0-7. Example 0x1110 0101 Low nybble is 0x0101: ~{IRQDEV0} goes to CPU 0 at Priority 0x101 (5). High nybble is 0x1110 ~{IRQDEV1} goes to CPU 1 at Priority 0x110 (6)."
- note removed: "Control Register IRQ Nybble ----- ---- ~{IRQDEV0} low ~{IRQDEV1} high"
- note removed: "Programmable Interrupt Controller (PIC)"
- moved on the sheet: U?

Commit message: wug
Other:
- note added: "Programmable Interrupt Controller (8 Priority x 4 Target CPUs)"
- note removed: "Programmable Interrupt Controller (8 Priority x 4 Target PIC)"
Changed lines of the file:
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@@
     (effects (font (size 5 5)) (justify left bottom))
   )
-  (text "Programmable Interrupt Controller \n(8 Priority x 4 Target PIC)\n"
+  (text "Programmable Interrupt Controller \n(8 Priority x 4 Target CPUs)\n"
     (at 21.59 53.34 0)
     (effects (font (size 10 10)) (justify left bottom))

Commit message: xcvx
Parts:
- added J? (x8): PIC, symbol Connector_Generic:Conn_02x13_Odd_Even
- added J? (x9): B, symbol Connector_Generic:Conn_02x08_Odd_Even
- added J? (x9): C, symbol Connector_Generic:Conn_02x08_Odd_Even
- added J? (x9): A, symbol Connector_Generic:Conn_02x08_Odd_Even
- added J?: $38 (8B), symbol Connector_Generic:Conn_02x18_Odd_Even
- added J? (x9): D, symbol Connector_Generic:Conn_02x08_Odd_Even
- added U?: 74ACH138, symbol Vega816:74ACH138
- J?: value IRQ Bus Channel A -> IRQ Bus Channel D
- J?: value IRQ Bus Channel A -> IRQ Bus Channel C
Connections:
- net D0: now also J?.25 (Pin_25), J?.25 (Pin_25), J?.25 (Pin_25), J?.25 (Pin_25), J?.25 (Pin_25), J?.25 (Pin_25), J?.25 (Pin_25), J?.25 (Pin_25), J?.35 (Pin_35)
- net D1: now also J?.23 (Pin_23), J?.23 (Pin_23), J?.23 (Pin_23), J?.23 (Pin_23), J?.23 (Pin_23), J?.23 (Pin_23), J?.23 (Pin_23), J?.23 (Pin_23), J?.33 (Pin_33)
- net D2: now also J?.21 (Pin_21), J?.21 (Pin_21), J?.21 (Pin_21), J?.21 (Pin_21), J?.21 (Pin_21), J?.21 (Pin_21), J?.21 (Pin_21), J?.21 (Pin_21), J?.31 (Pin_31)
- net D3: now also J?.19 (Pin_19), J?.19 (Pin_19), J?.19 (Pin_19), J?.19 (Pin_19), J?.19 (Pin_19), J?.19 (Pin_19), J?.19 (Pin_19), J?.19 (Pin_19), J?.29 (Pin_29)
- net D4: now also J?.17 (Pin_17), J?.17 (Pin_17), J?.17 (Pin_17), J?.17 (Pin_17), J?.17 (Pin_17), J?.17 (Pin_17), J?.17 (Pin_17), J?.17 (Pin_17), J?.27 (Pin_27)
- net D5: now also J?.15 (Pin_15), J?.15 (Pin_15), J?.15 (Pin_15), J?.15 (Pin_15), J?.15 (Pin_15), J?.15 (Pin_15), J?.15 (Pin_15), J?.15 (Pin_15), J?.25 (Pin_25)
- net D6: now also J?.13 (Pin_13), J?.13 (Pin_13), J?.13 (Pin_13), J?.13 (Pin_13), J?.13 (Pin_13), J?.13 (Pin_13), J?.13 (Pin_13), J?.13 (Pin_13), J?.23 (Pin_23)
- net D7: now also J?.11 (Pin_11), J?.11 (Pin_11), J?.11 (Pin_11), J?.11 (Pin_11), J?.11 (Pin_11), J?.11 (Pin_11), J?.11 (Pin_11), J?.11 (Pin_11), J?.21 (Pin_21)
- net GND: now also J?.10 (Pin_10), J?.10 (Pin_10), J?.10 (Pin_10), J?.10 (Pin_10), J?.10 (Pin_10), J?.10 (Pin_10), J?.10 (Pin_10), J?.10 (Pin_10), J?.10 (Pin_10), J?.10 (Pin_10), J?.10 (Pin_10), J?.10 (Pin_10), J?.10 (Pin_10), J?.10 (Pin_10), J?.10 (Pin_10), J?.10 (Pin_10), J?.10 (Pin_10), J?.10 (Pin_10), J?.10 (Pin_10), J?.10 (Pin_10), J?.10 (Pin_10), J?.10 (Pin_10), J?.10 (Pin_10), J?.10 (Pin_10), J?.10 (Pin_10), J?.10 (Pin_10), J?.10 (Pin_10), J?.10 (Pin_10), J?.10 (Pin_10), J?.10 (Pin_10), J?.10 (Pin_10), J?.10 (Pin_10), J?.10 (Pin_10), J?.10 (Pin_10), J?.10 (Pin_10), J?.10 (Pin_10), J?.10 (Pin_10), J?.10 (Pin_10), J?.10 (Pin_10), J?.10 (Pin_10), J?.10 (Pin_10), J?.10 (Pin_10), J?.10 (Pin_10), J?.10 (Pin_10), J?.10 (Pin_10), J?.12 (Pin_12), J?.12 (Pin_12), J?.12 (Pin_12), J?.12 (Pin_12), J?.12 (Pin_12), J?.12 (Pin_12), J?.12 (Pin_12), J?.12 (Pin_12), J?.12 (Pin_12), J?.12 (Pin_12), J?.12 (Pin_12), J?.12 (Pin_12), J?.12 (Pin_12), J?.12 (Pin_12), J?.12 (Pin_12), J?.12 (Pin_12), J?.12 (Pin_12), J?.12 (Pin_12), J?.12 (Pin_12), J?.12 (Pin_12), J?.12 (Pin_12), J?.12 (Pin_12), J?.12 (Pin_12), J?.12 (Pin_12), J?.12 (Pin_12), J?.12 (Pin_12), J?.12 (Pin_12), J?.12 (Pin_12), J?.12 (Pin_12), J?.12 (Pin_12), J?.12 (Pin_12), J?.12 (Pin_12), J?.12 (Pin_12), J?.12 (Pin_12), J?.12 (Pin_12), J?.12 (Pin_12), J?.12 (Pin_12), J?.12 (Pin_12), J?.12 (Pin_12), J?.12 (Pin_12), J?.12 (Pin_12), J?.12 (Pin_12), J?.12 (Pin_12), J?.12 (Pin_12), J?.12 (Pin_12), J?.14 (Pin_14), J?.14 (Pin_14), J?.14 (Pin_14), J?.14 (Pin_14), J?.14 (Pin_14), J?.14 (Pin_14), J?.14 (Pin_14), J?.14 (Pin_14), J?.14 (Pin_14), J?.14 (Pin_14), J?.14 (Pin_14), J?.14 (Pin_14), J?.14 (Pin_14), J?.14 (Pin_14), J?.14 (Pin_14), J?.14 (Pin_14), J?.14 (Pin_14), J?.14 (Pin_14), J?.14 (Pin_14), J?.14 (Pin_14), J?.14 (Pin_14), J?.14 (Pin_14), J?.14 (Pin_14), J?.14 (Pin_14), J?.14 (Pin_14), J?.14 (Pin_14), J?.14 (Pin_14), J?.14 (Pin_14), J?.14 (Pin_14), J?.14 (Pin_14), J?.14 (Pin_14), J?.14 (Pin_14), J?.14 (Pin_14), J?.14 (Pin_14), J?.14 (Pin_14), J?.14 (Pin_14), J?.14 (Pin_14), J?.14 (Pin_14), J?.14 (Pin_14), J?.14 (Pin_14), J?.14 (Pin_14), J?.14 (Pin_14), J?.14 (Pin_14), J?.14 (Pin_14), J?.14 (Pin_14), J?.16 (Pin_16), J?.16 (Pin_16), J?.16 (Pin_16), J?.16 (Pin_16), J?.16 (Pin_16), J?.16 (Pin_16), J?.16 (Pin_16), J?.16 (Pin_16), J?.16 (Pin_16), J?.16 (Pin_16), J?.16 (Pin_16), J?.16 (Pin_16), J?.16 (Pin_16), J?.16 (Pin_16), J?.16 (Pin_16), J?.16 (Pin_16), J?.16 (Pin_16), J?.16 (Pin_16), J?.16 (Pin_16), J?.16 (Pin_16), J?.16 (Pin_16), J?.16 (Pin_16), J?.16 (Pin_16), J?.16 (Pin_16), J?.16 (Pin_16), J?.16 (Pin_16), J?.16 (Pin_16), J?.16 (Pin_16), J?.16 (Pin_16), J?.16 (Pin_16), J?.16 (Pin_16), J?.16 (Pin_16), J?.16 (Pin_16), J?.16 (Pin_16), J?.16 (Pin_16), J?.16 (Pin_16), J?.16 (Pin_16), J?.16 (Pin_16), J?.16 (Pin_16), J?.16 (Pin_16), J?.16 (Pin_16), J?.16 (Pin_16), J?.16 (Pin_16), J?.16 (Pin_16), J?.16 (Pin_16), J?.18 (Pin_18), J?.18 (Pin_18), J?.18 (Pin_18), J?.18 (Pin_18), J?.18 (Pin_18), J?.18 (Pin_18), J?.18 (Pin_18), J?.18 (Pin_18), J?.18 (Pin_18), J?.2 (Pin_2), J?.2 (Pin_2), J?.2 (Pin_2), J?.2 (Pin_2), J?.2 (Pin_2), J?.2 (Pin_2), J?.2 (Pin_2), J?.2 (Pin_2), J?.2 (Pin_2), J?.2 (Pin_2), J?.2 (Pin_2), J?.2 (Pin_2), J?.2 (Pin_2), J?.2 (Pin_2), J?.2 (Pin_2), J?.2 (Pin_2), J?.2 (Pin_2), J?.2 (Pin_2), J?.2 (Pin_2), J?.2 (Pin_2), J?.2 (Pin_2), J?.2 (Pin_2), J?.2 (Pin_2), J?.2 (Pin_2), J?.2 (Pin_2), J?.2 (Pin_2), J?.2 (Pin_2), J?.2 (Pin_2), J?.2 (Pin_2), J?.2 (Pin_2), J?.2 (Pin_2), J?.2 (Pin_2), J?.2 (Pin_2), J?.2 (Pin_2), J?.2 (Pin_2), J?.2 (Pin_2), J?.2 (Pin_2), J?.2 (Pin_2), J?.2 (Pin_2), J?.2 (Pin_2), J?.2 (Pin_2), J?.2 (Pin_2), J?.2 (Pin_2), J?.2 (Pin_2), J?.2 (Pin_2), J?.20 (Pin_20), J?.20 (Pin_20), J?.20 (Pin_20), J?.20 (Pin_20), J?.20 (Pin_20), J?.20 (Pin_20), J?.20 (Pin_20), J?.20 (Pin_20), J?.20 (Pin_20), J?.22 (Pin_22), J?.22 (Pin_22), J?.22 (Pin_22), J?.22 (Pin_22), J?.22 (Pin_22), J?.22 (Pin_22), J?.22 (Pin_22), J?.22 (Pin_22), J?.22 (Pin_22), J?.24 (Pin_24), J?.24 (Pin_24), J?.24 (Pin_24), J?.24 (Pin_24), J?.24 (Pin_24), J?.24 (Pin_24), J?.24 (Pin_24), J?.24 (Pin_24), J?.24 (Pin_24), J?.26 (Pin_26), J?.26 (Pin_26), J?.26 (Pin_26), J?.26 (Pin_26), J?.26 (Pin_26), J?.26 (Pin_26), J?.26 (Pin_26), J?.26 (Pin_26), J?.26 (Pin_26), J?.28 (Pin_28), J?.3 (Pin_3), J?.3 (Pin_3), J?.3 (Pin_3), J?.3 (Pin_3), J?.3 (Pin_3), J?.3 (Pin_3), J?.3 (Pin_3), J?.3 (Pin_3), J?.30 (Pin_30), J?.32 (Pin_32), J?.34 (Pin_34), J?.36 (Pin_36), J?.4 (Pin_4), J?.4 (Pin_4), J?.4 (Pin_4), J?.4 (Pin_4), J?.4 (Pin_4), J?.4 (Pin_4), J?.4 (Pin_4), J?.4 (Pin_4), J?.4 (Pin_4), J?.4 (Pin_4), J?.4 (Pin_4), J?.4 (Pin_4), J?.4 (Pin_4), J?.4 (Pin_4), J?.4 (Pin_4), J?.4 (Pin_4), J?.4 (Pin_4), J?.4 (Pin_4), J?.4 (Pin_4), J?.4 (Pin_4), J?.4 (Pin_4), J?.4 (Pin_4), J?.4 (Pin_4), J?.4 (Pin_4), J?.4 (Pin_4), J?.4 (Pin_4), J?.4 (Pin_4), J?.4 (Pin_4), J?.4 (Pin_4), J?.4 (Pin_4), J?.4 (Pin_4), J?.4 (Pin_4), J?.4 (Pin_4), J?.4 (Pin_4), J?.4 (Pin_4), J?.4 (Pin_4), J?.4 (Pin_4), J?.4 (Pin_4), J?.4 (Pin_4), J?.4 (Pin_4), J?.4 (Pin_4), J?.4 (Pin_4), J?.4 (Pin_4), J?.4 (Pin_4), J?.4 (Pin_4), J?.6 (Pin_6), J?.6 (Pin_6), J?.6 (Pin_6), J?.6 (Pin_6), J?.6 (Pin_6), J?.6 (Pin_6), J?.6 (Pin_6), J?.6 (Pin_6), J?.6 (Pin_6), J?.6 (Pin_6), J?.6 (Pin_6), J?.6 (Pin_6), J?.6 (Pin_6), J?.6 (Pin_6), J?.6 (Pin_6), J?.6 (Pin_6), J?.6 (Pin_6), J?.6 (Pin_6), J?.6 (Pin_6), J?.6 (Pin_6), J?.6 (Pin_6), J?.6 (Pin_6), J?.6 (Pin_6), J?.6 (Pin_6), J?.6 (Pin_6), J?.6 (Pin_6), J?.6 (Pin_6), J?.6 (Pin_6), J?.6 (Pin_6), J?.6 (Pin_6), J?.6 (Pin_6), J?.6 (Pin_6), J?.6 (Pin_6), J?.6 (Pin_6), J?.6 (Pin_6), J?.6 (Pin_6), J?.6 (Pin_6), J?.6 (Pin_6), J?.6 (Pin_6), J?.6 (Pin_6), J?.6 (Pin_6), J?.6 (Pin_6), J?.6 (Pin_6), J?.6 (Pin_6), J?.6 (Pin_6), J?.7 (Pin_7), J?.8 (Pin_8), J?.8 (Pin_8), J?.8 (Pin_8), J?.8 (Pin_8), J?.8 (Pin_8), J?.8 (Pin_8), J?.8 (Pin_8), J?.8 (Pin_8), J?.8 (Pin_8), J?.8 (Pin_8), J?.8 (Pin_8), J?.8 (Pin_8), J?.8 (Pin_8), J?.8 (Pin_8), J?.8 (Pin_8), J?.8 (Pin_8), J?.8 (Pin_8), J?.8 (Pin_8), J?.8 (Pin_8), J?.8 (Pin_8), J?.8 (Pin_8), J?.8 (Pin_8), J?.8 (Pin_8), J?.8 (Pin_8), J?.8 (Pin_8), J?.8 (Pin_8)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
- net R~{W}: now also J?.13 (Pin_13), J?.9 (Pin_9), J?.9 (Pin_9), J?.9 (Pin_9), J?.9 (Pin_9), J?.9 (Pin_9), J?.9 (Pin_9), J?.9 (Pin_9), J?.9 (Pin_9)
- net VCC: now also J?.1 (Pin_1), J?.1 (Pin_1), J?.1 (Pin_1), J?.1 (Pin_1), J?.1 (Pin_1), J?.1 (Pin_1), J?.1 (Pin_1), J?.1 (Pin_1), J?.5 (Pin_5), U?.16 (VCC), U?.6 (E3)
- net ~{CS}: now also J?.3 (Pin_3), J?.7 (Pin_7), J?.7 (Pin_7), J?.7 (Pin_7), J?.7 (Pin_7), J?.7 (Pin_7), J?.7 (Pin_7), J?.7 (Pin_7), J?.7 (Pin_7), U?.10 (O5), U?.11 (O4), U?.12 (O3), U?.13 (O2), U?.14 (O1), U?.15 (O0), U?.4 (E1), U?.5 (E2), U?.7 (O7), U?.9 (O6)
- net ~{IRQ0}: now also J?.15 (Pin_15), J?.15 (Pin_15), J?.15 (Pin_15), J?.15 (Pin_15), J?.15 (Pin_15), J?.15 (Pin_15), J?.15 (Pin_15), J?.15 (Pin_15), J?.15 (Pin_15), J?.15 (Pin_15), J?.15 (Pin_15), J?.15 (Pin_15), J?.15 (Pin_15), J?.15 (Pin_15), J?.15 (Pin_15), J?.15 (Pin_15), J?.15 (Pin_15), J?.15 (Pin_15), J?.15 (Pin_15), J?.15 (Pin_15), J?.15 (Pin_15), J?.15 (Pin_15), J?.15 (Pin_15), J?.15 (Pin_15), J?.15 (Pin_15), J?.15 (Pin_15), J?.15 (Pin_15), J?.15 (Pin_15), J?.15 (Pin_15), J?.15 (Pin_15), J?.15 (Pin_15), J?.15 (Pin_15), J?.15 (Pin_15), J?.15 (Pin_15), J?.15 (Pin_15), J?.15 (Pin_15)
- net ~{IRQ1}: now also J?.13 (Pin_13), J?.13 (Pin_13), J?.13 (Pin_13), J?.13 (Pin_13), J?.13 (Pin_13), J?.13 (Pin_13), J?.13 (Pin_13), J?.13 (Pin_13), J?.13 (Pin_13), J?.13 (Pin_13), J?.13 (Pin_13), J?.13 (Pin_13), J?.13 (Pin_13), J?.13 (Pin_13), J?.13 (Pin_13), J?.13 (Pin_13), J?.13 (Pin_13), J?.13 (Pin_13), J?.13 (Pin_13), J?.13 (Pin_13), J?.13 (Pin_13), J?.13 (Pin_13), J?.13 (Pin_13), J?.13 (Pin_13), J?.13 (Pin_13), J?.13 (Pin_13), J?.13 (Pin_13), J?.13 (Pin_13), J?.13 (Pin_13), J?.13 (Pin_13), J?.13 (Pin_13), J?.13 (Pin_13), J?.13 (Pin_13), J?.13 (Pin_13), J?.13 (Pin_13), J?.13 (Pin_13)
- net ~{IRQ2}: now also J?.11 (Pin_11), J?.11 (Pin_11), J?.11 (Pin_11), J?.11 (Pin_11), J?.11 (Pin_11), J?.11 (Pin_11), J?.11 (Pin_11), J?.11 (Pin_11), J?.11 (Pin_11), J?.11 (Pin_11), J?.11 (Pin_11), J?.11 (Pin_11), J?.11 (Pin_11), J?.11 (Pin_11), J?.11 (Pin_11), J?.11 (Pin_11), J?.11 (Pin_11), J?.11 (Pin_11), J?.11 (Pin_11), J?.11 (Pin_11), J?.11 (Pin_11), J?.11 (Pin_11), J?.11 (Pin_11), J?.11 (Pin_11), J?.11 (Pin_11), J?.11 (Pin_11), J?.11 (Pin_11), J?.11 (Pin_11), J?.11 (Pin_11), J?.11 (Pin_11), J?.11 (Pin_11), J?.11 (Pin_11), J?.11 (Pin_11), J?.11 (Pin_11), J?.11 (Pin_11), J?.11 (Pin_11)
- net ~{IRQ3}: now also J?.9 (Pin_9), J?.9 (Pin_9), J?.9 (Pin_9), J?.9 (Pin_9), J?.9 (Pin_9), J?.9 (Pin_9), J?.9 (Pin_9), J?.9 (Pin_9), J?.9 (Pin_9), J?.9 (Pin_9), J?.9 (Pin_9), J?.9 (Pin_9), J?.9 (Pin_9), J?.9 (Pin_9), J?.9 (Pin_9), J?.9 (Pin_9), J?.9 (Pin_9), J?.9 (Pin_9), J?.9 (Pin_9), J?.9 (Pin_9), J?.9 (Pin_9), J?.9 (Pin_9), J?.9 (Pin_9), J?.9 (Pin_9), J?.9 (Pin_9), J?.9 (Pin_9), J?.9 (Pin_9), J?.9 (Pin_9), J?.9 (Pin_9), J?.9 (Pin_9), J?.9 (Pin_9), J?.9 (Pin_9), J?.9 (Pin_9), J?.9 (Pin_9), J?.9 (Pin_9), J?.9 (Pin_9)
- net ~{IRQ4}: now also J?.7 (Pin_7), J?.7 (Pin_7), J?.7 (Pin_7), J?.7 (Pin_7), J?.7 (Pin_7), J?.7 (Pin_7), J?.7 (Pin_7), J?.7 (Pin_7), J?.7 (Pin_7), J?.7 (Pin_7), J?.7 (Pin_7), J?.7 (Pin_7), J?.7 (Pin_7), J?.7 (Pin_7), J?.7 (Pin_7), J?.7 (Pin_7), J?.7 (Pin_7), J?.7 (Pin_7), J?.7 (Pin_7), J?.7 (Pin_7), J?.7 (Pin_7), J?.7 (Pin_7), J?.7 (Pin_7), J?.7 (Pin_7), J?.7 (Pin_7), J?.7 (Pin_7), J?.7 (Pin_7), J?.7 (Pin_7), J?.7 (Pin_7), J?.7 (Pin_7), J?.7 (Pin_7), J?.7 (Pin_7), J?.7 (Pin_7), J?.7 (Pin_7), J?.7 (Pin_7), J?.7 (Pin_7)
- net ~{IRQ5}: now also J?.5 (Pin_5), J?.5 (Pin_5), J?.5 (Pin_5), J?.5 (Pin_5), J?.5 (Pin_5), J?.5 (Pin_5), J?.5 (Pin_5), J?.5 (Pin_5), J?.5 (Pin_5), J?.5 (Pin_5), J?.5 (Pin_5), J?.5 (Pin_5), J?.5 (Pin_5), J?.5 (Pin_5), J?.5 (Pin_5), J?.5 (Pin_5), J?.5 (Pin_5), J?.5 (Pin_5), J?.5 (Pin_5), J?.5 (Pin_5), J?.5 (Pin_5), J?.5 (Pin_5), J?.5 (Pin_5), J?.5 (Pin_5), J?.5 (Pin_5), J?.5 (Pin_5), J?.5 (Pin_5), J?.5 (Pin_5), J?.5 (Pin_5), J?.5 (Pin_5), J?.5 (Pin_5), J?.5 (Pin_5), J?.5 (Pin_5), J?.5 (Pin_5), J?.5 (Pin_5), J?.5 (Pin_5)
- net ~{IRQ6}: now also J?.3 (Pin_3), J?.3 (Pin_3), J?.3 (Pin_3), J?.3 (Pin_3), J?.3 (Pin_3), J?.3 (Pin_3), J?.3 (Pin_3), J?.3 (Pin_3), J?.3 (Pin_3), J?.3 (Pin_3), J?.3 (Pin_3), J?.3 (Pin_3), J?.3 (Pin_3), J?.3 (Pin_3), J?.3 (Pin_3), J?.3 (Pin_3), J?.3 (Pin_3), J?.3 (Pin_3), J?.3 (Pin_3), J?.3 (Pin_3), J?.3 (Pin_3), J?.3 (Pin_3), J?.3 (Pin_3), J?.3 (Pin_3), J?.3 (Pin_3), J?.3 (Pin_3), J?.3 (Pin_3), J?.3 (Pin_3), J?.3 (Pin_3), J?.3 (Pin_3), J?.3 (Pin_3), J?.3 (Pin_3), J?.3 (Pin_3), J?.3 (Pin_3), J?.3 (Pin_3), J?.3 (Pin_3)
- net ~{IRQ7}: now also J?.1 (Pin_1), J?.1 (Pin_1), J?.1 (Pin_1), J?.1 (Pin_1), J?.1 (Pin_1), J?.1 (Pin_1), J?.1 (Pin_1), J?.1 (Pin_1), J?.1 (Pin_1), J?.1 (Pin_1), J?.1 (Pin_1), J?.1 (Pin_1), J?.1 (Pin_1), J?.1 (Pin_1), J?.1 (Pin_1), J?.1 (Pin_1), J?.1 (Pin_1), J?.1 (Pin_1), J?.1 (Pin_1), J?.1 (Pin_1), J?.1 (Pin_1), J?.1 (Pin_1), J?.1 (Pin_1), J?.1 (Pin_1), J?.1 (Pin_1), J?.1 (Pin_1), J?.1 (Pin_1), J?.1 (Pin_1), J?.1 (Pin_1), J?.1 (Pin_1), J?.1 (Pin_1), J?.1 (Pin_1), J?.1 (Pin_1), J?.1 (Pin_1), J?.1 (Pin_1), J?.1 (Pin_1)
- net ~{IRQ}: now also J?.1 (Pin_1), J?.5 (Pin_5), J?.5 (Pin_5), J?.5 (Pin_5), J?.5 (Pin_5), J?.5 (Pin_5), J?.5 (Pin_5), J?.5 (Pin_5), J?.5 (Pin_5)
- net at U?.5 (A3), U?.9 (O3): no longer U?.1 (A0)
- net at U?.12 (O4), U?.6 (A4): now also U?.1 (A0); no longer U?.2 (A1)
- net at U?.15 (O5), U?.7 (A5): now also U?.2 (A1); no longer U?.3 (A2)
- net at U?.16 (O6), U?.8 (A6): now also U?.3 (A2)
- new net A0: J?.19 (Pin_19), U?.1 (A0)
- new net A1: J?.17 (Pin_17), U?.2 (A1)
- new net A2: J?.15 (Pin_15), U?.3 (A2)
- new net CLK: J?.11 (Pin_11)
- new net ~{RST}: J?.9 (Pin_9)
Other:
- note added: "Control Register format: Bit #: 76543210 Value: XTTTXPPP"
- note removed: "Control Register format: Bit #: 76543210 Value: XXTTTPPP"
- moved on the sheet: D?, J?, U?

Commit message: Big
Parts:
- removed J? (x9): PIC, symbol Connector_Generic:Conn_02x13_Odd_Even
- removed J? (x9): B, symbol Connector_Generic:Conn_02x08_Odd_Even
- removed J? (x9): C, symbol Connector_Generic:Conn_02x08_Odd_Even
- removed J? (x9): A, symbol Connector_Generic:Conn_02x08_Odd_Even
- removed J?: $38 (8B), symbol Connector_Generic:Conn_02x18_Odd_Even
- removed J? (x9): D, symbol Connector_Generic:Conn_02x08_Odd_Even
- removed U? (x3): 74LS02, symbol 74xx:74LS02
- removed U?: 74HC541, symbol Vega816:74HC541
- removed U?: 74HC373, symbol 74xx:74HC373
- removed U?: 74ACH138, symbol Vega816:74ACH138
- added J28: Sysctl Reg, Connector_PinHeader_2.54mm:PinHeader_2x08_P2.54mm_Vertical, symbol Vega816:Conn_02x08_Odd_Even
Connections:
- net GND: now also J28.10 (Pin_10), J28.12 (Pin_12), J28.14 (Pin_14), J28.16 (Pin_16), J28.2 (Pin_2), J28.4 (Pin_4), J28.6 (Pin_6), J28.8 (Pin_8)
- net at U?.1 (A0): now also J28.7 (Pin_7)
- net at U?.2 (A1): now also J28.5 (Pin_5)
- net at U?.3 (A2): now also J28.3 (Pin_3)
- net at U?.1 (A0): now also J28.15 (Pin_15)
- net at U?.2 (A1): now also J28.13 (Pin_13)
- net at U?.3 (A2): now also J28.11 (Pin_11)
- net ~{IRQ} renamed ~{IRQ_IN}
- no-connect marks 4 -> 6
Other:
- note added: "Target"
- note removed: "(CPU E-H, etc.)"
- note removed: "Control Register"
- note removed: "Latch Enable"
- note removed: "Latch Output Enable"
- note removed: "Read Control Register"
- note removed: "Target Select"
- moved on the sheet: D?, J?, U?
