File: kicad/Vega816/MemoryExpansionBus/C64_IO_Decoder.kicad_sch (KiCad schematic)
At the start: 37 parts, among them J0A1 Conn_02x40_Odd_Even, J0B1 CPU, J43 VPA/VDA

Commit message: push
Parts:
- removed J?: DEV0-1 PIC, symbol Connector_Generic:Conn_02x31_Odd_Even
- removed J? (x2): DEV2-3 PIC, symbol Connector_Generic:Conn_02x31_Odd_Even
- removed J? (x2): 16B, symbol Connector_Generic:Conn_02x20_Odd_Even
- removed J?: IRQ_OUT, symbol Connector_Generic:Conn_02x16_Odd_Even
- removed U?: 74HC00, symbol 74xx:74HC00
- removed U? (x2): 74ACH138, symbol Vega816:74ACH138
Connections:
- net ~{WR} is gone; now on net R~{W}: J0A1.39 (Pin_39)
- net VCC: no longer J0A1.19 (Pin_19), J0A1.41 (Pin_41), J?.15 (Pin_15), J?.17 (Pin_17), J?.20 (Pin_20), J?.3 (Pin_3), J?.7 (Pin_7), J?.9 (Pin_9), U?.10 (O5), U?.11 (O4), U?.20 (VCC), U?.21 (~{IRQ}), U?.21 (~{IRQ}), U?.23 (~{CS2}), U?.23 (~{CS2}), U?.24 (CS1), U?.3, U?.3, U?.4 (E1), U?.4 (E1)
- new net: U?.20 (VCC), U?.24 (CS1)
- new net ~{$DC00-$DCFF}: J?.17 (Pin_17), J?.9 (Pin_9), U?.10 (O5), U?.11 (O4), U?.23 (~{CS2}), U?.23 (~{CS2}), U?.3, U?.3
- new net ~{BANK0}: J0A1.41 (Pin_41), U?.4 (E1), U?.4 (E1)
- new net ~{IRQ}: J0A1.19 (Pin_19), J?.15 (Pin_15), J?.20 (Pin_20), J?.7 (Pin_7)
- new net ~{KBD_IRQ}: J?.3 (Pin_3)
Other:
- note added: "$D000-$D1FF VIC-II $D400-$D7FF SID $D800-$DBFF Color RAM $DC00-$DCFF CIA#1; inputs (keyboard, joystick, mouse), datasette, IRQ control $DD00-$DDFF CIA#2; serial bus, RS232, NMI control $DE00-$DEFF I/O Area #1 (SID #2) $DF00-$DFFF I/O Area #2"
- note added: "VIA #1"
- note added: "VIA #2"
- note added: "~{WR}"
- note removed: "$D000-$D1FF VIC-II; video display $D200 PIC #1 $D201 PIC #2 $D400-$D7FF SID; audio $D800-$DBFF Color RAM $DC00-$DCFF CIA#1; inputs (keyboard, joystick, mouse), datasette, IRQ control $DD00-$DDFF CIA#2; serial bus, RS232, NMI control $DE00-$DEFF I/O Area #1 $DF00-$DFFF I/O Area #2"
- note removed: "VIA (CIA) #2"
- moved on the sheet: J?, U?

Commit message: dfsg
Parts:
- removed J0A1: Conn_02x40_Odd_Even, Connector_PinHeader_2.54mm:PinHeader_2x40_P2.54mm_Vertical, symbol Connector_Generic:Conn_02x40_Odd_Even
- removed J0B1: CPU, Connector_PinHeader_2.54mm:PinHeader_2x18_P2.54mm_Vertical, symbol Connector_Generic:Conn_02x18_Odd_Even
- removed J43: VPA/VDA, symbol Connector:Conn_01x02_Male
- removed J?: Joystick 2, symbol Connector:DB9_Male
- removed J?: C64 KBD, symbol Connector_Generic:Conn_01x20
- removed J?: 6510 P0-P5, symbol Connector_Generic:Conn_02x08_Counter_Clockwise
- removed J?: C64 Expansion Port, symbol Connector_Generic:Conn_02x40_Odd_Even
- removed J?: $00 (64 B), symbol Connector_Generic:Conn_02x28_Odd_Even
- removed J?: POTXY, symbol Connector_Generic:Conn_02x04_Odd_Even
- removed J?: Joystick 1, symbol Connector:DB9_Male
- removed J?: VIA Port, symbol Connector_Generic:Conn_02x22_Odd_Even
- removed J?: $80 (32B), symbol Connector_Generic:Conn_02x24_Odd_Even
- removed J?: C64_CASSETTE, symbol Vega816:C64_CASSETTE
- removed U?: CD4066B, symbol Vega816:CD4066B
- removed U? (x3): CD4082BE, symbol Vega816:CD4082BE
- removed U? (x2): 74HC08, symbol Vega816:74HC08
- removed U? (x4): 74ACH138, symbol Vega816:74ACH138
- removed U? (x2): W65C22SxP, Package_DIP:DIP-40_W15.24mm_Socket, symbol Vega816:W65C22SxP
- removed U?: 4082, symbol 4xxx_IEEE:4082
- removed U?: 82S100, Package_DIP:DIP-28_W15.24mm, symbol Vega816:82S100
- removed U?: 74HC00, symbol 74xx:74HC00
Connections:
- no-connect marks 14 -> 0
Other:
- note removed: "$D000-$D1FF VIC-II $D400-$D7FF SID $D800-$DBFF Color RAM $DC00-$DCFF CIA#1; inputs (keyboard, joystick, mouse), datasette, IRQ control $DD00-$DDFF CIA#2; serial bus, RS232, NMI control $DE00-$DEFF I/O Area #1 (SID #2) $DF00-$DFFF I/O Area #2"
- note removed: "Dual SID"
- note removed: "SID 1"
- note removed: "SID 2"
- note removed: "VIA #1"
- note removed: "VIA #2"
- note removed: "VIC-II"
- note removed: "~{C64_CIA_1}"
- note removed: "~{C64_CIA_2}"
- note removed: "~{C64_IO1}"
- note removed: "~{C64_IO2}"
- note removed: "~{WR}"
