File: kicad/Vega816/DMA/CPU Buffer/CPU Buffer.kicad_sch (KiCad schematic)
At the start: 21 parts, among them J10 VPA/VDA, J11 Conn_02x40_Odd_Even, J12 DMA, J3 VPA/VDA, J4 Conn_02x40_Odd_Even, J5 AUX, J6 VPA/VDA, J7 Conn_02x40_Odd_Even, J8 CPU, J9 DMA CTRL, U16 74HC541, U17 74AHCT245, U18 74HC541, U19 74HC541, U20 74HC541, U21 74HC541, U22 74HC541, U23 74HC541

Commit message: Update CPU Buffer
Other:
- note added: "Stackable CPU Buffer Module for Kohlbecker W65C816 Breakout Board (1 per CPU per DMA channel)"
- note removed: "CPU Buffer Module (Stackable, 1 per CPU per DMA channel)"
- title: (none) -> Stackable CPU Buffer Module for Kohlbecker W65C816 Breakout

Commit message: images
Parts:
- added R?: 1 K, symbol Device:R
Connections:
- net GND: now also R?.2
- net ~{DMA}: now also R?.1
Other:
- note added: "Stackable CPU Buffer Module for Kohlbecker W65C816 Breakout Board"
- note removed: "Stackable CPU Buffer Module for Kohlbecker W65C816 Breakout Board (1 per CPU per DMA channel)"
- moved on the sheet: J9
Changed lines of the file:
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@@
   (junction (at 120.65 208.28) (diameter 0) (color 0 0 0 0)
   )
+  (junction (at 135.89 355.6) (diameter 0) (color 0 0 0 0)
+  )
   (junction (at 473.6271 162.56) (diameter 0) (color 0 0 0 0)
   )
@@
   (junction (at 82.55 254) (diameter 0) (color 0 0 0 0)
   )
-  (junction (at 161.29 327.66) (diameter 0) (color 0 0 0 0)
-  )
   (junction (at 422.91 160.02) (diameter 0) (color 0 0 0 0)
   )
@@
   (junction (at 435.61 163.83) (diameter 0) (color 0 0 0 0)
   )
+  (junction (at 147.32 347.98) (diameter 0) (color 0 0 0 0)
+  )
   (junction (at 135.89 259.08) (diameter 0) (color 0 0 0 0)
   )
@@
   (junction (at 120.65 254) (diameter 0) (color 0 0 0 0)
   )
-  (junction (at 147.32 299.72) (diameter 0) (color 0 0 0 0)
-  )
   (junction (at 82.55 220.98) (diameter 0) (color 0 0 0 0)
   )
@@
   (junction (at 120.65 276.86) (diameter 0) (color 0 0 0 0)
   )
+  (junction (at 143.51 347.98) (diameter 0) (color 0 0 0 0)
+  )
   (junction (at 135.89 185.42) (diameter 0) (color 0 0 0 0)
   )
@@
   (junction (at 322.58 118.11) (diameter 0) (color 0 0 0 0)
   )
+  (junction (at 161.29 347.98) (diameter 0) (color 0 0 0 0)
+  )
   (junction (at 120.65 165.1) (diameter 0) (color 0 0 0 0)
   )
@@
     (stroke (width 0) (type default) (color 0 0 0 0))
   )
-  (wire (pts (xy 161.29 327.66) (xy 161.29 322.58))
+  (wire (pts (xy 161.29 322.58) (xy 161.29 347.98))
     (stroke (width 0) (type default) (color 0 0 0 0))
   )
@@
     (stroke (width 0) (type default) (color 0 0 0 0))
   )
+  (wire (pts (xy 143.51 347.98) (xy 147.32 347.98))
+    (stroke (width 0) (type default) (color 0 0 0 0))
+  )
   (wire (pts (xy 173.99 322.58) (xy 173.99 340.36))
     (stroke (width 0) (type default) (color 0 0 0 0))
@@
     (stroke (width 0) (type default) (color 0 0 0 0))
   )
+  (wire (pts (xy 147.32 80.01) (xy 147.32 347.98))
+    (stroke (width 0) (type default) (color 0 0 0 0))
+  )
   (wire (pts (xy 135.89 173.99) (xy 118.11 173.99))
     (stroke (width 0) (type default) (color 0 0 0 0))
@@
     (stroke (width 0) (type default) (color 0 0 0 0))
   )
-  (wire (pts (xy 135.89 302.26) (xy 135.89 308.61))
+  (wire (pts (xy 135.89 350.52) (xy 135.89 355.6))
     (stroke (width 0) (type default) (color 0 0 0 0))
   )
@@
     (stroke (width 0) (type default) (color 0 0 0 0))
   )
+  (wire (pts (xy 135.89 355.6) (xy 135.89 356.87))
+    (stroke (width 0) (type default) (color 0 0 0 0))
+  )
   (wire (pts (xy 422.91 289.56) (xy 422.91 292.1))
     (stroke (width 0) (type default) (color 0 0 0 0))
@@
     (stroke (width 0) (type default) (color 0 0 0 0))
   )
-  (wire (pts (xy 147.32 80.01) (xy 147.32 299.72))
-    (stroke (width 0) (type default) (color 0 0 0 0))
-  )
   (wire (pts (xy 135.89 196.85) (xy 118.11 196.85))
     (stroke (width 0) (type default) (color 0 0 0 0))
@@
     (stroke (width 0) (type default) (color 0 0 0 0))
   )
-  (wire (pts (xy 147.32 327.66) (xy 161.29 327.66))
+  (wire (pts (xy 147.32 347.98) (xy 161.29 347.98))
     (stroke (width 0) (type default) (color 0 0 0 0))
   )
@@
     (stroke (width 0) (type default) (color 0 0 0 0))
   )
-  (wire (pts (xy 147.32 299.72) (xy 147.32 327.66))
-    (stroke (width 0) (type default) (color 0 0 0 0))
-  )
   (wire (pts (xy 226.06 297.18) (xy 227.33 297.18))
     (stroke (width 0) (type default) (color 0 0 0 0))
@@
     (stroke (width 0) (type default) (color 0 0 0 0))
   )
-  (wire (pts (xy 135.89 299.72) (xy 147.32 299.72))
+  (wire (pts (xy 135.89 347.98) (xy 143.51 347.98))
     (stroke (width 0) (type default) (color 0 0 0 0))
   )
@@
     (stroke (width 0) (type default) (color 0 0 0 0))
   )
+  (wire (pts (xy 135.89 355.6) (xy 143.51 355.6))
+    (stroke (width 0) (type default) (color 0 0 0 0))
+  )
   (wire (pts (xy 118.11 196.85) (xy 118.11 198.12))
     (stroke (width 0) (type default) (color 0 0 0 0))
@@
     (stroke (width 0) (type default) (color 0 0 0 0))
   )
-  (wire (pts (xy 161.29 347.98) (xy 161.29 327.66))
-    (stroke (width 0) (type default) (color 0 0 0 0))
-  )
   (wire (pts (xy 165.1 105.41) (xy 165.1 87.63))
     (stroke (width 0) (type default) (color 0 0 0 0))
@@
     (stroke (width 0) (type default) (color 0 0 0 0))
   )
-  (text "Stackable CPU Buffer Module for Kohlbecker W65C816 Breakout Board\n\n(1 per CPU per DMA channel)"
-    (at 23.495 75.565 0)
+  (text "Stackable CPU Buffer Module \nfor Kohlbecker W65C816 Breakout Board"
+    (at 28.575 62.865 0)
     (effects (font (size 10 10)) (justify left bottom))
   )
@@
     (effects (font (size 1.27 1.27)) (justify left bottom))
   )
-  (label "~{DMA}" (at 138.43 299.72 0)
+  (label "~{DMA}" (at 135.89 347.98 0)
     (effects (font (size 1.27 1.27)) (justify left bottom))
   )
@@
     (pin "9")
   )
-  (symbol (lib_id "power:GND") (at 135.89 308.61 0) (unit 1)
+  (symbol (lib_id "power:GND") (at 135.89 356.87 0) (unit 1)
     (in_bom yes) (on_board yes)
-    (property "Reference" "#PWR?" (id 0) (at 135.89 314.96 0)
+    (property "Reference" "#PWR?" (id 0) (at 135.89 363.22 0)
       (effects (font (size 1.27 1.27)) hide)
     )
-    (property "Value" "GND" (id 1) (at 135.89 312.42 0))
-    (property "Footprint" "" (id 2) (at 135.89 308.61 0)
+    (property "Value" "GND" (id 1) (at 135.89 360.68 0))
+    (property "Footprint" "" (id 2) (at 135.89 356.87 0)
       (effects (font (size 1.27 1.27)) hide)
     )
-    (property "Datasheet" "" (id 3) (at 135.89 308.61 0)
+    (property "Datasheet" "" (id 3) (at 135.89 356.87 0)
       (effects (font (size 1.27 1.27)) hide)
     )
@@
     (pin "1")
   )
+  (symbol (lib_id "Device:R") (at 143.51 351.79 0) (unit 1)
+    (in_bom yes) (on_board yes)
+    (property "Reference" "R?" (id 0) (at 139.7 349.2499 0)
+      (effects (font (size 1.27 1.27)) (justify left))
+    )
+    (property "Value" "1 K" (id 1) (at 143.51 354.3299 90)
+      (effects (font (size 1.27 1.27)) (justify left))
+    )
+    (property "Footprint" "" (id 2) (at 141.732 351.79 90)
+      (effects (font (size 1.27 1.27)) hide)
+    )
+    (property "Datasheet" "~" (id 3) (at 143.51 351.79 0)
+      (effects (font (size 1.27 1.27)) hide)
+    )
+    (pin "1")
+    (pin "2")
+  )
   (symbol (lib_id "power:VCC") (at 257.81 118.11 0) (unit 1)
     (in_bom yes) (on_board yes) (fields_autoplaced)
@@
     (pin "1")
   )
-  (symbol (lib_id "Connector:Conn_01x02_Male") (at 130.81 299.72 0) (unit 1)
+  (symbol (lib_id "Connector:Conn_01x02_Male") (at 130.81 347.98 0) (unit 1)
     (in_bom yes) (on_board yes)
-    (property "Reference" "J9" (id 0) (at 127 299.72 0)
+    (property "Reference" "J9" (id 0) (at 127 347.98 0)
       (effects (font (size 1.27 1.27)) (justify right))
     )
-    (property "Value" "DMA CTRL" (id 1) (at 128.27 302.26 0)
+    (property "Value" "DMA CTRL" (id 1) (at 128.27 350.52 0)
       (effects (font (size 1.27 1.27)) (justify right))
     )
-    (property "Footprint" "" (id 2) (at 130.81 299.72 0)
+    (property "Footprint" "" (id 2) (at 130.81 347.98 0)
       (effects (font (size 1.27 1.27)) hide)
     )
-    (property "Datasheet" "~" (id 3) (at 130.81 299.72 0)
+    (property "Datasheet" "~" (id 3) (at 130.81 347.98 0)
       (effects (font (size 1.27 1.27)) hide)
     )
@@
       (reference "J?") (unit 1) (value "Conn_02x40_Odd_Even") (footprint "Connector_PinHeader_2.54mm:PinHeader_2x40_P2.54mm_Vertical")
     )
+    (path "/c704cbbe-e57c-4287-ac30-25735541d498"
+      (reference "R?") (unit 1) (value "1 K") (footprint "")
+    )
     (path "/6539240f-32f3-440a-b657-9628431f5085"

Commit message: Big push, Sysctl, DMA Reg
Parts:
- removed J3, J?: VPA/VDA, symbol Connector:Conn_01x02_Male
- removed J4, J?: Conn_02x40_Odd_Even, Connector_PinHeader_2.54mm:PinHeader_2x40_P2.54mm_Vertical, symbol Connector_Generic:Conn_02x40_Odd_Even
- removed J5: AUX, Connector_PinHeader_2.54mm:PinHeader_2x18_P2.54mm_Vertical, symbol Connector_Generic:Conn_02x18_Odd_Even
- removed J9: DMA CTRL, symbol Connector:Conn_01x02_Male
- removed J?: DMA, Connector_PinHeader_2.54mm:PinHeader_2x18_P2.54mm_Vertical, symbol Connector_Generic:Conn_02x18_Odd_Even
- removed R?: 1 K, symbol Device:R
- added C1, C10, C11, C12, C13, C14, C15, C16, C17, C2, C3, C4, C5, C6, C7, C8, C9: 100n, Capacitor_THT:C_Disc_D3.4mm_W2.1mm_P2.50mm, symbol Device:C
- added H1, H2: MountingHole_Pad, MountingHole:MountingHole_3.2mm_M3_Pad, symbol Mechanical:MountingHole_Pad
- added J1, J14, J17, J4: VPA/VDA, Connector_PinHeader_2.54mm:PinHeader_1x02_P2.54mm_Vertical, symbol Connector_Generic:Conn_01x02
- added J12: CPU, Connector_PinHeader_2.54mm:PinHeader_2x18_P2.54mm_Vertical, symbol Connector_Generic:Conn_02x18_Odd_Even
- added J15, J18, J2, J5: Conn_02x40_Odd_Even, Connector_PinHeader_2.54mm:PinHeader_2x40_P2.54mm_Vertical, symbol Connector_Generic:Conn_02x40_Odd_Even
- added J16, J19, J3: DMA, Connector_PinHeader_2.54mm:PinHeader_2x18_P2.54mm_Vertical, symbol Connector_Generic:Conn_02x18_Odd_Even
- added J20: DMA Shim ~{DMA0-3}, Connector_PinHeader_2.54mm:PinHeader_2x04_P2.54mm_Vertical, symbol Vega816:Conn_02x04_Odd_Even
- added U10, U11, U13, U14, U15, U16, U17, U18, U19, U20, U21, U22, U23, U25, U26, U29, U30, U31, U32, U33, U34: 74HC541, Package_DIP:DIP-20_W7.62mm_Socket, symbol Vega816:74HC541
- added U12, U24, U27: 74AHCT245, Package_DIP:DIP-20_W7.62mm_Socket, symbol Vega816:74AHCT245
- added U28, U?: 74HC00, Package_DIP:DIP-14_W7.62mm_Socket, symbol Vega816:74HC00
- J?: renamed from J6; footprint (none) -> Connector_PinHeader_2.54mm:PinHeader_1x02_P2.54mm_Vertical; symbol Connector:Conn_01x02_Male -> Connector_Generic:Conn_01x02
- J?: renamed from J10; footprint (none) -> Connector_PinHeader_2.54mm:PinHeader_1x02_P2.54mm_Vertical; symbol Connector:Conn_01x02_Male -> Connector_Generic:Conn_01x02
- U?: renamed from U21; footprint (none) -> Package_DIP:DIP-20_W7.62mm_Socket
- U?: renamed from U18; footprint (none) -> Package_DIP:DIP-20_W7.62mm_Socket
- U?: renamed from U20; footprint (none) -> Package_DIP:DIP-20_W7.62mm_Socket
- U?: renamed from U16; footprint (none) -> Package_DIP:DIP-20_W7.62mm_Socket
- U?: renamed from U23; footprint (none) -> Package_DIP:DIP-20_W7.62mm_Socket
- U?: renamed from U19; footprint (none) -> Package_DIP:DIP-20_W7.62mm_Socket
- U?: renamed from U22; footprint (none) -> Package_DIP:DIP-20_W7.62mm_Socket
- renumbered J11 to J?, J7 to J?, J12 to J?, J8 to J?, U17 to U?
Connections:
- net A0: now also J12.19 (Pin_19), U13.2 (A0), U22.2 (A0), U29.9 (A7)
- net A1: now also J12.17 (Pin_17), U13.3 (A1), U22.3 (A1), U29.8 (A6)
- net A10: now also J5.79 (Pin_79), U15.4 (A2), U20.4 (A2), U31.7 (A5)
- net A11: now also J5.77 (Pin_77), U15.5 (A3), U20.5 (A3), U31.6 (A4)
- net A12: now also J5.75 (Pin_75), U15.6 (A4), U20.6 (A4), U31.5 (A3)
- net A13: now also J5.73 (Pin_73), U15.7 (A5), U20.7 (A5), U31.4 (A2)
- net A14: now also J5.71 (Pin_71), U15.8 (A6), U20.8 (A6), U31.3 (A1)
- net A15: now also J5.69 (Pin_69), U15.9 (A7), U20.9 (A7), U31.2 (A0)
- net A16: now also J5.67 (Pin_67), U17.2 (A0), U19.2 (A0), U33.9 (A7)
- net A17: now also J5.65 (Pin_65), U17.3 (A1), U19.3 (A1), U33.8 (A6)
- net A18: now also J5.63 (Pin_63), U17.4 (A2), U19.4 (A2), U33.7 (A5)
- net A19: now also J5.61 (Pin_61), U17.5 (A3), U19.5 (A3), U33.6 (A4)
- net A2: now also J12.15 (Pin_15), U13.4 (A2), U22.4 (A2), U29.7 (A5)
- net A20: now also J5.59 (Pin_59), U17.6 (A4), U19.6 (A4), U33.5 (A3)
- net A21: now also J5.57 (Pin_57), U17.7 (A5), U19.7 (A5), U33.4 (A2)
- net A22: now also J5.55 (Pin_55), U17.8 (A6), U19.8 (A6), U33.3 (A1)
- net A23: now also J5.53 (Pin_53), U17.9 (A7), U19.9 (A7), U33.2 (A0)
- net A3: now also J12.13 (Pin_13), U13.5 (A3), U22.5 (A3), U29.6 (A4)
- net A4: now also J12.11 (Pin_11), U13.6 (A4), U22.6 (A4), U29.5 (A3)
- net A5: now also J12.9 (Pin_9), U13.7 (A5), U22.7 (A5), U29.4 (A2)
- net A6: now also J12.7 (Pin_7), U13.8 (A6), U22.8 (A6), U29.3 (A1)
- net A7: now also J12.5 (Pin_5), U13.9 (A7), U22.9 (A7), U29.2 (A0)
- net A8: now also J12.3 (Pin_3), U15.2 (A0), U20.2 (A0), U31.9 (A7)
- net A9: now also J12.1 (Pin_1), U15.3 (A1), U20.3 (A1), U31.8 (A6)
- net AA0: now also J16.19 (Pin_19), U29.11 (Y7); no longer J?.19 (Pin_19), U?.11 (Y7)
- net AA1: now also J16.17 (Pin_17), U29.12 (Y6); no longer J?.17 (Pin_17), U?.12 (Y6)
- net AA10: now also J15.79 (Pin_79), U31.13 (Y5); no longer J?.79 (Pin_79), U?.13 (Y5)
- net AA11: now also J15.77 (Pin_77), U31.14 (Y4); no longer J?.77 (Pin_77), U?.14 (Y4)
- net AA12: now also J15.75 (Pin_75), U31.15 (Y3); no longer J?.75 (Pin_75), U?.15 (Y3)
- net AA13: now also J15.73 (Pin_73), U31.16 (Y2); no longer J?.73 (Pin_73), U?.16 (Y2)
- net AA14: now also J15.71 (Pin_71), U31.17 (Y1); no longer J?.71 (Pin_71), U?.17 (Y1)
- net AA15: now also J15.69 (Pin_69), U31.18 (Y0); no longer J?.69 (Pin_69), U?.18 (Y0)
- net AA16: now also J15.67 (Pin_67), U33.11 (Y7); no longer J?.67 (Pin_67), U?.11 (Y7)
- net AA17: now also J15.65 (Pin_65), U33.12 (Y6); no longer J?.65 (Pin_65), U?.12 (Y6)
- net AA18: now also J15.63 (Pin_63), U33.13 (Y5); no longer J?.63 (Pin_63), U?.13 (Y5)
- net AA19: now also J15.61 (Pin_61), U33.14 (Y4); no longer J?.61 (Pin_61), U?.14 (Y4)
- net AA2: now also J16.15 (Pin_15), U29.13 (Y5); no longer J?.15 (Pin_15), U?.13 (Y5)
- net AA20: now also J15.59 (Pin_59), U33.15 (Y3); no longer J?.59 (Pin_59), U?.15 (Y3)
- net AA21: now also J15.57 (Pin_57), U33.16 (Y2); no longer J?.57 (Pin_57), U?.16 (Y2)
- net AA22: now also J15.55 (Pin_55), U33.17 (Y1); no longer J?.55 (Pin_55), U?.17 (Y1)
- net AA23: now also J15.53 (Pin_53), U33.18 (Y0); no longer J?.53 (Pin_53), U?.18 (Y0)
- net AA3: now also J16.13 (Pin_13), U29.14 (Y4); no longer J?.13 (Pin_13), U?.14 (Y4)
- net AA4: now also J16.11 (Pin_11), U29.15 (Y3); no longer J?.11 (Pin_11), U?.15 (Y3)
- net AA5: now also J16.9 (Pin_9), U29.16 (Y2); no longer J?.9 (Pin_9), U?.16 (Y2)
- net AA6: now also J16.7 (Pin_7), U29.17 (Y1); no longer J?.7 (Pin_7), U?.17 (Y1)
- net AA7: now also J16.5 (Pin_5), U29.18 (Y0); no longer J?.5 (Pin_5), U?.18 (Y0)
- net AA8: now also J16.3 (Pin_3), U31.11 (Y7); no longer J?.3 (Pin_3), U?.11 (Y7)
- net AA9: now also J16.1 (Pin_1), U31.12 (Y6); no longer J?.1 (Pin_1), U?.12 (Y6)
- net ABE: now also J15.25 (Pin_25), U34.3 (A1); no longer J?.25 (Pin_25), U?.7 (A5)
- net ACLK: now also J15.15 (Pin_15), U30.16 (Y2); no longer J?.15 (Pin_15), U?.13 (Y5)
- net ACLK_SRC: now also J15.13 (Pin_13), U34.7 (A5); no longer J?.13 (Pin_13), U?.3 (A1)
- net AD0: now also J16.35 (Pin_35), U27.2 (A0); no longer J?.35 (Pin_35), U?.9 (A7)
- net AD1: now also J16.33 (Pin_33), U27.3 (A1); no longer J?.33 (Pin_33), U?.8 (A6)
- net AD2: now also J16.31 (Pin_31), U27.4 (A2); no longer J?.31 (Pin_31), U?.7 (A5)
- net AD3: now also J16.29 (Pin_29), U27.5 (A3); no longer J?.29 (Pin_29), U?.6 (A4)
- net AD4: now also J16.27 (Pin_27), U27.6 (A4); no longer J?.27 (Pin_27), U?.5 (A3)
- net AD5: now also J16.25 (Pin_25), U27.7 (A5); no longer J?.25 (Pin_25), U?.4 (A2)
- net AD6: now also J16.23 (Pin_23), U27.8 (A6); no longer J?.23 (Pin_23), U?.3 (A1)
- net AD7: now also J16.21 (Pin_21), U27.9 (A7); no longer J?.21 (Pin_21), U?.2 (A0)
- net AM: now also J15.45 (Pin_45), U26.14 (Y4); no longer J?.45 (Pin_45), U?.14 (Y4)
- net ARDY_IN: now also J15.27 (Pin_27), U34.2 (A0); no longer J?.27 (Pin_27), U?.8 (A6)
- net ARST: now also J15.9 (Pin_9), U30.17 (Y1); no longer J?.9 (Pin_9), U?.12 (Y6)
- net AR~{W}: now also J15.35 (Pin_35), U30.11 (Y7); no longer J?.35 (Pin_35), U?.18 (Y0)
- net ASYNC: now also J15.31 (Pin_31), U30.13 (Y5); no longer J?.31 (Pin_31), U?.16 (Y2)
- net AVA: now also J15.33 (Pin_33), U30.12 (Y6); no longer J?.33 (Pin_33), U?.17 (Y1)
- net AVDA: now also J14.2 (Pin_2), U32.17 (Y1); no longer J?.2 (Pin_2), U?.12 (Y6)
- net AVPA: now also J14.1 (Pin_1), U32.18 (Y0); no longer J?.1 (Pin_1), U?.11 (Y7)
- net AX: now also J15.47 (Pin_47), U26.13 (Y5); no longer J?.47 (Pin_47), U?.13 (Y5)
- net BE: now also U?.17 (Y1), J5.25 (Pin_25), U16.13 (Y5), U18.13 (Y5), U34.17 (Y1); no longer U?.13 (Y5)
- net CLK: now also U?.4 (A2), J5.15 (Pin_15), U11.7 (A5), U23.7 (A5), U30.4 (A2); no longer U?.7 (A5)
- net CLK_SRC: now also U?.13 (Y5), J5.13 (Pin_13), U16.17 (Y1), U18.17 (Y1), U34.13 (Y5); no longer U?.17 (Y1)
- net D0: now also U?.18 (B0), J12.35 (Pin_35), U12.11 (B7), U24.11 (B7), U27.18 (B0); no longer U?.11 (B7)
- net D1: now also U?.17 (B1), J12.33 (Pin_33), U12.12 (B6), U24.12 (B6), U27.17 (B1); no longer U?.12 (B6)
- net D2: now also U?.16 (B2), J12.31 (Pin_31), U12.13 (B5), U24.13 (B5), U27.16 (B2); no longer U?.13 (B5)
- net D3: now also U?.15 (B3), J12.29 (Pin_29), U12.14 (B4), U24.14 (B4), U27.15 (B3); no longer U?.14 (B4)
- net D4: now also U?.14 (B4), J12.27 (Pin_27), U12.15 (B3), U24.15 (B3), U27.14 (B4); no longer U?.15 (B3)
- net D5: now also U?.13 (B5), J12.25 (Pin_25), U12.16 (B2), U24.16 (B2), U27.13 (B5); no longer U?.16 (B2)
- net D6: now also U?.12 (B6), J12.23 (Pin_23), U12.17 (B1), U24.17 (B1), U27.12 (B6); no longer U?.17 (B1)
- net D7: now also U?.11 (B7), J12.21 (Pin_21), U12.18 (B0), U24.18 (B0), U27.11 (B7); no longer U?.18 (B0)
- net E: now also J5.43 (Pin_43), U10.6 (A4), U25.6 (A4), U26.5 (A3)
- net GND: now also U?.19 (G2), U?.19 (G2), U?.19 (G2), U?.19 (G2), U?.19 (G2), U?.19 (G2), U?.19 (G2), U?.7 (A5), U?.8 (A6), U?.9 (A7), C1.2, C10.2, C11.2, C12.2, C13.2, C14.2, C15.2, C16.2, C17.2, C2.2, C3.2, C4.2, C5.2, C6.2, C7.2, C8.2, C9.2, H1.1, H2.1, J12.10 (Pin_10), J12.12 (Pin_12), J12.14 (Pin_14), J12.16 (Pin_16), J12.18 (Pin_18), J12.2 (Pin_2), J12.20 (Pin_20), J12.22 (Pin_22), J12.24 (Pin_24), J12.26 (Pin_26), J12.28 (Pin_28), J12.30 (Pin_30), J12.32 (Pin_32), J12.34 (Pin_34), J12.36 (Pin_36), J12.4 (Pin_4), J12.6 (Pin_6), J12.8 (Pin_8), J15.10 (Pin_10), J15.12 (Pin_12), J15.14 (Pin_14), J15.16 (Pin_16), J15.18 (Pin_18), J15.2 (Pin_2), J15.20 (Pin_20), J15.22 (Pin_22), J15.24 (Pin_24), J15.26 (Pin_26), J15.28 (Pin_28), J15.3 (Pin_3), J15.30 (Pin_30), J15.32 (Pin_32), J15.34 (Pin_34), J15.36 (Pin_36), J15.38 (Pin_38), J15.4 (Pin_4), J15.40 (Pin_40), J15.42 (Pin_42), J15.44 (Pin_44), J15.46 (Pin_46), J15.48 (Pin_48), J15.50 (Pin_50), J15.52 (Pin_52), J15.54 (Pin_54), J15.56 (Pin_56), J15.58 (Pin_58), J15.6 (Pin_6), J15.60 (Pin_60), J15.62 (Pin_62), J15.64 (Pin_64), J15.66 (Pin_66), J15.68 (Pin_68), J15.70 (Pin_70), J15.72 (Pin_72), J15.74 (Pin_74), J15.76 (Pin_76), J15.78 (Pin_78), J15.8 (Pin_8), J15.80 (Pin_80), J16.10 (Pin_10), J16.12 (Pin_12), J16.14 (Pin_14), J16.16 (Pin_16), J16.18 (Pin_18), J16.2 (Pin_2), J16.20 (Pin_20), J16.22 (Pin_22), J16.24 (Pin_24), J16.26 (Pin_26), J16.28 (Pin_28), J16.30 (Pin_30), J16.32 (Pin_32), J16.34 (Pin_34), J16.36 (Pin_36), J16.4 (Pin_4), J16.6 (Pin_6), J16.8 (Pin_8), J18.10 (Pin_10), J18.12 (Pin_12), J18.14 (Pin_14), J18.16 (Pin_16), J18.18 (Pin_18), J18.2 (Pin_2), J18.20 (Pin_20), J18.22 (Pin_22), J18.24 (Pin_24), J18.26 (Pin_26), J18.28 (Pin_28), J18.3 (Pin_3), J18.30 (Pin_30), J18.32 (Pin_32), J18.34 (Pin_34), J18.36 (Pin_36), J18.38 (Pin_38), J18.4 (Pin_4), J18.40 (Pin_40), J18.42 (Pin_42), J18.44 (Pin_44), J18.46 (Pin_46), J18.48 (Pin_48), J18.50 (Pin_50), J18.52 (Pin_52), J18.54 (Pin_54), J18.56 (Pin_56), J18.58 (Pin_58), J18.6 (Pin_6), J18.60 (Pin_60), J18.62 (Pin_62), J18.64 (Pin_64), J18.66 (Pin_66), J18.68 (Pin_68), J18.70 (Pin_70), J18.72 (Pin_72), J18.74 (Pin_74), J18.76 (Pin_76), J18.78 (Pin_78), J18.8 (Pin_8), J18.80 (Pin_80), J19.10 (Pin_10), J19.12 (Pin_12), J19.14 (Pin_14), J19.16 (Pin_16), J19.18 (Pin_18), J19.2 (Pin_2), J19.20 (Pin_20), J19.22 (Pin_22), J19.24 (Pin_24), J19.26 (Pin_26), J19.28 (Pin_28), J19.30 (Pin_30), J19.32 (Pin_32), J19.34 (Pin_34), J19.36 (Pin_36), J19.4 (Pin_4), J19.6 (Pin_6), J19.8 (Pin_8), J2.10 (Pin_10), J2.12 (Pin_12), J2.14 (Pin_14), J2.16 (Pin_16), J2.18 (Pin_18), J2.2 (Pin_2), J2.20 (Pin_20), J2.22 (Pin_22), J2.24 (Pin_24), J2.26 (Pin_26), J2.28 (Pin_28), J2.3 (Pin_3), J2.30 (Pin_30), J2.32 (Pin_32), J2.34 (Pin_34), J2.36 (Pin_36), J2.38 (Pin_38), J2.4 (Pin_4), J2.40 (Pin_40), J2.42 (Pin_42), J2.44 (Pin_44), J2.46 (Pin_46), J2.48 (Pin_48), J2.50 (Pin_50), J2.52 (Pin_52), J2.54 (Pin_54), J2.56 (Pin_56), J2.58 (Pin_58), J2.6 (Pin_6), J2.60 (Pin_60), J2.62 (Pin_62), J2.64 (Pin_64), J2.66 (Pin_66), J2.68 (Pin_68), J2.70 (Pin_70), J2.72 (Pin_72), J2.74 (Pin_74), J2.76 (Pin_76), J2.78 (Pin_78), J2.8 (Pin_8), J2.80 (Pin_80), J20.2 (Pin_2), J20.4 (Pin_4), J20.6 (Pin_6), J20.8 (Pin_8), J3.10 (Pin_10), J3.12 (Pin_12), J3.14 (Pin_14), J3.16 (Pin_16), J3.18 (Pin_18), J3.2 (Pin_2), J3.20 (Pin_20), J3.22 (Pin_22), J3.24 (Pin_24), J3.26 (Pin_26), J3.28 (Pin_28), J3.30 (Pin_30), J3.32 (Pin_32), J3.34 (Pin_34), J3.36 (Pin_36), J3.4 (Pin_4), J3.6 (Pin_6), J3.8 (Pin_8), J5.10 (Pin_10), J5.12 (Pin_12), J5.14 (Pin_14), J5.16 (Pin_16), J5.18 (Pin_18), J5.2 (Pin_2), J5.20 (Pin_20), J5.22 (Pin_22), J5.24 (Pin_24), J5.26 (Pin_26), J5.28 (Pin_28), J5.3 (Pin_3), J5.30 (Pin_30), J5.32 (Pin_32), J5.34 (Pin_34), J5.36 (Pin_36), J5.38 (Pin_38), J5.4 (Pin_4), J5.40 (Pin_40), J5.42 (Pin_42), J5.44 (Pin_44), J5.46 (Pin_46), J5.48 (Pin_48), J5.50 (Pin_50), J5.52 (Pin_52), J5.54 (Pin_54), J5.56 (Pin_56), J5.58 (Pin_58), J5.6 (Pin_6), J5.60 (Pin_60), J5.62 (Pin_62), J5.64 (Pin_64), J5.66 (Pin_66), J5.68 (Pin_68), J5.70 (Pin_70), J5.72 (Pin_72), J5.74 (Pin_74), J5.76 (Pin_76), J5.78 (Pin_78), J5.8 (Pin_8), J5.80 (Pin_80), U10.10 (GND), U10.19 (G2), U11.10 (GND), U11.19 (G2), U12.10 (GND), U13.10 (GND), U13.19 (G2), U14.10 (GND), U14.19 (G2), U14.2 (A0), U14.3 (A1), U14.4 (A2), U14.5 (A3), U14.6 (A4), U15.10 (GND), U15.19 (G2), U16.10 (GND), U16.19 (G2), U16.9 (A7), U17.10 (GND), U17.19 (G2), U18.10 (GND), U18.19 (G2), U18.9 (A7), U19.10 (GND), U19.19 (G2), U20.10 (GND), U20.19 (G2), U21.10 (GND), U21.19 (G2), U21.2 (A0), U21.3 (A1), U21.4 (A2), U21.5 (A3), U21.6 (A4), U22.10 (GND), U22.19 (G2), U23.10 (GND), U23.19 (G2), U24.10 (GND), U25.10 (GND), U25.19 (G2), U26.10 (GND), U26.19 (G2), U27.10 (GND), U28.7 (GND), U29.10 (GND), U29.19 (G2), U30.10 (GND), U30.19 (G2), U31.10 (GND), U31.19 (G2), U32.10 (GND), U32.19 (G2), U32.5 (A3), U32.6 (A4), U32.7 (A5), U32.8 (A6), U32.9 (A7), U33.10 (GND), U33.19 (G2), U34.10 (GND), U34.19 (G2), U34.9 (A7), U?.7 (GND); no longer J?.1 (Pin_1), J?.1 (Pin_1), U?.2 (A0), U?.20 (VCC), U?.20 (VCC), U?.20 (VCC), U?.20 (VCC), U?.20 (VCC), U?.20 (VCC), U?.20 (VCC), U?.20 (VCC), U?.3 (A1), U?.4 (A2)
- net M: now also J5.45 (Pin_45), U10.5 (A3), U25.5 (A3), U26.6 (A4)
- net RDY_IN: now also U?.18 (Y0), J5.27 (Pin_27), U16.12 (Y6), U18.12 (Y6), U34.18 (Y0); no longer U?.12 (Y6)
- net RST: now also U?.3 (A1), J5.9 (Pin_9), U11.8 (A6), U23.8 (A6), U30.3 (A1); no longer U?.8 (A6)
- net R~{W}: now also U?.9 (A7), J5.35 (Pin_35), U11.2 (A0), U12.1 (A->B), U23.2 (A0), U24.1 (A->B), U27.1 (A->B), U30.9 (A7); no longer U?.2 (A0)
- net SYNC: now also U?.7 (A5), J5.31 (Pin_31), U11.4 (A2), U23.4 (A2), U30.7 (A5); no longer U?.4 (A2)
- net VA: now also U?.8 (A6), J5.33 (Pin_33), U11.3 (A1), U23.3 (A1), U30.8 (A6); no longer U?.3 (A1)
- net VDA: now also U?.3 (A1), J4.2 (Pin_2), U14.8 (A6), U21.8 (A6), U32.3 (A1); no longer U?.8 (A6)
- net VPA: now also U?.2 (A0), J4.1 (Pin_1), U14.9 (A7), U21.9 (A7), U32.2 (A0); no longer U?.9 (A7)
- net X: now also J5.47 (Pin_47), U10.4 (A2), U25.4 (A2), U26.7 (A5)
- net ~{AABORT}: now also J15.23 (Pin_23), U34.4 (A2); no longer J?.23 (Pin_23), U?.6 (A4)
- net ~{ABANK0}: now also J15.41 (Pin_41), U26.16 (Y2); no longer J?.41 (Pin_41), U?.16 (Y2)
- net ~{ABORT}: now also U?.16 (Y2), J5.23 (Pin_23), U16.14 (Y4), U18.14 (Y4), U34.16 (Y2); no longer U?.14 (Y4)
- net ~{ACLK_EN}: now also J15.11 (Pin_11), U34.8 (A6); no longer J?.11 (Pin_11), U?.2 (A0)
- net ~{ACLK}: now also J15.17 (Pin_17), U30.15 (Y3); no longer J?.17 (Pin_17), U?.14 (Y4)
- net ~{AIRQ}: now also J15.19 (Pin_19), U34.6 (A4); no longer J?.19 (Pin_19), U?.4 (A2)
- net ~{AML}: now also J15.51 (Pin_51), U26.11 (Y7); no longer J?.51 (Pin_51), U?.11 (Y7)
- net ~{AMR}⎒: now also J15.5 (Pin_5), U32.16 (Y2); no longer J?.5 (Pin_5), U?.13 (Y5)
- net ~{ANMI}: now also J15.21 (Pin_21), U34.5 (A3); no longer J?.21 (Pin_21), U?.5 (A3)
- net ~{ARD}: now also J15.37 (Pin_37), U26.18 (Y0); no longer J?.37 (Pin_37), U?.18 (Y0)
- net ~{ARST}: now also J15.7 (Pin_7), U30.18 (Y0); no longer J?.7 (Pin_7), U?.11 (Y7)
- net ~{AVP}: now also J15.49 (Pin_49), U26.12 (Y6); no longer J?.49 (Pin_49), U?.12 (Y6)
- net ~{AWAI}: now also J15.29 (Pin_29), U30.14 (Y4); no longer J?.29 (Pin_29), U?.15 (Y3)
- net ~{AWR}: now also J15.39 (Pin_39), U26.17 (Y1); no longer J?.39 (Pin_39), U?.17 (Y1)
- net ~{BANK0}: now also J5.41 (Pin_41), U10.7 (A5), U25.7 (A5), U26.4 (A2)
- net ~{CLK_EN}: now also U?.12 (Y6), J5.11 (Pin_11), U16.18 (Y0), U18.18 (Y0), U34.12 (Y6); no longer U?.18 (Y0)
- net ~{CLK}: now also U?.5 (A3), J5.17 (Pin_17), U11.6 (A4), U23.6 (A4), U30.5 (A3); no longer U?.6 (A4)
- net ~{IRQ}: now also U?.14 (Y4), J5.19 (Pin_19), U16.16 (Y2), U18.16 (Y2), U34.14 (Y4); no longer U?.16 (Y2)
- net ~{ML}: now also J5.51 (Pin_51), U10.2 (A0), U25.2 (A0), U26.9 (A7)
- net ~{MR}⎒: now also U?.4 (A2), J5.5 (Pin_5), U14.7 (A5), U21.7 (A5), U32.4 (A2); no longer U?.7 (A5)
- net ~{NMI}: now also J5.21 (Pin_21), U16.15 (Y3), U18.15 (Y3), U34.15 (Y3)
- net ~{RD}: now also J5.37 (Pin_37), U10.9 (A7), U25.9 (A7), U26.2 (A0)
- net ~{RST}: now also U?.2 (A0), J5.7 (Pin_7), U11.9 (A7), U23.9 (A7), U30.2 (A0); no longer U?.9 (A7)
- net ~{VP}: now also J5.49 (Pin_49), U10.3 (A1), U25.3 (A1), U26.8 (A6)
- net ~{WAI}: now also U?.6 (A4), J5.29 (Pin_29), U11.5 (A3), U23.5 (A3), U30.6 (A4); no longer U?.5 (A3)
- net ~{WR}: now also J5.39 (Pin_39), U10.8 (A6), U25.8 (A6), U26.3 (A1)
- net ~{CMR}⎒: now reaches U?.16 (Y2)
- net ~{CMR}⎒: now also J?.5 (Pin_5)
- net CVDA: now reaches U?.17 (Y1)
- net CVDA: now also J?.2 (Pin_2)
- net CVPA: now reaches U?.18 (Y0)
- net CVPA: now also J?.1 (Pin_1)
- net AE renamed CEM
- net ~{DMA} renamed ~{C_DMA}
- net ~{C_DMA}: now also J20.5 (Pin_5); no longer U?.19 (G2), U?.19 (G2), U?.19 (G2), U?.19 (G2), U?.19 (G2), U?.19 (G2), U?.19 (G2)
- new net AEM: J15.43 (Pin_43), U26.15 (Y3)
- new net BA0: J3.19 (Pin_19), U22.18 (Y0)
- new net BA1: J3.17 (Pin_17), U22.17 (Y1)
- new net BA10: J2.79 (Pin_79), U20.16 (Y2)
- new net BA11: J2.77 (Pin_77), U20.15 (Y3)
- new net BA12: J2.75 (Pin_75), U20.14 (Y4)
- new net BA13: J2.73 (Pin_73), U20.13 (Y5)
- new net BA14: J2.71 (Pin_71), U20.12 (Y6)
- new net BA15: J2.69 (Pin_69), U20.11 (Y7)
- new net BA16: J2.67 (Pin_67), U19.18 (Y0)
- new net BA17: J2.65 (Pin_65), U19.17 (Y1)
- new net BA18: J2.63 (Pin_63), U19.16 (Y2)
- new net BA19: J2.61 (Pin_61), U19.15 (Y3)
- new net BA2: J3.15 (Pin_15), U22.16 (Y2)
- new net BA20: J2.59 (Pin_59), U19.14 (Y4)
- new net BA21: J2.57 (Pin_57), U19.13 (Y5)
- new net BA22: J2.55 (Pin_55), U19.12 (Y6)
- new net BA23: J2.53 (Pin_53), U19.11 (Y7)
- new net BA3: J3.13 (Pin_13), U22.15 (Y3)
- new net BA4: J3.11 (Pin_11), U22.14 (Y4)
- new net BA5: J3.9 (Pin_9), U22.13 (Y5)
- new net BA6: J3.7 (Pin_7), U22.12 (Y6)
- new net BA7: J3.5 (Pin_5), U22.11 (Y7)
- new net BA8: J3.3 (Pin_3), U20.18 (Y0)
- new net BA9: J3.1 (Pin_1), U20.17 (Y1)
- new net BBE: J2.25 (Pin_25), U18.7 (A5)
- new net BCLK: J2.15 (Pin_15), U23.13 (Y5)
- new net BCLK_SRC: J2.13 (Pin_13), U18.3 (A1)
- new net BD0: J3.35 (Pin_35), U24.9 (A7)
- new net BD1: J3.33 (Pin_33), U24.8 (A6)
- new net BD2: J3.31 (Pin_31), U24.7 (A5)
- new net BD3: J3.29 (Pin_29), U24.6 (A4)
- new net BD4: J3.27 (Pin_27), U24.5 (A3)
- new net BD5: J3.25 (Pin_25), U24.4 (A2)
- new net BD6: J3.23 (Pin_23), U24.3 (A1)
- new net BD7: J3.21 (Pin_21), U24.2 (A0)
- new net BEM: J2.43 (Pin_43), U25.14 (Y4)
- new net BM: J2.45 (Pin_45), U25.15 (Y3)
- new net BRDY_IN: J2.27 (Pin_27), U18.8 (A6)
- new net BRST: J2.9 (Pin_9), U23.12 (Y6)
- new net BR~{W}: J2.35 (Pin_35), U23.18 (Y0)
- new net BSYNC: J2.31 (Pin_31), U23.16 (Y2)
- new net BVA: J2.33 (Pin_33), U23.17 (Y1)
- new net BVDA: J1.2 (Pin_2), U21.12 (Y6)
- new net BVPA: J1.1 (Pin_1), U21.11 (Y7)
- new net BX: J2.47 (Pin_47), U25.16 (Y2)
- new net CA0: J?.19 (Pin_19), U?.11 (Y7)
- new net CA1: J?.17 (Pin_17), U?.12 (Y6)
- new net CA10: J?.79 (Pin_79), U?.13 (Y5)
- new net CA11: J?.77 (Pin_77), U?.14 (Y4)
- new net CA12: J?.75 (Pin_75), U?.15 (Y3)
- new net CA13: J?.73 (Pin_73), U?.16 (Y2)
- new net CA14: J?.71 (Pin_71), U?.17 (Y1)
- new net CA15: J?.69 (Pin_69), U?.18 (Y0)
- new net CA16: J?.67 (Pin_67), U?.11 (Y7)
- new net CA17: J?.65 (Pin_65), U?.12 (Y6)
- new net CA18: J?.63 (Pin_63), U?.13 (Y5)
- new net CA19: J?.61 (Pin_61), U?.14 (Y4)
- new net CA2: J?.15 (Pin_15), U?.13 (Y5)
- new net CA20: J?.59 (Pin_59), U?.15 (Y3)
- new net CA21: J?.57 (Pin_57), U?.16 (Y2)
- new net CA22: J?.55 (Pin_55), U?.17 (Y1)
- new net CA23: J?.53 (Pin_53), U?.18 (Y0)
- new net CA3: J?.13 (Pin_13), U?.14 (Y4)
- new net CA4: J?.11 (Pin_11), U?.15 (Y3)
- new net CA5: J?.9 (Pin_9), U?.16 (Y2)
- new net CA6: J?.7 (Pin_7), U?.17 (Y1)
- new net CA7: J?.5 (Pin_5), U?.18 (Y0)
- new net CA8: J?.3 (Pin_3), U?.11 (Y7)
- new net CA9: J?.1 (Pin_1), U?.12 (Y6)
- new net CBE: J?.25 (Pin_25), U?.3 (A1)
- new net CCLK: J?.15 (Pin_15), U?.16 (Y2)
- new net CCLK_SRC: J?.13 (Pin_13), U?.7 (A5)
- new net CD0: J?.35 (Pin_35), U?.2 (A0)
- new net CD1: J?.33 (Pin_33), U?.3 (A1)
- new net CD2: J?.31 (Pin_31), U?.4 (A2)
- new net CD3: J?.29 (Pin_29), U?.5 (A3)
- new net CD4: J?.27 (Pin_27), U?.6 (A4)
- new net CD5: J?.25 (Pin_25), U?.7 (A5)
- new net CD6: J?.23 (Pin_23), U?.8 (A6)
- new net CD7: J?.21 (Pin_21), U?.9 (A7)
- new net CM: J?.45 (Pin_45), U?.14 (Y4)
- new net CRDY_IN: J?.27 (Pin_27), U?.2 (A0)
- new net CRST: J?.9 (Pin_9), U?.17 (Y1)
- new net CR~{W}: J?.35 (Pin_35), U?.11 (Y7)
- new net CSYNC: J?.31 (Pin_31), U?.13 (Y5)
- new net CVA: J?.33 (Pin_33), U?.12 (Y6)
- new net CX: J?.47 (Pin_47), U?.13 (Y5)
- new net DA0: J19.19 (Pin_19), U13.18 (Y0)
- new net DA1: J19.17 (Pin_17), U13.17 (Y1)
- new net DA10: J18.79 (Pin_79), U15.16 (Y2)
- new net DA11: J18.77 (Pin_77), U15.15 (Y3)
- new net DA12: J18.75 (Pin_75), U15.14 (Y4)
- new net DA13: J18.73 (Pin_73), U15.13 (Y5)
- new net DA14: J18.71 (Pin_71), U15.12 (Y6)
- new net DA15: J18.69 (Pin_69), U15.11 (Y7)
- new net DA16: J18.67 (Pin_67), U17.18 (Y0)
- new net DA17: J18.65 (Pin_65), U17.17 (Y1)
- new net DA18: J18.63 (Pin_63), U17.16 (Y2)
- new net DA19: J18.61 (Pin_61), U17.15 (Y3)
- new net DA2: J19.15 (Pin_15), U13.16 (Y2)
- new net DA20: J18.59 (Pin_59), U17.14 (Y4)
- new net DA21: J18.57 (Pin_57), U17.13 (Y5)
- new net DA22: J18.55 (Pin_55), U17.12 (Y6)
- new net DA23: J18.53 (Pin_53), U17.11 (Y7)
- new net DA3: J19.13 (Pin_13), U13.15 (Y3)
- new net DA4: J19.11 (Pin_11), U13.14 (Y4)
- new net DA5: J19.9 (Pin_9), U13.13 (Y5)
- new net DA6: J19.7 (Pin_7), U13.12 (Y6)
- new net DA7: J19.5 (Pin_5), U13.11 (Y7)
- new net DA8: J19.3 (Pin_3), U15.18 (Y0)
- new net DA9: J19.1 (Pin_1), U15.17 (Y1)
- new net DBE: J18.25 (Pin_25), U16.7 (A5)
- new net DCLK: J18.15 (Pin_15), U11.13 (Y5)
- new net DCLK_SRC: J18.13 (Pin_13), U16.3 (A1)
- new net DD0: J19.35 (Pin_35), U12.9 (A7)
- new net DD1: J19.33 (Pin_33), U12.8 (A6)
- new net DD2: J19.31 (Pin_31), U12.7 (A5)
- new net DD3: J19.29 (Pin_29), U12.6 (A4)
- new net DD4: J19.27 (Pin_27), U12.5 (A3)
- new net DD5: J19.25 (Pin_25), U12.4 (A2)
- new net DD6: J19.23 (Pin_23), U12.3 (A1)
- new net DD7: J19.21 (Pin_21), U12.2 (A0)
- new net DEM: J18.43 (Pin_43), U10.14 (Y4)
- new net DM: J18.45 (Pin_45), U10.15 (Y3)
- new net DRDY_IN: J18.27 (Pin_27), U16.8 (A6)
- new net DRST: J18.9 (Pin_9), U11.12 (Y6)
- new net DR~{W}: J18.35 (Pin_35), U11.18 (Y0)
- new net DSYNC: J18.31 (Pin_31), U11.16 (Y2)
- new net DVA: J18.33 (Pin_33), U11.17 (Y1)
- new net DVDA: J17.2 (Pin_2), U14.12 (Y6)
- new net DVPA: J17.1 (Pin_1), U14.11 (Y7)
- new net DX: J18.47 (Pin_47), U10.16 (Y2)
- new net VCC: C1.1, C10.1, C11.1, C12.1, C13.1, C14.1, C15.1, C16.1, C17.1, C2.1, C3.1, C4.1, C5.1, C6.1, C7.1, C8.1, C9.1, J15.1 (Pin_1), J18.1 (Pin_1), J2.1 (Pin_1), J5.1 (Pin_1), J?.1 (Pin_1), J?.1 (Pin_1), U10.20 (VCC), U11.20 (VCC), U12.20 (VCC), U13.20 (VCC), U14.20 (VCC), U15.20 (VCC), U16.20 (VCC), U17.20 (VCC), U18.20 (VCC), U19.20 (VCC), U20.20 (VCC), U21.20 (VCC), U22.20 (VCC), U23.20 (VCC), U24.20 (VCC), U25.20 (VCC), U26.20 (VCC), U27.20 (VCC), U28.14 (VCC), U29.20 (VCC), U30.20 (VCC), U31.20 (VCC), U32.20 (VCC), U33.20 (VCC), U34.20 (VCC), U?.14 (VCC), U?.20 (VCC), U?.20 (VCC), U?.20 (VCC), U?.20 (VCC), U?.20 (VCC), U?.20 (VCC), U?.20 (VCC), U?.20 (VCC)
- new net ~{A_DMA}: J20.1 (Pin_1), U26.1 (G1), U27.19 (CE), U29.1 (G1), U30.1 (G1), U31.1 (G1), U32.1 (G1), U33.1 (G1), U34.1 (G1)
- new net ~{BABORT}: J2.23 (Pin_23), U18.6 (A4)
- new net ~{BBANK0}: J2.41 (Pin_41), U25.13 (Y5)
- new net ~{BCLK_EN}: J2.11 (Pin_11), U18.2 (A0)
- new net ~{BCLK}: J2.17 (Pin_17), U23.14 (Y4)
- new net ~{BIRQ}: J2.19 (Pin_19), U18.4 (A2)
- new net ~{BML}: J2.51 (Pin_51), U25.18 (Y0)
- new net ~{BMR}⎒: J2.5 (Pin_5), U21.13 (Y5)
- new net ~{BNMI}: J2.21 (Pin_21), U18.5 (A3)
- new net ~{BRD}: J2.37 (Pin_37), U25.11 (Y7)
- new net ~{BRST}: J2.7 (Pin_7), U23.11 (Y7)
- new net ~{BVP}: J2.49 (Pin_49), U25.17 (Y1)
- new net ~{BWAI}: J2.29 (Pin_29), U23.15 (Y3)
- new net ~{BWR}: J2.39 (Pin_39), U25.12 (Y6)
- new net ~{B_DMA}: J20.3 (Pin_3), U18.1 (G1), U19.1 (G1), U20.1 (G1), U21.1 (G1), U22.1 (G1), U23.1 (G1), U24.19 (CE), U25.1 (G1)
- new net ~{CABORT}: J?.23 (Pin_23), U?.4 (A2)
- new net ~{CBANK0}: J?.41 (Pin_41), U?.16 (Y2)
- new net ~{CCLK_EN}: J?.11 (Pin_11), U?.8 (A6)
- new net ~{CCLK}: J?.17 (Pin_17), U?.15 (Y3)
- new net ~{CIRQ}: J?.19 (Pin_19), U?.6 (A4)
- new net ~{CML}: J?.51 (Pin_51), U?.11 (Y7)
- new net ~{CNMI}: J?.21 (Pin_21), U?.5 (A3)
- new net ~{CRD}: J?.37 (Pin_37), U?.18 (Y0)
- new net ~{CRST}: J?.7 (Pin_7), U?.18 (Y0)
- new net ~{CVP}: J?.49 (Pin_49), U?.12 (Y6)
- new net ~{CWAI}: J?.29 (Pin_29), U?.14 (Y4)
- new net ~{CWR}: J?.39 (Pin_39), U?.17 (Y1)
- new net ~{DABORT}: J18.23 (Pin_23), U16.6 (A4)
- new net ~{DBANK0}: J18.41 (Pin_41), U10.13 (Y5)
- new net ~{DCLK_EN}: J18.11 (Pin_11), U16.2 (A0)
- new net ~{DCLK}: J18.17 (Pin_17), U11.14 (Y4)
- new net ~{DIRQ}: J18.19 (Pin_19), U16.4 (A2)
- new net ~{DML}: J18.51 (Pin_51), U10.18 (Y0)
- new net ~{DMR}⎒: J18.5 (Pin_5), U14.13 (Y5)
- new net ~{DNMI}: J18.21 (Pin_21), U16.5 (A3)
- new net ~{DRD}: J18.37 (Pin_37), U10.11 (Y7)
- new net ~{DRST}: J18.7 (Pin_7), U11.11 (Y7)
- new net ~{DVP}: J18.49 (Pin_49), U10.17 (Y1)
- new net ~{DWAI}: J18.29 (Pin_29), U11.15 (Y3)
- new net ~{DWR}: J18.39 (Pin_39), U10.12 (Y6)
- new net ~{D_DMA}: J20.7 (Pin_7), U10.1 (G1), U11.1 (G1), U12.19 (CE), U13.1 (G1), U14.1 (G1), U15.1 (G1), U16.1 (G1), U17.1 (G1)
- no-connect marks 6 -> 24
Other:
- note added: "65816 Breakout 4 Channel Buffer"
- note added: "Channel A"
- note added: "Channel B"
- note added: "Channel C"
- note added: "Channel D"
- note added: "for Kohlbecker 65816 Breakout Rev. A.27"
- note removed: "Stackable CPU Buffer Module for Kohlbecker W65C816 Breakout Board"
- moved on the sheet: J?, U?
