File: kicad/Vega816/C64 Hardware/C64 Hardware.kicad_sch (KiCad schematic)
At the start: 54 parts, among them J0A1 Conn_02x40_Odd_Even, J0B1 CPU, J39 C64 Expansion Port, J43 VPA/VDA, J44 ~{IO_AREA_OUT}

Commit message: Big ol update
Parts:
- removed J0A1: Conn_02x40_Odd_Even, Connector_PinHeader_2.54mm:PinHeader_2x40_P2.54mm_Vertical, symbol Connector_Generic:Conn_02x40_Odd_Even
- removed J0B1: CPU, Connector_PinHeader_2.54mm:PinHeader_2x18_P2.54mm_Vertical, symbol Connector_Generic:Conn_02x18_Odd_Even
- removed J39: C64 Expansion Port, symbol Connector_Generic:Conn_02x40_Odd_Even
- removed J43: VPA/VDA, symbol Connector:Conn_01x02_Male
- removed J?: 6510 P0-P5, symbol Connector_Generic:Conn_02x08_Counter_Clockwise
- removed J?: $02-$03, symbol Connector_Generic:Conn_01x03
- removed J?: Port A, symbol Connector_Generic:Conn_02x08_Counter_Clockwise
- removed J?: Port B, symbol Connector_Generic:Conn_02x08_Counter_Clockwise
- removed J?: PORT A/B, symbol Connector_Generic:Conn_02x03_Counter_Clockwise
- removed J?: Page IO Range, symbol Connector_Generic:Conn_02x08_Odd_Even
- removed J?: 4K IO Range, symbol Connector_Generic:Conn_02x08_Odd_Even
- removed JP?: HI_16KB, symbol Jumper:Jumper_3_Open
- removed JP?: HI_32KB, symbol Jumper:Jumper_3_Open
- removed R?: 10K, symbol Device:R
- removed U? (x2): 74LS138, symbol 74xx:74LS138
- removed U? (x7): 74HC00, symbol 74xx:74HC00
- removed U?: CD4078BE, symbol Vega816:CD4078BE
- removed U? (x2): W65C22SxP, Package_DIP:DIP-40_W15.24mm_Socket, symbol Vega816:W65C22SxP
- added J4: C64 Expansion Port, symbol Vega816:C64_Expansion_Port
- added J?: Port A, symbol Connector_Generic:Conn_02x08_Counter_Clockwise
- added U5 (x2), U6 (x3): 74AHC32, Package_DIP:DIP-14_W7.62mm, symbol 74xx:74LS32
- added U?: 74HC00, symbol 74xx:74HC00
- added U? (x2): W65C22SxP, Package_DIP:DIP-40_W15.24mm_Socket, symbol Vega816:W65C22SxP
Connections:
- net A2 is gone; now on net A0: J0B1.15 (Pin_15), J?.19 (Pin_19), J?.19 (Pin_19), U?.36 (RS2)
- net A3 is gone; now on net A1: J0B1.13 (Pin_13), J?.17 (Pin_17), J?.17 (Pin_17), U?.35 (RS3)
- net A4 is gone; now on net A0: J0B1.11 (Pin_11), J?.15 (Pin_15), J?.15 (Pin_15)
- net A5 is gone; now on net A1: J0B1.9 (Pin_9), J?.13 (Pin_13), J?.13 (Pin_13), U?.2, U?.9 (O6)
- net PA3 is gone; now on net P3_CASS_WRITE: J?.33 (Pin_33), U?.5 (PA3)
- net PA5 is gone; now on net P5_CASS_MOTOR: J?.29 (Pin_29), U?.7 (PA5)
- net ~{P0_LORAM} is gone; now on net PA0: U?.8 (~{LORAM})
- net ~{P1_HIRAM} is gone; now on net PA1: U?.7 (~{HIRAM})
- net ~{P2_CHAREN} is gone; now on net PA2: U?.6 (~{CHAREN})
- net A0: now also J4.A0 (Pin_Y), J4.A2 (Pin_W), J4.A4 (Pin_U), U5.12, U5.2, U?.27 (D6), U?.29 (D4), U?.36 (RS2), U?.38 (RS0)
- net A1: now also J4.A1 (Pin_X), J4.A3 (Pin_V), J4.A5 (Pin_T), U5.1, U5.13, U5.4, U?.26 (D7), U?.28 (D5), U?.35 (RS3), U?.37 (RS1)
- net A10: now also J4.A10 (Pin_M), U5.2
- net A11: now also J4.A11 (Pin_L), U5.13
- net A12: now also J4.A12 (Pin_K), U5.12
- net A13: now also J4.A13 (Pin_J), U5.4
- net A14: now also J4.A14 (Pin_H), U5.5
- net A15: now also J4.A15 (Pin_F), U5.10
- net A6: now also J4.A6 (Pin_S), U5.5
- net A7: now also J4.A7 (Pin_R), U5.10
- net A8: now also J4.A8 (Pin_P), U5.9
- net A9: now also J4.A9 (Pin_N), U5.1
- net CLK: now also J4.PHI2 (Pin_E), U?.25 (ϕ2), U?.25 (ϕ2)
- net D0: now also J4.D0 (Pin_21), U?.1, U?.2, U?.33 (D0)
- net D1: now also J4.D1 (Pin_20), U?.32 (D1)
- net D2: now also J4.D2 (Pin_19), U?.31 (D2)
- net D3: now also J4.D3 (Pin_18), U?.30 (D3)
- net D4: now also J4.D4 (Pin_17), U?.29 (D4), U?.33 (D0)
- net D5: now also J4.D5 (Pin_16), U?.28 (D5), U?.32 (D1)
- net D6: now also J4.D6 (Pin_15), U?.27 (D6), U?.31 (D2)
- net D7: now also J4.D7 (Pin_14), U?.26 (D7), U?.30 (D3)
- net GND: now also J?.2 (Pin_2), J?.4 (Pin_4), J?.6 (Pin_6), J?.8 (Pin_8), J4.GND (Pin_Z), J?.10 (Pin_10), J?.11 (Pin_11), J?.12 (Pin_12), J?.13 (Pin_13), J?.14 (Pin_14), J?.15 (Pin_15), J?.16 (Pin_16), J?.9 (Pin_9), U?.1 (VSS), U?.1 (VSS), U?.35 (RS3), U?.36 (RS2)
- net P3_CASS_WRITE: now also J?.5 (Pin_5), U?.5 (PA3)
- net P5_CASS_MOTOR: now also J?.3 (Pin_3), U?.7 (PA5)
- net PA0: now also J?.8 (Pin_8), U?.2 (PA0)
- net PA1: now also J?.7 (Pin_7), U?.3 (PA1)
- net PA2: now also J?.6 (Pin_6), U?.4 (PA2)
- net PA6: now also J?.2 (Pin_2), U?.8 (PA6)
- net PA7: now also J?.1 (Pin_1), U?.9 (PA7)
- net POTX: now also J?.5 (Pin_5), J?.7 (Pin_7)
- net R~{W}: no longer J0A1.39 (Pin_39), J?.9 (Pin_9), J?.9 (Pin_9), U?.22 (R/~{W})
- net VCC: now also J?.2 (+5VDC), J?.B (+5VDC), J4.+5V (Pin_3), U?.20 (VCC), U?.20 (VCC), U?.24 (CS1), U?.24 (CS1), U?.38 (RS0); no longer J?.6 (SENSE), J?.F (SENSE)
- net ~{$DC00-$DCFF}: no longer U?.23 (~{CS2})
- net ~{A0}: now also U?.3, U?.37 (RS1)
- net ~{BANK0}: now also U5.9
- net ~{RST}: now also J4.~{RESET} (Pin_C), U?.34 (~{RES}), U?.34 (~{RES})
- net at D?.1 (K): now also U6.8, U?.23 (~{CS2})
- net at J?.10 (Pin_10), J?.3: now also U?.12 (PB2)
- net at J?.11 (Pin_11), J?.2: now also U?.11 (PB1)
- net at J?.1, J?.12 (Pin_12): now also U?.10 (PB0)
- net at J?.1, J?.13 (Pin_13): now also U?.2 (PA0)
- net at J?.14 (Pin_14), U?.12 (CD), U?.6 (CC): now also U?.8 (PA6)
- net at J?.15 (Pin_15): now also U?.7 (PA5)
- net at J?.16 (Pin_16), J?.6: now also U?.6 (PA4)
- net at J?.17 (Pin_17), J?.4: now also U?.5 (PA3)
- net at J?.18 (Pin_18), J?.3: now also U?.4 (PA2)
- net at J?.19 (Pin_19), J?.2: now also U?.3 (PA1)
- net at J?.20 (Pin_20), J?.6, U?.13 (CA)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: now also U?.9 (PA7)
- net at J?.4, J?.5 (Pin_5): now also U?.13 (PB3)
- net at J?.6 (Pin_6): now also U?.16 (PB6)
- net at J?.7 (Pin_7): now also U?.15 (PB5)
- net at J?.8 (Pin_8): now also U?.14 (PB4)
- net at J?.9 (Pin_9): now also U?.17 (PB7)
- net PA4 renamed P4_CASS_SENSE
- net P4_CASS_SENSE: now also J?.6 (SENSE), J?.F (SENSE), J?.4 (Pin_4), U?.6 (PA4)
- new net: U5.3, U6.5 (x2)
- new net: U6.10, U6.8
- new net: U6.8, U6.9
- new net: U5.11, U6.4 (x2)
- new net: U6.6, U6.9 (x2)
- new net: U5.6, U6.2 (x2)
- new net: U5.8, U6.1 (x2)
- new net: U6.10, U6.3 (x2)
- new net ~{WR}: J0A1.39 (Pin_39), J4.R/~{W} (Pin_5), J?.9 (Pin_9), J?.9 (Pin_9), U?.22 (R/~{W}), U?.22 (R/~{W}), U?.22 (R/~{W})
- no-connect marks 8 -> 14
Other:
- note added: "6510 $0001"
- note added: "Commodore 64 Hardware"
- note added: "Memory Map $0000-$0001 6510 Registers $D000-$D1FF VIC-II $D400-$D7FF SID #1 $D800-$DBFF Color RAM $DC00-$DCFF CIA#1; inputs (keyboard, joystick, mouse), datasette, IRQ control $DD00-$DDFF CIA#2; serial bus, RS232, NMI control $DE00-$DEFF I/O Area #1 (SID #2) $DF00-$DFFF I/O Area #2"
- note removed: "$D000-$D1FF VIC-II $D400-$D7FF SID $D800-$DBFF Color RAM $DC00-$DCFF CIA#1; inputs (keyboard, joystick, mouse), datasette, IRQ control $DD00-$DDFF CIA#2; serial bus, RS232, NMI control $DE00-$DEFF I/O Area #1 (SID #2) $DF00-$DFFF I/O Area #2"
- note removed: "A1"
- note removed: "PORT A"
- note removed: "PORT B"
- note removed: "Page $00-$3F"
- note removed: "Page $00-$7F"
- note removed: "Page $40-$7F"
- note removed: "Page $80-$FF"
- note removed: "~{A0} drives RS1 (DDR, Port) A1 drives RS0 if two register pairs selected Else jumper selects RS0 high or low (Port A/B) $00 Port A DDR $01 Port A $02 Port B DDR (optional) $03 Port B (optional)"
- moved on the sheet: D?, J0A1, J0B1, J43, J?, U?, U?A, U?B
