File: kicad/Vega816/C64 Hardware/SID.kicad_sch (KiCad schematic)
At the start: 36 parts, among them J34 Audio Out, J38 Audio In, Q1 2SC1815, U28 74HC00, U64 6581_SID, U85 74HC00

Commit message: Big ol update
Parts:
- removed J34, J?: Audio Out, symbol Connector:AudioJack2
- removed J38, J?: Audio In, symbol Connector:AudioJack2_SwitchT
- removed J?: I/O Port, symbol Connector_Generic:Conn_02x20_Odd_Even
- added C34 (x2), C58 (x2), C65, C70, C71: 100n, symbol Device:C_Small
- added J26: Stereo Out, symbol Connector_Audio:AudioJack3
- added J48: Stereo In, symbol Connector_Audio:AudioJack3_SwitchTR
Connections:
- net POTX is gone; now on net GND: C34.1, C?.1, U64.24 (POT_X), U?.24 (POT_X)
- net R~{W} is gone; now on net ~{WR}: U?.7 (R/~{W})
- net CLK: now also U64.6 (ϕ2)
- net GND: now also U85.7 (GND), C34.2, C34.2, C58.2, C58.2, C65.2, C70.2, C71.2, J26.S, J48.RN, J48.S, J48.TN
- net VCC: now also U85.14 (VCC), C34.1, C34.1, C58.1, C58.1, C65.1, C70.1, C71.1
- net ~{RST}: now also U64.5 (~{RES})
- net at C?.1, R?.1: now also J48.T
- net at C35.1: now also J26.R
- net at C?.2, U?.2 (CAP1B): now also C?.1, U?.3 (CAP2A)
- net at C?.1: now also J26.T
- net at C30.1, R19.1: now also J48.R
- net at C28.2, U64.2 (CAP1B): now also C29.1, U64.3 (CAP2A)
- net ~{WR}: now reaches U64.7 (R/~{W})
Other:
- moved on the sheet: C28, C29, C30, C31, C32, C33, C34, C35, C?, J?, Q1, Q?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
