File: kicad/Vega816/Front Console/Front Console.kicad_sch (KiCad schematic)
At the start: 13 parts

Commit message: Big ol update
Parts:
- removed J?: VIA Port, symbol Connector_Generic:Conn_02x22_Odd_Even
- added C34: 100n, symbol Device:C_Small
Connections:
- net GND: now also C34.2
- net VCC: now also C34.1
