File: kicad/Vega816/IOBus/IOBus.kicad_sch (KiCad schematic)
At the start: 17 parts, among them J0A? Conn_02x40_Odd_Even, J0B? CPU, U1 74HC00, U92 74ACH138, U93 74ACH138, U94 74ACH138

Commit message: Big ol update
Parts:
- removed J?: I/O 0, symbol Connector_Generic:Conn_02x20_Odd_Even
- removed J?: I/O 1, symbol Connector_Generic:Conn_02x20_Odd_Even
- removed J?: I/O 3, symbol Connector_Generic:Conn_02x20_Odd_Even
- removed U94: 74ACH138, Package_DIP:DIP-14_W7.62mm_Socket, symbol Vega816:74ACH138
- added C34 (x4): 100n, symbol Device:C_Small
- added U2: 74HC139, symbol Vega816:74HC139
Connections:
- net A6: now also U2.14 (A0)
- net A7: now also U2.13 (A1)
- net CLK: now also J?.3 (Pin_3); no longer J?.7 (Pin_7)
- net GND: now also C34.2, C34.2, C34.2, C34.2, U2.8 (GND); no longer J?.2 (Pin_2), J?.2 (Pin_2), J?.2 (Pin_2), J?.3 (Pin_3)
- net R~{W}: no longer J?.9 (Pin_9)
- net VCC: now also J?.2 (Pin_2), C34.1, C34.1, C34.1, C34.1, U2.16 (VCC); no longer J?.1 (Pin_1)
- net ~{BANK0}: now also U92.4 (E1); no longer U92.5 (E2)
- net ~{CS0}: now also U2.12 (O0)
- net ~{CS1}: now also U2.11 (O1)
- net ~{CS2}: now also U2.10 (O2); no longer J?.11 (Pin_11)
- net ~{CS3}: now also U2.9 (O3)
- net ~{IRQ}: now also J?.5 (Pin_5)
- net ~{RD}: now also J?.7 (Pin_7)
- net ~{RST}: now also J?.1 (Pin_1); no longer J?.5 (Pin_5)
- net ~{WR}: now also J?.9 (Pin_9)
- net at JP?.2 (C): no longer U92.6 (E3)
- net at D?.1 (K), J?.1 (Pin_1), J?.11 (Pin_11)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: now also U2.15 (E)
- net at JP3.2 (C): no longer U92.4 (E1)
- new net: J?.2 (Pin_2), J?.2 (Pin_2)
- new net ~{CS}: J?.11 (Pin_11)
- no-connect marks 34 -> 27
Other:
- added sheet Dual SID (../C64 Hardware/SID.kicad_sch)
- added sheet Quad VIA (../System Devices/QuadVIA.kicad_sch)
- added sheet System Devices (../System Devices/System Devices.kicad_sch)
- note added: "Single Page IO Bus"
- note removed: "Single Page Quad IO Bus"
- moved on the sheet: D?, J0A?, J0B?, J?, JP3, JP?, U1A, U1B, U1C, U1D, U1E, U92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
