File: kicad/Vega816/System Devices/System Devices.kicad_sch (KiCad schematic)
At the start: 27 parts, among them J21 VIA Port, J22 VIA Port, J25 ACIA0, J26 ACIA1, J27 ACIA2, J36 ACIA3, U75 W65C22SxP, U76 W65C22SxP, U77 W65C51NxP, U80 W65C51NxP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

Commit message: Big ol update
Parts:
- removed C22, C23, C36, C37, C38, C39, C40, C41, C?: 100n, symbol Device:C_Small
- removed J21, J22, J?: VIA Port, symbol Connector_Generic:Conn_02x22_Odd_Even
- removed J25: ACIA0, symbol Connector_Generic:Conn_02x04_Odd_Even
- removed J26: ACIA1, symbol Connector_Generic:Conn_02x04_Odd_Even
- removed J27: ACIA2, symbol Connector_Generic:Conn_02x04_Odd_Even
- removed J36: ACIA3, symbol Connector_Generic:Conn_02x04_Odd_Even
- removed J?: I/O Port, symbol Connector_Generic:Conn_02x20_Odd_Even
- removed U75, U76, U?: W65C22SxP, Package_DIP:DIP-40_W15.24mm_Socket, symbol Vega816:W65C22SxP
- removed U77, U80, U83, U86: W65C51NxP, symbol BB816:W65C51NxP
- removed U81, U82: 74ACH138, Package_DIP:DIP-14_W7.62mm_Socket, symbol Vega816:74ACH138
- removed X2: 1.8432MHz, Oscillator:Oscillator_DIP-8, symbol Oscillator:CXO_DIP8
- added C34: 100n, symbol Device:C_Small
- added U2: 74HC139, symbol Vega816:74HC139
Connections:
- net A4: now also U2.2 (A0)
- net A5: now also U2.3 (A1)
- net GND: now also C34.2, U2.8 (GND)
- net VCC: now also C34.1, U2.13 (A1), U2.14 (A0), U2.15 (E), U2.16 (VCC)
- net ~{CS}: now also U2.1 (E)
- new net ~{UART3}: U2.7 (O3)
- new net ~{VIA0}: U2.4 (O0)
- new net ~{VIA1}: U2.5 (O1)
- new net ~{VIA2}: U2.6 (O2)
- no-connect marks 28 -> 4
Other:
- added sheet Dual PS2 (../Accessories/EaterPS2Interface.kicad_sch)
- added sheet Dual SPI (../Accessories/DualSPI.kicad_sch)
- added sheet Front Console (../Front Console/Front Console.kicad_sch)
- added sheet UART (XR88C192.kicad_sch)
- added sheet VIA0 (VIAPortNoConn.kicad_sch)
- added sheet VIA1 (VIAPortNoConn.kicad_sch)
- added sheet VIA2 (VIAPort.kicad_sch)
- note added: "Dev Device Service 0 W65C22S VIA Front Panel 1 W65C22S VIA Sysctrl Register 2 W65C22S VIA Dual PS2 3 XR88C192 UART Dual Channel RS-232/USB/I2C"
- note added: "System Devices"
- note removed: "System I/O 3 x VIA + 4 x ACIA"
- title: (none) -> System Devices (3xVIA, 1xXR88C192)
