File: kicad/Vega816/CPU Buffer/CPU Buffer.kicad_sch (KiCad schematic)
At the start: 72 parts, among them J1 VPA/VDA, J12 CPU, J14 VPA/VDA, J15 Conn_02x40_Odd_Even, J16 DMA, J17 VPA/VDA, J18 Conn_02x40_Odd_Even, J19 DMA, J2 Conn_02x40_Odd_Even, J20 DMA Shim ~{DMA0-3}, J3 DMA, J4 VPA/VDA, J5 Conn_02x40_Odd_Even, U10 74HC541, U11 74HC541, U12 74AHCT245, U13 74HC541, U14 74HC541, U15 74HC541, U16 74HC541, U17 74HC541, U18 74HC541, U19 74HC541, U20 74HC541, U21 74HC541, U22 74HC541, U23 74HC541, U24 74AHCT245, U25 74HC541, U26 74HC541, U27 74AHCT245, U28 74HC00, U29 74HC541, U30 74HC541, U31 74HC541, U32 74HC541, U33 74HC541, U34 74HC541

Commit message: push
Parts:
- J20: value DMA Shim ~{DMA0-3} -> DMA Shim
Connections:
- net CD0 is gone; now on net GND: J?.35 (Pin_35), U?.2 (A0)
- net CD1 is gone; now on net GND: J?.33 (Pin_33), U?.3 (A1)
- net CD2 is gone; now on net GND: J?.31 (Pin_31), U?.4 (A2)
- net CD3 is gone; now on net GND: J?.29 (Pin_29), U?.5 (A3)
- net CD4 is gone; now on net GND: J?.27 (Pin_27), U?.6 (A4)
- net CD5 is gone; now on net GND: J?.25 (Pin_25), U?.7 (A5)
- net CD6 is gone; now on net GND: J?.23 (Pin_23), U?.8 (A6)
- net CD7 is gone; now on net GND: J?.21 (Pin_21), U?.9 (A7)
- net R~{W}: no longer U12.1 (A->B), U24.1 (A->B), U27.1 (A->B), U?.1 (A->B)
- net ~{WR}: now also U12.1 (A->B), U24.1 (A->B), U27.1 (A->B), U?.1 (A->B)
Other:
- moved on the sheet: U27, U?

Commit message: Big ol update
Parts:
- J?: value CPU -> AUX
Changed lines of the file:
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@@
       (effects (font (size 1.27 1.27)))
     )
-    (property "Value" "CPU" (at 660.654 558.0888 0)
+    (property "Value" "AUX" (at 660.654 558.0888 0)
       (effects (font (size 3 3)))
     )
@@
     )
   )
+  (sheet_instances
+    (path "/" (page "1"))
+  )
 )
