File: kicad/Vega816/CPU Shim/CPU Shim.kicad_sch (KiCad schematic)
At the start: 33 parts, among them J5 DMA Bypass, J6 DMA Ctrl Reg, J8 ~{DMA0-3}, U1 74HC08, U6 74HC08, U8 74LS253, U9 74HC08

Commit message: push
Parts:
- removed J?: VP Shim, symbol Connector_Generic:Conn_02x08_Odd_Even
- removed RN?: 10K, Resistor_THT:R_Array_SIP9, symbol Device:R_Network08
- removed unit 5 of U1
- removed U? (x7): 74AHC32, Package_DIP:DIP-14_W7.62mm, symbol 74xx:74LS32
- added D? (x2): 1N4148, Diode_THT:D_DO-35_SOD27_P7.62mm_Horizontal, symbol Diode:1N4148
- added J31: ~{IRQ7_NMI}, symbol Connector_Generic:Conn_02x02_Odd_Even
- added J37: ~{IRQ IN}, symbol Connector_Generic:Conn_02x08_Odd_Even
- added R1, R15: 1K, symbol Device:R
- added R10, R13, R14, R20, R21, R22, R23, R3, R8, R9: 10K, symbol Device:R
- added U2: 74HC08, Package_DIP:DIP-14_W7.62mm_Socket, symbol Vega816:74HC08
- added unit 1 of U3
- added U5: 74HC32, Package_DIP:DIP-14_W7.62mm_Socket, symbol Vega816:74HC32
- added U6, U7: 74HC30, symbol Vega816:CD74HC30
- added U89: 74LS348, symbol 74xx:74LS348
- J6: value DMA Ctrl Reg -> DMA Sysctrl
- J8: value ~{DMA0-3} -> CPU Buffer
- J?: value DMA Ctrl -> DMA Controller
- gave numbers to parts that had none: 3
- renumbered U6 to U1, U9 to U2
Connections:
- net AA4 is gone; now on net A4: J?.11 (Pin_11), J?.8 (Pin_8), U9.4 (S1)
- net DMA3_SUB_LO is gone; now on net DMA2_SUB_LO: J6.13 (Pin_13), U8.3 (I3a)
- net DMA_REQ_PRI is gone; now on net DMA2_SUB_LO: J6.3 (Pin_3), J?.14 (Pin_14)
- net A1*A2*A3: now also U4.9; no longer U4.10
- net A16: now also U7.12
- net A17: now also U7.11
- net A18: now also U7.6
- net A19: now also U7.5
- net A20: now also U7.4
- net A21: now also U7.3
- net A22: now also U7.2
- net A23: now also U7.1; no longer J?.39 (Pin_39), J?.39 (Pin_39)
- net DMA_REQ_EN: now also U2.4; no longer U2.2, U2.4
- net E: now also U3.1, U3.2
- net GND: now also J37.10 (Pin_10), J37.12 (Pin_12), J37.14 (Pin_14), J37.16 (Pin_16), J37.2 (Pin_2), J37.3 (Pin_3), J37.4 (Pin_4), J37.6 (Pin_6), J37.8 (Pin_8), R1.2, R15.2, R8.1, U6.11, U89.11 (1), U89.8 (GND)
- net RDY_IN: now also U3.6; no longer U3.3
- net VCC: now also R10.2, R13.1, R14.1, R20.2, R21.2, R22.2, R23.2, R3.2, R8.2, R9.2, U89.16 (VCC)
- net VP: now also U3.11, U4.10; no longer U3.3, U4.9
- net VP_REQ: now also U89.5 (EI)
- net Y1: now also U89.9 (A0)
- net Y2: now also U89.7 (A1)
- net Y3: now also U89.6 (A2)
- net ~{BANK0}: now also U7.8
- net ~{IRQ}: now also D?.1 (K), D?.2 (A), U6.8
- net ~{NMI}: now also D?.1 (K), D?.2 (A), U5.3
- net ~{VP}: now also U3.12, U3.13; no longer U3.1, U3.2
- new net: U5.6, U6.12, U89.10 (0)
- new net: U1.11, U3.4, U3.5
- new net: J31.3 (Pin_3), R14.2, U5.5
- new net: U2.5, U3.3
- new net: U2.2, U2.4, U2.6
- new net: J31.2 (Pin_2), R1.1
- new net: J31.1 (Pin_1), R13.2, U5.1
- new net: J31.4 (Pin_4), R15.1
- new net ~{IRQ0}: J37.15 (Pin_15), R23.1, U6.1, U89.4 (7)
- new net ~{IRQ1}: J37.13 (Pin_13), R22.1, U6.2, U89.3 (6)
- new net ~{IRQ2}: J37.11 (Pin_11), R21.1, U6.3, U89.2 (5)
- new net ~{IRQ3}: J37.9 (Pin_9), R20.1, U6.4, U89.1 (4)
- new net ~{IRQ4}: J37.7 (Pin_7), R10.1, U6.5, U89.13 (3)
- new net ~{IRQ5}: J37.5 (Pin_5), R9.1, U6.6, U89.12 (2)
- new net ~{IRQ7}: J37.1 (Pin_1), R3.1, U5.2, U5.4
- new net ~{WR}: J?.39 (Pin_39), J?.39 (Pin_39)
- no-connect marks 2 -> 4
Other:
- note added: "DMA Control"
- note added: "VPB Rewrite"
- note removed: "DMA Control Shim"
- note removed: "Vector Pull Rewrite Shim"
- moved on the sheet: J5, J6, J8, J?, R?, U1A, U1B, U1C, U1D, U2A, U2B, U3B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

Commit message: Big ol update
Parts:
- removed U5: 74HC32, Package_DIP:DIP-14_W7.62mm_Socket, symbol Vega816:74HC32
- removed U6, U7: 74HC30, symbol Vega816:CD74HC30
- added U10, U4: 74AHC32, Package_DIP:DIP-14_W7.62mm, symbol 74xx:74LS32
Connections:
- net A22: no longer J5.3 (Pin_3), J?.55 (Pin_55), U8.7 (Za)
- net A23: no longer J5.1 (Pin_1), J?.53 (Pin_53), U8.9 (Zb)
- net A4: no longer J?.11 (Pin_11), J?.8 (Pin_8), U9.4 (S1)
- net ~{BANK0}: now also U10.2; no longer J?.41 (Pin_41)
- net ~{IRQ7}: now also J31.2 (Pin_2), J31.4 (Pin_4)
- net ~{IRQ}: now also R14.2, U89.14 (GS)
- net ~{NMI}: now also J31.1 (Pin_1), R13.2
- net at U89.10 (0): now also J31.3 (Pin_3)
- net at R1.1: no longer J31.2 (Pin_2)
- net at R15.1: no longer J31.4 (Pin_4)
- new net: U10.1, U4.8
- new net A22A: J5.3 (Pin_3), J?.55 (Pin_55), U4.9, U8.7 (Za)
- new net A23A: J5.1 (Pin_1), J?.53 (Pin_53), U4.10, U8.9 (Zb)
- new net AA4: J?.11 (Pin_11), J?.8 (Pin_8), U9.4 (S1)
- new net ~{BANK0A}: J?.41 (Pin_41), U10.3
- no-connect marks 4 -> 2
Other:
- note added: "BB816 W65C816 Breakout Rev. A.27"
- note added: "CPU Shim for BB816 W65816 Breakout"
- note added: "DMA Request Settings DMA Enable (This CPU) Priority (This CPU can pause others) A23/A22 bank selection for DMA channels 1-3 (per channel)"
- note added: "IRQ Priority"
- note added: "IRQ VP Detection"
- note added: "Output from DMA Controller: 1-of-4 DMA Channel Selection (Active Low, may be none). Input to DMA Controller: Requested channel (high bit, low bit) Priority Bit (can pause other Bus Masters)."
- note added: "Output to CPU Buffer: 1-of-4 DMA Channel Selection (Active Low)"
- note added: "To CPU Buffer"
- note added: "Vector Address Rewrite"
- note added: "~{VPB}+~{IRQ} Rewrite"
- note removed: "CPU Shim"
- note removed: "VPB Rewrite"
- moved on the sheet: D?, J31, J37, J5, J6, J8, J?, R1, R10, R13, R14, R15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
