File: kicad/Vega816/Sysctrl Registers/Sysctrl Registers.kicad_sch (KiCad schematic)
At the start: 68 parts, among them J1 Sysctrl $7, J10 Sysctrl $A, J102 VIA Port, J11 Sysctrl $B, J12 Sysctrl $C, J13 Sysctrl $D, J16 Sysctrl $E, J17 Sysctrl $F, J18 Sysctrl $8, J2 Sysctrl $6, J3 Sysctrl $5, J4 Sysctrl $4, J5 Sysctrl $3, J6 Sysctrl $2, J7 Sysctrl $1, J8 Sysctrl $0, J9 Sysctrl $9, U11 74HC32, U15 74HC259, U17 74HC373, U18 74HC32, U2 74ACH138, U20 74HC259, U21 74HC02, U22 74HC32, U3 74ACH138, U30 74HC259, U32 74HC32, U4 74HC04, U47 74HC259, U48 74HC373, U49 74HC32, U5 74HC259, U51 74HC259, U52 74HC02, U53 74HC32, U55 74HC259, U57 74HC32, U59 74HC259, U6 74HC32, U60 74HC373, U61 74HC02, U63 74HC373, U65 74HC02, U67 74HC373, U68 74HC02, U7 74HC02, U70 74HC373, U71 74HC02, U73 74HC373, U74 74HC02

Commit message: Big ol update
Parts:
- removed J1: Sysctrl $7, Connector_PinHeader_2.54mm:PinHeader_2x08_P2.54mm_Vertical, symbol Vega816:Conn_02x08_Odd_Even
- removed J102: VIA Port, symbol Connector_Generic:Conn_02x22_Odd_Even
- removed J12: Sysctrl $C, Connector_PinHeader_2.54mm:PinHeader_2x08_P2.54mm_Vertical, symbol Vega816:Conn_02x08_Odd_Even
- removed J13: Sysctrl $D, Connector_PinHeader_2.54mm:PinHeader_2x08_P2.54mm_Vertical, symbol Vega816:Conn_02x08_Odd_Even
- removed J16: Sysctrl $E, Connector_PinHeader_2.54mm:PinHeader_2x08_P2.54mm_Vertical, symbol Vega816:Conn_02x08_Odd_Even
- removed J18: Sysctrl $8, Connector_PinHeader_2.54mm:PinHeader_2x08_P2.54mm_Vertical, symbol Vega816:Conn_02x08_Odd_Even
- removed J2: Sysctrl $6, Connector_PinHeader_2.54mm:PinHeader_2x08_P2.54mm_Vertical, symbol Vega816:Conn_02x08_Odd_Even
- removed J3: Sysctrl $5, Connector_PinHeader_2.54mm:PinHeader_2x08_P2.54mm_Vertical, symbol Vega816:Conn_02x08_Odd_Even
- removed J4: Sysctrl $4, Connector_PinHeader_2.54mm:PinHeader_2x08_P2.54mm_Vertical, symbol Vega816:Conn_02x08_Odd_Even
- removed J5: Sysctrl $3, Connector_PinHeader_2.54mm:PinHeader_2x08_P2.54mm_Vertical, symbol Vega816:Conn_02x08_Odd_Even
- removed J6: Sysctrl $2, Connector_PinHeader_2.54mm:PinHeader_2x08_P2.54mm_Vertical, symbol Vega816:Conn_02x08_Odd_Even
- removed U11, U18, U22, U32, U6: 74HC32, Package_DIP:DIP-14_W7.62mm_Socket, symbol Vega816:74HC32
- removed U15, U20, U30, U47, U5, U51, U55: 74HC259, symbol Vega816:74HC259
- removed U17, U48, U60, U63, U67, U70, U?: 74HC373, symbol 74xx:74HC373
- removed U21, U52, U61, U65, U68, U7, U71: 74HC02, symbol 74xx:74HC02
- removed U? (x14): 74HC541, symbol Vega816:74HC541
- added C150, C151, C152, C153, C154, C155, C156, C157, C158, C159, C160, C161, C162, C163, C164, C165, C166, C167, C168, C169, C170, C171, C172, C173, C174, C175, C176, C177, C178, C179, C180, C181, C182, C183, C184, C185, C186: 100n, symbol Device:C_Small
- added J38: Sysctrl $2, Connector_PinHeader_2.54mm:PinHeader_2x08_P2.54mm_Vertical, symbol Vega816:Conn_02x08_Odd_Even
- added J49: Sysctrl $D, Connector_PinHeader_2.54mm:PinHeader_2x08_P2.54mm_Vertical, symbol Vega816:Conn_02x08_Odd_Even
- added J50, J51: Sysctrl $8, Connector_PinHeader_2.54mm:PinHeader_2x08_P2.54mm_Vertical, symbol Vega816:Conn_02x08_Odd_Even
- added J52: Sysctrl $6, Connector_PinHeader_2.54mm:PinHeader_2x08_P2.54mm_Vertical, symbol Vega816:Conn_02x08_Odd_Even
- added J53: Sysctrl $9, Connector_PinHeader_2.54mm:PinHeader_2x08_P2.54mm_Vertical, symbol Vega816:Conn_02x08_Odd_Even
- added J54: Sysctrl $5, Connector_PinHeader_2.54mm:PinHeader_2x08_P2.54mm_Vertical, symbol Vega816:Conn_02x08_Odd_Even
- added J55: Sysctrl $A, Connector_PinHeader_2.54mm:PinHeader_2x08_P2.54mm_Vertical, symbol Vega816:Conn_02x08_Odd_Even
- added J56: Sysctrl $4, Connector_PinHeader_2.54mm:PinHeader_2x08_P2.54mm_Vertical, symbol Vega816:Conn_02x08_Odd_Even
- added J57: Sysctrl $B, Connector_PinHeader_2.54mm:PinHeader_2x08_P2.54mm_Vertical, symbol Vega816:Conn_02x08_Odd_Even
- added U101, U108, U116, U122, U54, U62, U68: 74HC373, symbol 74xx:74HC373
- added U102, U109, U117, U47, U69: 74HC32, Package_DIP:DIP-14_W7.62mm_Socket, symbol Vega816:74HC32
- added U105, U112, U119, U50, U56, U65, U71: 74HC259, symbol Vega816:74HC259
- added U106, U113, U120, U51, U60, U66, U90: 74HC02, symbol 74xx:74HC02
- added U? (x14): 74HC541, symbol Vega816:74HC541
- J10: value Sysctrl $A -> Sysctrl $3
- J11: value Sysctrl $B -> Sysctrl $C
- J9: value Sysctrl $9 -> Sysctrl $E
Connections:
- net CA2_~{LE} is gone; now on net CA2: U74.3
- net PB0_A0 is gone; now on net PA1: U59.1 (A0)
- net PB1_A1 is gone; now on net PA2: U59.2 (A1)
- net PB2_A2 is gone; now on net PA3: U59.3 (A2)
- net GND: now also J7.10 (Pin_10), J7.12 (Pin_12), J7.14 (Pin_14), J7.16 (Pin_16), J7.2 (Pin_2), J7.4 (Pin_4), J7.6 (Pin_6), J7.8 (Pin_8), C150.2, C151.2, C152.2, C153.2, C154.2, C155.2, C156.2, C157.2, C158.2, C159.2, C160.2, C161.2, C162.2, C163.2, C164.2, C165.2, C166.2, C167.2, C168.2, C169.2, C170.2, C171.2, C172.2, C173.2, C174.2, C175.2, C176.2, C177.2, C178.2, C179.2, C180.2, C181.2, C182.2, C183.2, C184.2, C185.2, C186.2, J38.10 (Pin_10), J38.12 (Pin_12), J38.14 (Pin_14), J38.16 (Pin_16), J38.2 (Pin_2), J38.4 (Pin_4), J38.6 (Pin_6), J38.8 (Pin_8), J49.10 (Pin_10), J49.12 (Pin_12), J49.14 (Pin_14), J49.16 (Pin_16), J49.2 (Pin_2), J49.4 (Pin_4), J49.6 (Pin_6), J49.8 (Pin_8), J50.10 (Pin_10), J50.12 (Pin_12), J50.14 (Pin_14), J50.16 (Pin_16), J50.2 (Pin_2), J50.4 (Pin_4), J50.6 (Pin_6), J50.8 (Pin_8), J51.10 (Pin_10), J51.12 (Pin_12), J51.14 (Pin_14), J51.16 (Pin_16), J51.2 (Pin_2), J51.4 (Pin_4), J51.6 (Pin_6), J51.8 (Pin_8), J52.10 (Pin_10), J52.12 (Pin_12), J52.14 (Pin_14), J52.16 (Pin_16), J52.2 (Pin_2), J52.4 (Pin_4), J52.6 (Pin_6), J52.8 (Pin_8), J53.10 (Pin_10), J53.12 (Pin_12), J53.14 (Pin_14), J53.16 (Pin_16), J53.2 (Pin_2), J53.4 (Pin_4), J53.6 (Pin_6), J53.8 (Pin_8), J54.10 (Pin_10), J54.12 (Pin_12), J54.14 (Pin_14), J54.16 (Pin_16), J54.2 (Pin_2), J54.4 (Pin_4), J54.6 (Pin_6), J54.8 (Pin_8), J55.10 (Pin_10), J55.12 (Pin_12), J55.14 (Pin_14), J55.16 (Pin_16), J55.2 (Pin_2), J55.4 (Pin_4), J55.6 (Pin_6), J55.8 (Pin_8), J56.10 (Pin_10), J56.12 (Pin_12), J56.14 (Pin_14), J56.16 (Pin_16), J56.2 (Pin_2), J56.4 (Pin_4), J56.6 (Pin_6), J56.8 (Pin_8), J57.10 (Pin_10), J57.12 (Pin_12), J57.14 (Pin_14), J57.16 (Pin_16), J57.2 (Pin_2), J57.4 (Pin_4), J57.6 (Pin_6), J57.8 (Pin_8), U101.1 (OE), U101.10 (GND), U105.8 (GND), U108.1 (OE), U108.10 (GND), U112.8 (GND), U116.1 (OE), U116.10 (GND), U119.8 (GND), U122.1 (OE), U122.10 (GND), U50.8 (GND), U54.1 (OE), U54.10 (GND), U56.8 (GND), U62.1 (OE), U62.10 (GND), U65.8 (GND), U68.1 (OE), U68.10 (GND), U71.8 (GND), U?.10 (GND), U?.10 (GND), U?.10 (GND), U?.10 (GND), U?.10 (GND), U?.10 (GND), U?.10 (GND), U?.10 (GND), U?.10 (GND), U?.10 (GND), U?.10 (GND), U?.10 (GND), U?.10 (GND), U?.10 (GND)
- net PA1: now also U101.4 (D1), U105.1 (A0), U108.4 (D1), U112.1 (A0), U116.4 (D1), U119.1 (A0), U122.4 (D1), U50.1 (A0), U54.4 (D1), U56.1 (A0), U62.4 (D1), U65.1 (A0), U68.4 (D1), U71.1 (A0), U?.12 (Y6), U?.12 (Y6), U?.12 (Y6), U?.12 (Y6), U?.12 (Y6), U?.12 (Y6), U?.12 (Y6), U?.17 (Y1), U?.17 (Y1), U?.17 (Y1), U?.17 (Y1), U?.17 (Y1), U?.17 (Y1), U?.17 (Y1)
- net PA2: now also U101.7 (D2), U105.2 (A1), U108.7 (D2), U112.2 (A1), U116.7 (D2), U119.2 (A1), U122.7 (D2), U50.2 (A1), U54.7 (D2), U56.2 (A1), U62.7 (D2), U65.2 (A1), U68.7 (D2), U71.2 (A1), U?.13 (Y5), U?.13 (Y5), U?.13 (Y5), U?.13 (Y5), U?.13 (Y5), U?.13 (Y5), U?.13 (Y5), U?.16 (Y2), U?.16 (Y2), U?.16 (Y2), U?.16 (Y2), U?.16 (Y2), U?.16 (Y2), U?.16 (Y2)
- net PA3: now also U101.8 (D3), U105.3 (A2), U108.8 (D3), U112.3 (A2), U116.8 (D3), U119.3 (A2), U122.8 (D3), U50.3 (A2), U54.8 (D3), U56.3 (A2), U62.8 (D3), U65.3 (A2), U68.8 (D3), U71.3 (A2), U?.14 (Y4), U?.14 (Y4), U?.14 (Y4), U?.14 (Y4), U?.14 (Y4), U?.14 (Y4), U?.14 (Y4), U?.15 (Y3), U?.15 (Y3), U?.15 (Y3), U?.15 (Y3), U?.15 (Y3), U?.15 (Y3), U?.15 (Y3)
- net PA4: now also U101.13 (D4), U108.13 (D4), U116.13 (D4), U122.13 (D4), U54.13 (D4), U62.13 (D4), U68.13 (D4), U?.14 (Y4), U?.14 (Y4), U?.14 (Y4), U?.14 (Y4), U?.14 (Y4), U?.14 (Y4), U?.14 (Y4), U?.15 (Y3), U?.15 (Y3), U?.15 (Y3), U?.15 (Y3), U?.15 (Y3), U?.15 (Y3), U?.15 (Y3)
- net PA5: now also U101.14 (D5), U108.14 (D5), U116.14 (D5), U122.14 (D5), U54.14 (D5), U62.14 (D5), U68.14 (D5), U?.13 (Y5), U?.13 (Y5), U?.13 (Y5), U?.13 (Y5), U?.13 (Y5), U?.13 (Y5), U?.13 (Y5), U?.16 (Y2), U?.16 (Y2), U?.16 (Y2), U?.16 (Y2), U?.16 (Y2), U?.16 (Y2), U?.16 (Y2)
- net PA6: now also U101.17 (D6), U108.17 (D6), U116.17 (D6), U122.17 (D6), U54.17 (D6), U62.17 (D6), U68.17 (D6), U?.12 (Y6), U?.12 (Y6), U?.12 (Y6), U?.12 (Y6), U?.12 (Y6), U?.12 (Y6), U?.12 (Y6), U?.17 (Y1), U?.17 (Y1), U?.17 (Y1), U?.17 (Y1), U?.17 (Y1), U?.17 (Y1), U?.17 (Y1)
- net PA7: now also U101.18 (D7), U108.18 (D7), U116.18 (D7), U122.18 (D7), U54.18 (D7), U62.18 (D7), U68.18 (D7), U?.11 (Y7), U?.11 (Y7), U?.11 (Y7), U?.11 (Y7), U?.11 (Y7), U?.11 (Y7), U?.11 (Y7), U?.18 (Y0), U?.18 (Y0), U?.18 (Y0), U?.18 (Y0), U?.18 (Y0), U?.18 (Y0), U?.18 (Y0)
- net VCC: now also C150.1, C151.1, C152.1, C153.1, C154.1, C155.1, C156.1, C157.1, C158.1, C159.1, C160.1, C161.1, C162.1, C163.1, C164.1, C165.1, C166.1, C167.1, C168.1, C169.1, C170.1, C171.1, C172.1, C173.1, C174.1, C175.1, C176.1, C177.1, C178.1, C179.1, C180.1, C181.1, C182.1, C183.1, C184.1, C185.1, C186.1, U101.20 (VCC), U105.16 (VCC), U108.20 (VCC), U112.16 (VCC), U116.20 (VCC), U119.16 (VCC), U122.20 (VCC), U50.16 (VCC), U54.20 (VCC), U56.16 (VCC), U62.20 (VCC), U65.16 (VCC), U68.20 (VCC), U71.16 (VCC), U?.20 (VCC), U?.20 (VCC), U?.20 (VCC), U?.20 (VCC), U?.20 (VCC), U?.20 (VCC), U?.20 (VCC), U?.20 (VCC), U?.20 (VCC), U?.20 (VCC), U?.20 (VCC), U?.20 (VCC), U?.20 (VCC), U?.20 (VCC)
- net ~{RD}: now reaches U4.2, U?.19 (G2), U?.19 (G2)
- net ~{RD}: now also U?.19 (G2), U?.19 (G2), U?.19 (G2), U?.19 (G2), U?.19 (G2), U?.19 (G2), U?.19 (G2), U?.19 (G2), U?.19 (G2), U?.19 (G2), U?.19 (G2), U?.19 (G2), U?.19 (G2), U?.19 (G2)
- net at U2.10 (O5): now also U109.2, U?.1 (G1)
- net at U2.12 (O3): now also U49.2, U?.1 (G1)
- net at U2.9 (O6): now also U102.2, U?.1 (G1)
- net at J10.1 (Pin_1): now also U56.12 (Q7), U?.9 (A7)
- net at J10.11 (Pin_11): now also U56.6 (Q2), U?.4 (A2)
- net at J10.13 (Pin_13): now also U56.5 (Q1), U?.3 (A1)
- net at J10.15 (Pin_15): now also U56.4 (Q0), U?.2 (A0)
- net at J10.3 (Pin_3): now also U56.11 (Q6), U?.8 (A6)
- net at J10.5 (Pin_5): now also U56.10 (Q5), U?.7 (A5)
- net at J10.7 (Pin_7): now also U56.9 (Q4), U?.6 (A4)
- net at J10.9 (Pin_9): now also U56.7 (Q3), U?.5 (A3)
- net at J7.1 (Pin_1): now also U50.12 (Q7), U?.9 (A7)
- net at J7.11 (Pin_11): now also U50.6 (Q2), U?.4 (A2)
- net at J7.13 (Pin_13): now also U50.5 (Q1), U?.3 (A1)
- net at J7.15 (Pin_15): now also U50.4 (Q0), U?.2 (A0)
- net at J7.3 (Pin_3): now also U50.11 (Q6), U?.8 (A6)
- net at J7.5 (Pin_5): now also U50.10 (Q5), U?.7 (A5)
- net at J7.7 (Pin_7): now also U50.9 (Q4), U?.6 (A4)
- net at J7.9 (Pin_9): now also U50.7 (Q3), U?.5 (A3)
- net at U3.13 (O2): now also U113.2, U?.1 (G1)
- net at J9.9 (Pin_9): now also U54.12 (O4), U?.6 (A4)
- net at J9.11 (Pin_11): now also U54.15 (O5), U?.7 (A5)
- net at J9.13 (Pin_13): now also U54.16 (O6), U?.8 (A6)
- net at J9.15 (Pin_15): now also U54.19 (O7), U?.9 (A7)
- net at J9.1 (Pin_1): now also U54.2 (O0), U?.2 (A0)
- net at J9.3 (Pin_3): now also U54.5 (O1), U?.3 (A1)
- net at J9.5 (Pin_5): now also U54.6 (O2), U?.4 (A2)
- net at J9.7 (Pin_7): now also U54.9 (O3), U?.5 (A3)
- net at U3.10 (O5): now also U66.2, U?.1 (G1)
- net at U3.11 (O4): now also U60.2, U?.1 (G1)
- net at U3.12 (O3): now also U120.2, U?.1 (G1)
- net at U3.14 (O1): now also U106.2, U?.1 (G1)
- net at U3.15 (O0): now also U90.2, U?.1 (G1)
- net at U3.9 (O6): now also U51.2, U?.1 (G1)
- net at U2.14 (O1): now also U47.2, U?.1 (G1); no longer U53.2
- net at J11.9 (Pin_9): now also U62.12 (O4), U?.6 (A4)
- net at J11.11 (Pin_11): now also U62.15 (O5), U?.7 (A5)
- net at J11.13 (Pin_13): now also U62.16 (O6), U?.8 (A6)
- net at J11.15 (Pin_15): now also U62.19 (O7), U?.9 (A7)
- net at J11.1 (Pin_1): now also U62.2 (O0), U?.2 (A0)
- net at J11.3 (Pin_3): now also U62.5 (O1), U?.3 (A1)
- net at J11.5 (Pin_5): now also U62.6 (O2), U?.4 (A2)
- net at J11.7 (Pin_7): now also U62.9 (O3), U?.5 (A3)
- net CA2: now reaches U53.1, U57.1
- net CA2: now also U49.1, U102.1, U106.3, U109.1, U113.3, U117.1, U120.3, U47.1, U51.3, U60.3, U66.3, U69.1, U90.3
- net at U53.3: now also U65.14 (E)
- net at U2.13 (O2): now also U53.2, U?.1 (G1); no longer U49.2
- net at U49.3: now also U56.14 (E)
- net at U2.11 (O4): now also U117.2, U?.1 (G1)
- net at U2.7 (O7): now also U69.2, U?.1 (G1)
- net CB2_CLR renamed CB2
- net CB2: now also U105.15 (Clr), U112.15 (Clr), U119.15 (Clr), U50.15 (Clr), U56.15 (Clr), U65.15 (Clr), U71.15 (Clr)
- net PA0_D renamed PA0
- net PA0: now also U101.3 (D0), U105.13 (D), U108.3 (D0), U112.13 (D), U116.3 (D0), U119.13 (D), U122.3 (D0), U50.13 (D), U54.3 (D0), U56.13 (D), U62.3 (D0), U65.13 (D), U68.3 (D0), U71.13 (D), U?.11 (Y7), U?.11 (Y7), U?.11 (Y7), U?.11 (Y7), U?.11 (Y7), U?.11 (Y7), U?.11 (Y7), U?.18 (Y0), U?.18 (Y0), U?.18 (Y0), U?.18 (Y0), U?.18 (Y0), U?.18 (Y0), U?.18 (Y0)
- net PB3_A3 renamed PB0
- net PB4_A4 renamed PB1
- net PB5_A5 renamed PB2
- net PB6_A6 renamed PB3
- net PB7_RD renamed PB4
- new net: J56.1 (Pin_1), U119.12 (Q7), U?.9 (A7)
- new net: J56.11 (Pin_11), U119.6 (Q2), U?.4 (A2)
- new net: J56.13 (Pin_13), U119.5 (Q1), U?.3 (A1)
- new net: J56.15 (Pin_15), U119.4 (Q0), U?.2 (A0)
- new net: J56.3 (Pin_3), U119.11 (Q6), U?.8 (A6)
- new net: J56.5 (Pin_5), U119.10 (Q5), U?.7 (A5)
- new net: J56.7 (Pin_7), U119.9 (Q4), U?.6 (A4)
- new net: J56.9 (Pin_9), U119.7 (Q3), U?.5 (A3)
- new net: U66.1, U68.11 (LE)
- new net: J49.9 (Pin_9), U68.12 (O4), U?.6 (A4)
- new net: J49.11 (Pin_11), U68.15 (O5), U?.7 (A5)
- new net: J49.13 (Pin_13), U68.16 (O6), U?.8 (A6)
- new net: J49.15 (Pin_15), U68.19 (O7), U?.9 (A7)
- new net: J49.1 (Pin_1), U68.2 (O0), U?.2 (A0)
- new net: J49.3 (Pin_3), U68.5 (O1), U?.3 (A1)
- new net: J49.5 (Pin_5), U68.6 (O2), U?.4 (A2)
- new net: J49.7 (Pin_7), U68.9 (O3), U?.5 (A3)
- new net: J53.1 (Pin_1), U108.2 (O0), U?.2 (A0)
- new net: J53.11 (Pin_11), U108.15 (O5), U?.7 (A5)
- new net: J53.13 (Pin_13), U108.16 (O6), U?.8 (A6)
- new net: J53.15 (Pin_15), U108.19 (O7), U?.9 (A7)
- new net: J53.3 (Pin_3), U108.5 (O1), U?.3 (A1)
- new net: J53.5 (Pin_5), U108.6 (O2), U?.4 (A2)
- new net: J53.7 (Pin_7), U108.9 (O3), U?.5 (A3)
- new net: J53.9 (Pin_9), U108.12 (O4), U?.6 (A4)
- new net: J52.5 (Pin_5), U105.10 (Q5), U?.7 (A5)
- new net: J52.3 (Pin_3), U105.11 (Q6), U?.8 (A6)
- new net: J52.1 (Pin_1), U105.12 (Q7), U?.9 (A7)
- new net: U102.3, U105.14 (E)
- new net: J52.15 (Pin_15), U105.4 (Q0), U?.2 (A0)
- new net: J52.13 (Pin_13), U105.5 (Q1), U?.3 (A1)
- new net: J52.11 (Pin_11), U105.6 (Q2), U?.4 (A2)
- new net: J52.9 (Pin_9), U105.7 (Q3), U?.5 (A3)
- new net: J52.7 (Pin_7), U105.9 (Q4), U?.6 (A4)
- new net: J55.1 (Pin_1), U116.2 (O0), U?.2 (A0)
- new net: J55.3 (Pin_3), U116.5 (O1), U?.3 (A1)
- new net: J55.5 (Pin_5), U116.6 (O2), U?.4 (A2)
- new net: J55.7 (Pin_7), U116.9 (O3), U?.5 (A3)
- new net: J55.9 (Pin_9), U116.12 (O4), U?.6 (A4)
- new net: J55.11 (Pin_11), U116.15 (O5), U?.7 (A5)
- new net: J55.13 (Pin_13), U116.16 (O6), U?.8 (A6)
- new net: J55.15 (Pin_15), U116.19 (O7), U?.9 (A7)
- new net: J57.1 (Pin_1), U122.2 (O0), U?.2 (A0)
- new net: J57.11 (Pin_11), U122.15 (O5), U?.7 (A5)
- new net: J57.13 (Pin_13), U122.16 (O6), U?.8 (A6)
- new net: J57.15 (Pin_15), U122.19 (O7), U?.9 (A7)
- new net: J57.3 (Pin_3), U122.5 (O1), U?.3 (A1)
- new net: J57.5 (Pin_5), U122.6 (O2), U?.4 (A2)
- new net: J57.7 (Pin_7), U122.9 (O3), U?.5 (A3)
- new net: J57.9 (Pin_9), U122.12 (O4), U?.6 (A4)
- new net: U101.11 (LE), U90.1
- new net: J51.9 (Pin_9), U101.12 (O4), U?.6 (A4)
- new net: J51.11 (Pin_11), U101.15 (O5), U?.7 (A5)
- new net: J51.13 (Pin_13), U101.16 (O6), U?.8 (A6)
- new net: J51.15 (Pin_15), U101.19 (O7), U?.9 (A7)
- new net: J51.1 (Pin_1), U101.2 (O0), U?.2 (A0)
- new net: J51.3 (Pin_3), U101.5 (O1), U?.3 (A1)
- new net: J51.5 (Pin_5), U101.6 (O2), U?.4 (A2)
- new net: J51.7 (Pin_7), U101.9 (O3), U?.5 (A3)
- new net: J54.15 (Pin_15), U112.4 (Q0), U?.2 (A0)
- new net: J54.13 (Pin_13), U112.5 (Q1), U?.3 (A1)
- new net: J54.11 (Pin_11), U112.6 (Q2), U?.4 (A2)
- new net: J54.9 (Pin_9), U112.7 (Q3), U?.5 (A3)
- new net: J54.7 (Pin_7), U112.9 (Q4), U?.6 (A4)
- new net: J54.5 (Pin_5), U112.10 (Q5), U?.7 (A5)
- new net: J54.3 (Pin_3), U112.11 (Q6), U?.8 (A6)
- new net: J54.1 (Pin_1), U112.12 (Q7), U?.9 (A7)
- new net: U47.3, U50.14 (E)
- new net: U120.1, U122.11 (LE)
- new net: U69.3, U71.14 (E)
- new net: U109.3, U112.14 (E)
- new net: U60.1, U62.11 (LE)
- new net: U113.1, U116.11 (LE)
- new net: U117.3, U119.14 (E)
- new net: J50.15 (Pin_15), U71.4 (Q0), U?.2 (A0)
- new net: J50.13 (Pin_13), U71.5 (Q1), U?.3 (A1)
- new net: J50.11 (Pin_11), U71.6 (Q2), U?.4 (A2)
- new net: J50.9 (Pin_9), U71.7 (Q3), U?.5 (A3)
- new net: J50.7 (Pin_7), U71.9 (Q4), U?.6 (A4)
- new net: J50.5 (Pin_5), U71.10 (Q5), U?.7 (A5)
- new net: J50.3 (Pin_3), U71.11 (Q6), U?.8 (A6)
- new net: J50.1 (Pin_1), U71.12 (Q7), U?.9 (A7)
- new net: U106.1, U108.11 (LE)
- new net: U51.1, U54.11 (LE)
- new net: J38.15 (Pin_15), U65.4 (Q0), U?.2 (A0)
- new net: J38.13 (Pin_13), U65.5 (Q1), U?.3 (A1)
- new net: J38.11 (Pin_11), U65.6 (Q2), U?.4 (A2)
- new net: J38.9 (Pin_9), U65.7 (Q3), U?.5 (A3)
- new net: J38.7 (Pin_7), U65.9 (Q4), U?.6 (A4)
- new net: J38.5 (Pin_5), U65.10 (Q5), U?.7 (A5)
- new net: J38.3 (Pin_3), U65.11 (Q6), U?.8 (A6)
- new net: J38.1 (Pin_1), U65.12 (Q7), U?.9 (A7)
- no-connect marks 2 -> 0
Other:
- moved on the sheet: J17, J8, U2, U3, U4A, U57A, U59, U73, U74A, U?

Commit message: Strip
Parts:
- renumbered C158 to C34, C165 to C34, C159 to C34, C152 to C34, C153 to C34, C179 to C40, C171 to C40, C174 to C40, C175 to C40, C172 to C58, C160 to C58, C154 to C58, C173 to C59, C182 to C59, C186 to C60, C185 to C60, C166 to C60, C176 to C60, C157 to C61, C168 to C61, C161 to C61, C184 to C61, C180 to C61, C151 to C61, C156 to C61, C181 to C61, C178 to C61, C155 to C61, C150 to C61, C169 to C61, C183 to C68, C170 to C69, C164 to C95, C163 to C?, C162 to C?, C167 to C?, C177 to C?

Commit message: wrtolei
Parts:
- gave numbers to parts that had none: 4
- renumbered C61 to C150, C61 to C151, C34 to C152, C34 to C153, C58 to C154, C61 to C155, C61 to C156, C61 to C157, C34 to C158, C34 to C159, C58 to C160, C61 to C161, C95 to C164, C34 to C165, C60 to C166, C61 to C168, C61 to C169, C69 to C170, C40 to C171, C58 to C172, C59 to C173, C40 to C174, C40 to C175, C60 to C176, C61 to C178, C40 to C179, C61 to C180, C61 to C181, C59 to C182, C68 to C183, C61 to C184, C60 to C185, C60 to C186
