File: kicad/Vega816/VectorPullRewrite/VectorPullRewrite.kicad_sch (KiCad schematic)
At the start: 28 parts, among them J10 ~{IRQ7_NMI}, J12 Conn_02x40_Odd_Even, J13 DMA, J5 Conn_02x40_Odd_Even, J6 CPU, J7 VP Bypass, J9 ~{IRQ IN}, U1 74HC08, U3 74HC283, U4 74HC00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

Commit message: vpb
Parts:
- added U2: 74HC74, symbol 74xx:74HC74
Connections:
- net VP: no longer names the net of U4.3
- net VP: now also U2.1 (~{R}); no longer U1.10
Changed lines of the file:
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@@
+    (stroke (width 0) (type default))
+  )
+  (wire (pts (xy 59.69 379.73) (xy 59.69 384.81))
     (stroke (width 0) (type default))
   )
@@
     (stroke (width 0) (type default))
   )
+  (wire (pts (xy 90.17 330.2) (xy 92.71 330.2))
+    (stroke (width 0) (type default))
+  )
   (wire (pts (xy 255.27 100.33) (xy 234.95 100.33))
     (stroke (width 0) (type default))
@@
     (stroke (width 0) (type default))
   )
+  (wire (pts (xy 86.36 332.74) (xy 86.36 359.41))
+    (stroke (width 0) (type default))
+  )
   (wire (pts (xy 34.29 142.24) (xy 234.95 142.24))
     (stroke (width 0) (type default))
@@
     (stroke (width 0) (type default))
   )
+  (wire (pts (xy 86.36 359.41) (xy 69.85 359.41))
+    (stroke (width 0) (type default))
+  )
   (wire (pts (xy 231.14 332.74) (xy 228.6 332.74))
     (stroke (width 0) (type default))
@@
     (stroke (width 0) (type default))
   )
+  (wire (pts (xy 90.17 373.38) (xy 90.17 330.2))
+    (stroke (width 0) (type default))
+  )
   (wire (pts (xy 255.27 143.51) (xy 255.27 144.78))
     (stroke (width 0) (type default))
@@
     (stroke (width 0) (type default))
   )
-  (wire (pts (xy 86.36 330.2) (xy 86.36 332.74))
-    (stroke (width 0) (type default))
-  )
   (wire (pts (xy 21.59 134.62) (xy 21.59 137.16))
     (stroke (width 0) (type default))
@@
     (stroke (width 0) (type default))
   )
+  (wire (pts (xy 69.85 359.41) (xy 69.85 384.81))
+    (stroke (width 0) (type default))
+  )
   (wire (pts (xy 34.29 213.36) (xy 46.99 213.36))
     (stroke (width 0) (type default))
@@
     (stroke (width 0) (type default))
   )
+  (wire (pts (xy 69.85 384.81) (xy 59.69 384.81))
+    (stroke (width 0) (type default))
+  )
   (wire (pts (xy 240.03 95.25) (xy 255.27 95.25))
     (stroke (width 0) (type default))
@@
   )
   (wire (pts (xy 255.27 204.47) (xy 255.27 205.74))
-    (stroke (width 0) (type default))
-  )
-  (wire (pts (xy 92.71 330.2) (xy 86.36 330.2))
     (stroke (width 0) (type default))
   )
@@
   )
   (label "X" (at 255.27 152.4 0) (fields_autoplaced)
-    (effects (font (size 1.27 1.27)) (justify left bottom))
-  )
-  (label "VP" (at 82.55 332.74 0) (fields_autoplaced)
     (effects (font (size 1.27 1.27)) (justify left bottom))
   )
@@
     )
   )
+  (symbol (lib_id "74xx:74HC74") (at 86.36 407.67 0) (unit 2)
+    (in_bom yes) (on_board yes) (dnp no) (fields_autoplaced)
+    (property "Reference" "U2" (at 88.5541 397.51 0)
+      (effects (font (size 1.27 1.27)) (justify left))
+    )
+    (property "Value" "74HC74" (at 88.5541 400.05 0)
+      (effects (font (size 1.27 1.27)) (justify left))
+    )
+    (property "Footprint" "" (at 86.36 407.67 0)
+      (effects (font (size 1.27 1.27)) hide)
+    )
+    (property "Datasheet" "74xx/74hc_hct74.pdf" (at 86.36 407.67 0)
+      (effects (font (size 1.27 1.27)) hide)
+    )
+    (pin "10")
+    (pin "3")
+    (pin "12")
+    (pin "8")
+    (pin "9")
+    (pin "7")
+    (pin "14")
+    (pin "4")
+    (pin "13")
+    (pin "6")
+    (pin "1")
+    (pin "5")
+    (pin "11")
+    (pin "2")
+    (instances
+      (project "VectorPullRewrite"
+        (path "/d5dd207c-6901-46da-bdf5-6dd9d69a2f13"
+          (reference "U2") (unit 2)
+        )
+      )
+    )
+  )
   (symbol (lib_id "power:GND") (at 73.66 309.88 0) (unit 1)
     (in_bom yes) (on_board yes) (dnp no)
@@
         (path "/d5dd207c-6901-46da-bdf5-6dd9d69a2f13"
           (reference "R15") (unit 1)
+        )
+      )
+    )
+  )
+  (symbol (lib_id "74xx:74HC74") (at 105.41 407.67 0) (unit 3)
+    (in_bom yes) (on_board yes) (dnp no) (fields_autoplaced)
+    (property "Reference" "U2" (at 111.76 406.4 0)
+      (effects (font (size 1.27 1.27)) (justify left))
+    )
+    (property "Value" "74HC74" (at 111.76 408.94 0)
+      (effects (font (size 1.27 1.27)) (justify left))
+    )
+    (property "Footprint" "" (at 105.41 407.67 0)
+      (effects (font (size 1.27 1.27)) hide)
+    )
+    (property "Datasheet" "74xx/74hc_hct74.pdf" (at 105.41 407.67 0)
+      (effects (font (size 1.27 1.27)) hide)
+    )
+    (pin "10")
+    (pin "3")
+    (pin "12")
+    (pin "8")
+    (pin "9")
+    (pin "7")
+    (pin "14")
+    (pin "4")
+    (pin "13")
+    (pin "6")
+    (pin "1")
+    (pin "5")
+    (pin "11")
+    (pin "2")
+    (instances
+      (project "VectorPullRewrite"
+        (path "/d5dd207c-6901-46da-bdf5-6dd9d69a2f13"
+          (reference "U2") (unit 3)
         )
       )
@@
         )
       )
+    )
+  )
+  (symbol (lib_id "74xx:74HC74") (at 59.69 372.11 0) (unit 1)
+    (in_bom yes) (on_board yes) (dnp no) (fields_autoplaced)
+    (property "Reference" "U2" (at 61.8841 361.95 0)
+      (effects (font (size 1.27 1.27)) (justify left))
+    )
+    (property "Value" "74HC74" (at 61.8841 364.49 0)
+      (effects (font (size 1.27 1.27)) (justify left))
+    )
+    (property "Footprint" "" (at 59.69 372.11 0)
+      (effects (font (size 1.27 1.27)) hide)
+    )
+    (property "Datasheet" "74xx/74hc_hct74.pdf" (at 59.69 372.11 0)
+      (effects (font (size 1.27 1.27)) hide)
+    )
+    (pin "10")
+    (pin "3")
+    (pin "12")
+    (pin "8")
+    (pin "9")
+    (pin "7")
+    (pin "14")
+    (pin "4")
+    (pin "13")
+    (pin "6")
+    (pin "1")
+    (pin "5")
+    (pin "11")
+    (pin "2")
+    (instances
+      (project "VectorPullRewrite"
+        (path "/d5dd207c-6901-46da-bdf5-6dd9d69a2f13"
+          (reference "U2") (unit 1)
+        )
+      )

Commit message: vpb
Parts:
- removed D1: 1N4148, Diode_THT:D_DO-35_SOD27_P7.62mm_Horizontal, symbol Diode:1N4148
- removed J10: ~{IRQ7_NMI}, symbol Connector_Generic:Conn_02x02_Odd_Even
- removed J12, J5: Conn_02x40_Odd_Even, Connector_PinHeader_2.54mm:PinHeader_2x40_P2.54mm_Vertical, symbol Connector_Generic:Conn_02x40_Odd_Even
- removed J13: DMA, Connector_PinHeader_2.54mm:PinHeader_2x18_P2.54mm_Vertical, symbol Connector_Generic:Conn_02x18_Odd_Even
- removed J6: CPU, Connector_PinHeader_2.54mm:PinHeader_2x18_P2.54mm_Vertical, symbol Connector_Generic:Conn_02x18_Odd_Even
- removed J7: VP Bypass, symbol Connector_Generic:Conn_02x04_Counter_Clockwise
- removed J9: ~{IRQ IN}, symbol Connector_Generic:Conn_02x08_Odd_Even
- removed R12, R13, R14: 10K, symbol Device:R
- removed U1: 74HC08, symbol Vega816:74HC08
- removed U2: 74HC74, symbol 74xx:74HC74
- removed U4: 74HC00, symbol 74xx:74HC00
- added U1: 74LS138, symbol 74xx:74LS138
- R1, R2: value 1K -> 10K
- renumbered D2 to D1, U9 to U2
Connections:
- net ~{IRQ7} is gone; now on net ~{IRQ4}: R6.1
- net ~{NMI} is gone; now on net VCC: R11.2
- net A1: now also U1.6 (E3)
- net A2: now also U1.1 (A0)
- net A3: now also U1.2 (A1)
- net A4: now also U1.3 (A2)
- net AA1: now also U3.4 (S1); no longer U3.10 (S4)
- net AA2: now also U3.1 (S2); no longer U3.13 (S3)
- net AA3: now also U3.13 (S3); no longer U3.1 (S2)
- net AA4: now also U3.10 (S4); no longer U3.4 (S1)
- net E: now also U1.4 (E1)
- net GND: now also U1.8 (GND); no longer R1.2, R2.2, R7.1, U2.11 (1)
- net VCC: now also R1.2, R2.2, U1.16 (VCC); no longer R11.1
- net VP_REQ: now also U1.12 (O3)
- net ~{IRQ0}: now also R10.1
- net ~{IRQ1}: now also R9.1
- net ~{IRQ2}: now also R8.1
- net ~{IRQ3}: now also R7.1; no longer R10.1
- net ~{IRQ4}: no longer R9.1
- net ~{IRQ5}: now also R2.1; no longer R8.1
- net ~{IRQ}: no longer D1.1 (K), U2.14 (GS)
- net at U2.10 (0): now also R11.1
- net ~{IRQ6}: now reaches R1.1
- net ~{IRQ6}: now also U2.11 (1)
- new net: D1.1 (K), U2.14 (GS)
- new net ~{VPB}: U1.5 (E2)
- no-connect marks 2 -> 9
Other:
- note added: "Active (low) when: E is low (native mode) AND VPB is low (vector pull active) AND A4 is low (pulling $Ex) AND A1-A3 are high (pulling $xE or $xF), indicating fetch of IRQ vector."
- note added: "Vector Pull Rewrite for W65C816"
- note added: "Vector Table (after rewrite) $FFE4 COP $FFE6 BRK $FFE8 ABORT $FFEA NMI $FFEE IRQ 0 $FFF0 IRQ 1 $FFF2 IRQ 2 $FFF4 IRQ 3 $FFF6 IRQ 4 $FFF8 IRQ 5 $FFFA IRQ 6 $FFFC RESET"
- note added: "Vector Table (before rewrite) $FFE4 COP $FFE6 BRK $FFE8 ABORT $FFEA NMI $FFEE IRQ $FFFC RESET"
- note removed: "4 bit adder"
- note removed: "BB816 CPU Breakout Rev. A.27"
- note removed: "IRQ Priority"
- note removed: "IRQ VP Detection"
- note removed: "To Bus"
- note removed: "VP_REQ is high when A1-A3 are high ($E or $F) and VP is active (low), indicating fetch of IRQ vector."
- note removed: "Vector Pull Rewrite for BB816 Breakout Board"
- company: (none) -> Alan Canon
- title: (none) -> Vector Pull Rewrite for W65C816
- moved on the sheet: D1, R15, R3, R4, R5, U2, U3
